File: untitled.kicad_sch (KiCad schematic)
At the start: 0 parts

Commit message: 23.09.2025
Parts:
- added C2, C3, C4: 10uF, Capacitor_SMD:C_1210_3225Metric, symbol #dzdb:s_cap/C-MUR-GRM32EC72A106KE05
