File: CM4_Module1A.kicad_sch (KiCad schematic)
At the start: 1 part

Commit message: multiple changes. fixed some mistakes, added jumper pins for wifi
Parts:
- added C10, C11, C12, C8, C9: 10pF, Capacitor_SMD:C_0603_1608Metric, symbol #dzdb:g_cap/C-10p-0603
- added C7: 100nF, Capacitor_SMD:C_0603_1608Metric, symbol #dzdb:g_cap/C-100n-0603
- added J7: 61300211121, dz_con:Wurth_Con_61300211121, symbol #dzdb:s_con/WURT-61300211121
Connections:
- net +5V: now also C10.1, C11.1, C12.1, C7.1, C8.1, C9.1
- net GND: now also C10.2, C11.2, C12.2, C7.2, C8.2, C9.2, J7.1
- net at Module1.84 (+3.3v_(Output)): no longer Module1.86 (+3.3v_(Output))
- net at Module1.88 (+1.8v_(Output)): no longer Module1.90 (+1.8v_(Output))
- net at Module1.89 (WL_nDisable): now also J7.2
- net ID_SC: no longer names the net of Module1.35 (ID_SC)
- net SD_CLK: no longer names the net of Module1.57 (SD_CLK)
- no-connect marks 12 -> 45
Other:
- note added: "sync todo!!!"
- note removed: "Serial needs clock?"
- note removed: "no."

Commit message: power led
Parts:
- added C13: 10pF, Capacitor_SMD:C_0603_1608Metric, symbol #dzdb:g_cap/C-10p-0603
Connections:
- net +5V: now also C13.1
- net GND: now also C13.2
Other:
- moved on the sheet: C10, C11, C12, C7, C8, C9
