File: 3.3V_Logic.kicad_sch (KiCad schematic)
At the start: 13 parts

Commit message: some PCB thoughts
Connections:
- net GND: no longer C28.2, C30.2, IC5.5 (OV1), R22.1
- new net: C28.2, C30.2, IC5.5 (OV1), R22.1
Changed lines of the file:
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@@
-	)
-	(junction
-		(at 74.93 96.52)
-		(diameter 0)
-		(color 0 0 0 0)
 	)
 	(junction
@@
 	(wire
 		(pts
-			(xy 74.93 96.52) (xy 74.93 107.95)
-		)
-		(stroke
+			(xy 63.5 107.95) (xy 74.93 107.95)
+		)
+		(stroke

Commit message: added Gyroscope and Accelerometer part (4x) over IIC
Parts:
- IC5: value ~ -> TPS2121RUXT
Changed lines of the file:
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@@
 			)
 		)
-		(property "Value" "~"
+		(property "Value" "TPS2121RUXT"
 			(at 139.7 118.11 0)
 			(effects

Commit message: new outline of board plus first traces
Connections:
- net GND: now also C28.2, C30.2, IC5.5 (OV1), R22.1
Changed lines of the file:
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@@
+	)
+	(junction
+		(at 74.93 96.52)
+		(diameter 0)
+		(color 0 0 0 0)
 	)
 	(junction
@@
 	(wire
 		(pts
+			(xy 74.93 107.95) (xy 74.93 96.52)
+		)
+		(stroke
+			(width 0)
+			(type default)
+		)
+	)
+	(wire
+		(pts
 			(xy 114.3 110.49) (xy 114.3 119.38)
 		)
@@
 		)
 		(stroke
-			(width 0)
-			(type default)
-		)
-	)
-	(wire
-		(pts
-			(xy 63.5 107.95) (xy 74.93 107.95)
-		)
-		(stroke

Commit message: multiple chainges on PCB
Parts:
- IC5: Order (none) -> Ordered=True
Changed lines of the file:
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@@
+			)
+		)
+		(property "Order" "Ordered=True"
+			(at 125.73 85.09 0)
+			(effects
+				(font
+					(size 1.27 1.27)
+				)
+				(hide yes)
 			)
 		)

Commit message: Power changes
Parts:
- renumbered C28 to C21, C29 to C22, C30 to C23, C31 to C24, C32 to C25, C33 to C26, C34 to C27, IC5 to IC3, R21 to R14, R22 to R16, R23 to R17, R24 to R18, R25 to R19
Changed lines of the file:
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@@
 		(dnp no)
 		(fields_autoplaced yes)
-		(property "Reference" "IC5"
+		(property "Reference" "IC3"
 			(at 139.7 115.57 0)
 			(effects
@@
 		)
 		(instances
-			(project ""
-				(path "/ce1819b2-f280-40ed-834f-6fe4d12f809d/c1998c4d-3f9a-4761-b447-a813532738a0/85d0d345-ed3a-4658-9370-48b549969854"
-					(reference "IC5")
+			(project "nautilus_mainboard"
+				(path "/ce1819b2-f280-40ed-834f-6fe4d12f809d/c1998c4d-3f9a-4761-b447-a813532738a0/b867d855-894b-4aa9-b170-e48a88a70717"
+					(reference "IC3")
 					(unit 1)
 				)
@@
 		(dnp no)
 		(fields_autoplaced yes)
-		(property "Reference" "R24"
+		(property "Reference" "R18"
 			(at 172.72 95.2499 0)
 			(effects
@@
 		(instances
 			(project "nautilus_mainboard"
-				(path "/ce1819b2-f280-40ed-834f-6fe4d12f809d/c1998c4d-3f9a-4761-b447-a813532738a0/85d0d345-ed3a-4658-9370-48b549969854"
-					(reference "R24")
+				(path "/ce1819b2-f280-40ed-834f-6fe4d12f809d/c1998c4d-3f9a-4761-b447-a813532738a0/b867d855-894b-4aa9-b170-e48a88a70717"
+					(reference "R18")
 					(unit 1)
 				)
@@
 		(on_board yes)
 		(dnp no)
-		(property "Reference" "C29"
+		(property "Reference" "C22"
 			(at 108.966 101.854 0)
 			(effects
@@
 		(instances
 			(project "nautilus_mainboard"
-				(path "/ce1819b2-f280-40ed-834f-6fe4d12f809d/c1998c4d-3f9a-4761-b447-a813532738a0/85d0d345-ed3a-4658-9370-48b549969854"
-					(reference "C29")
+				(path "/ce1819b2-f280-40ed-834f-6fe4d12f809d/c1998c4d-3f9a-4761-b447-a813532738a0/b867d855-894b-4aa9-b170-e48a88a70717"
+					(reference "C22")
 					(unit 1)
 				)
@@
 		(on_board yes)
 		(dnp no)
-		(property "Reference" "C31"
+		(property "Reference" "C24"
 			(at 117.348 102.108 0)
 			(effects
@@
 		(instances
 			(project "nautilus_mainboard"
-				(path "/ce1819b2-f280-40ed-834f-6fe4d12f809d/c1998c4d-3f9a-4761-b447-a813532738a0/85d0d345-ed3a-4658-9370-48b549969854"
-					(reference "C31")
+				(path "/ce1819b2-f280-40ed-834f-6fe4d12f809d/c1998c4d-3f9a-4761-b447-a813532738a0/b867d855-894b-4aa9-b170-e48a88a70717"
+					(reference "C24")
 					(unit 1)
 				)
@@
 		(dnp no)
 		(fields_autoplaced yes)
-		(property "Reference" "#PWR032"
+		(property "Reference" "#PWR015"
 			(at 162.56 125.73 0)
 			(effects
@@
 		(instances
 			(project "nautilus_mainboard"
-				(path "/ce1819b2-f280-40ed-834f-6fe4d12f809d/c1998c4d-3f9a-4761-b447-a813532738a0/85d0d345-ed3a-4658-9370-48b549969854"
-					(reference "#PWR032")
+				(path "/ce1819b2-f280-40ed-834f-6fe4d12f809d/c1998c4d-3f9a-4761-b447-a813532738a0/b867d855-894b-4aa9-b170-e48a88a70717"
+					(reference "#PWR015")
 					(unit 1)
 				)
@@
 		(on_board yes)
 		(dnp no)
-		(property "Reference" "C32"
+		(property "Reference" "C25"
 			(at 157.48 105.41 90)
 			(effects
@@
 		(instances
 			(project "nautilus_mainboard"
-				(path "/ce1819b2-f280-40ed-834f-6fe4d12f809d/c1998c4d-3f9a-4761-b447-a813532738a0/85d0d345-ed3a-4658-9370-48b549969854"
-					(reference "C32")
+				(path "/ce1819b2-f280-40ed-834f-6fe4d12f809d/c1998c4d-3f9a-4761-b447-a813532738a0/b867d855-894b-4aa9-b170-e48a88a70717"
+					(reference "C25")
 					(unit 1)
 				)
@@
 		(dnp no)
 		(fields_autoplaced yes)
-		(property "Reference" "R25"
+		(property "Reference" "R19"
 			(at 172.72 102.8699 0)
 			(effects
@@
 		(instances
 			(project "nautilus_mainboard"
-				(path "/ce1819b2-f280-40ed-834f-6fe4d12f809d/c1998c4d-3f9a-4761-b447-a813532738a0/85d0d345-ed3a-4658-9370-48b549969854"
-					(reference "R25")
+				(path "/ce1819b2-f280-40ed-834f-6fe4d12f809d/c1998c4d-3f9a-4761-b447-a813532738a0/b867d855-894b-4aa9-b170-e48a88a70717"
+					(reference "R19")
 					(unit 1)
 				)
@@
 		(on_board yes)
 		(dnp no)
-		(property "Reference" "C33"
+		(property "Reference" "C26"
 			(at 156.718 87.122 0)
 			(effects
@@
 		(instances
 			(project "nautilus_mainboard"
-				(path "/ce1819b2-f280-40ed-834f-6fe4d12f809d/c1998c4d-3f9a-4761-b447-a813532738a0/85d0d345-ed3a-4658-9370-48b549969854"
-					(reference "C33")
+				(path "/ce1819b2-f280-40ed-834f-6fe4d12f809d/c1998c4d-3f9a-4761-b447-a813532738a0/b867d855-894b-4aa9-b170-e48a88a70717"
+					(reference "C26")
 					(unit 1)
 				)
@@
 		(on_board yes)
 		(dnp no)
-		(property "Reference" "R23"
+		(property "Reference" "R17"
 			(at 157.48 102.87 90)
 			(effects
@@
 		)
 		(instances
-			(project ""
-				(path "/ce1819b2-f280-40ed-834f-6fe4d12f809d/c1998c4d-3f9a-4761-b447-a813532738a0/85d0d345-ed3a-4658-9370-48b549969854"
-					(reference "R23")
+			(project "nautilus_mainboard"
+				(path "/ce1819b2-f280-40ed-834f-6fe4d12f809d/c1998c4d-3f9a-4761-b447-a813532738a0/b867d855-894b-4aa9-b170-e48a88a70717"
+					(reference "R17")
 					(unit 1)
 				)
@@
 		(dnp no)
 		(fields_autoplaced yes)
-		(property "Reference" "R22"
+		(property "Reference" "R16"
 			(at 138.43 64.7699 0)
 			(effects
@@
 		(instances
 			(project "nautilus_mainboard"
-				(path "/ce1819b2-f280-40ed-834f-6fe4d12f809d/c1998c4d-3f9a-4761-b447-a813532738a0/85d0d345-ed3a-4658-9370-48b549969854"
-					(reference "R22")
+				(path "/ce1819b2-f280-40ed-834f-6fe4d12f809d/c1998c4d-3f9a-4761-b447-a813532738a0/b867d855-894b-4aa9-b170-e48a88a70717"
+					(reference "R16")
 					(unit 1)
 				)
@@
 		(on_board yes)
 		(dnp no)
-		(property "Reference" "R21"
+		(property "Reference" "R14"
 			(at 123.19 83.312 90)
 			(effects
@@
 		(instances
 			(project "nautilus_mainboard"
-				(path "/ce1819b2-f280-40ed-834f-6fe4d12f809d/c1998c4d-3f9a-4761-b447-a813532738a0/85d0d345-ed3a-4658-9370-48b549969854"
-					(reference "R21")
+				(path "/ce1819b2-f280-40ed-834f-6fe4d12f809d/c1998c4d-3f9a-4761-b447-a813532738a0/b867d855-894b-4aa9-b170-e48a88a70717"
+					(reference "R14")
 					(unit 1)
 				)
@@
 		(on_board yes)
 		(dnp no)
-		(property "Reference" "C28"
+		(property "Reference" "C21"
 			(at 108.966 86.614 0)
 			(effects
@@
 		(instances
 			(project "nautilus_mainboard"
-				(path "/ce1819b2-f280-40ed-834f-6fe4d12f809d/c1998c4d-3f9a-4761-b447-a813532738a0/85d0d345-ed3a-4658-9370-48b549969854"
-					(reference "C28")
+				(path "/ce1819b2-f280-40ed-834f-6fe4d12f809d/c1998c4d-3f9a-4761-b447-a813532738a0/b867d855-894b-4aa9-b170-e48a88a70717"
+					(reference "C21")
 					(unit 1)
 				)
@@
 		(on_board yes)
 		(dnp no)
-		(property "Reference" "C30"
+		(property "Reference" "C23"
 			(at 117.602 87.122 0)
 			(effects
@@
 		(instances
 			(project "nautilus_mainboard"
-				(path "/ce1819b2-f280-40ed-834f-6fe4d12f809d/c1998c4d-3f9a-4761-b447-a813532738a0/85d0d345-ed3a-4658-9370-48b549969854"
-					(reference "C30")
+				(path "/ce1819b2-f280-40ed-834f-6fe4d12f809d/c1998c4d-3f9a-4761-b447-a813532738a0/b867d855-894b-4aa9-b170-e48a88a70717"
+					(reference "C23")
 					(unit 1)
 				)
@@
 		(on_board yes)
 		(dnp no)
-		(property "Reference" "C34"
+		(property "Reference" "C27"
 			(at 164.846 86.614 0)
 			(effects
@@
 		(instances
 			(project "nautilus_mainboard"
-				(path "/ce1819b2-f280-40ed-834f-6fe4d12f809d/c1998c4d-3f9a-4761-b447-a813532738a0/85d0d345-ed3a-4658-9370-48b549969854"
-					(reference "C34")
+				(path "/ce1819b2-f280-40ed-834f-6fe4d12f809d/c1998c4d-3f9a-4761-b447-a813532738a0/b867d855-894b-4aa9-b170-e48a88a70717"
+					(reference "C27")
 					(unit 1)
 				)

Commit message: fix: 2 ERC errors fixed
Connections:
- net STM_IN_3.3V renamed +3.3V
Changed lines of the file:
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@@
 	(text "100nF CLOSE"
 		(exclude_from_sim no)
-		(at 122.936 97.536 0)
+		(at 116.332 98.044 0)
 		(effects
 			(font
@@
 			)
 			(justify right)
-		)
-	)
-	(hierarchical_label "STM_IN_3.3V"
-		(shape output)
-		(at 172.72 85.09 0)
-		(effects
-			(font
-				(size 1.27 1.27)
-			)
-			(justify left)
 		)
 	)
@@
 		(dnp no)
 		(property "Reference" "C22"
-			(at 108.966 101.854 0)
+			(at 106.172 101.854 0)
 			(effects
 				(font
@@
 		)
 		(property "Value" "10uF"
-			(at 108.458 106.426 0)
+			(at 105.41 106.426 0)
 			(effects
 				(font
@@
 		(dnp no)
 		(property "Reference" "C24"
-			(at 117.348 102.108 0)
+			(at 115.062 101.854 0)
 			(effects
 				(font
@@
 		)
 		(property "Value" "100nF"
-			(at 116.332 106.172 0)
+			(at 113.284 106.426 0)
 			(effects
 				(font
@@
 		(dnp no)
 		(property "Reference" "C25"
-			(at 157.48 105.41 90)
+			(at 160.782 105.41 90)
 			(effects
 				(font
@@
 		)
 		(property "Value" "330nF"
-			(at 157.734 107.95 90)
+			(at 161.798 108.204 90)
 			(effects
 				(font
@@
 	)
 	(symbol
+		(lib_id "power:+3.3V")
+		(at 172.72 85.09 0)
+		(unit 1)
+		(exclude_from_sim no)
+		(in_bom yes)
+		(on_board yes)
+		(dnp no)
+		(fields_autoplaced yes)
+		(property "Reference" "#PWR033"
+			(at 172.72 88.9 0)
+			(effects
+				(font
+					(size 1.27 1.27)
+				)
+				(hide yes)
+			)
+		)
+		(property "Value" "+3.3V"
+			(at 172.72 80.01 0)
+			(effects
+				(font
+					(size 1.27 1.27)
+				)
+			)
+		)
+		(property "Footprint" ""
+			(at 172.72 85.09 0)
+			(effects
+				(font
+					(size 1.27 1.27)
+				)
+				(hide yes)
+			)
+		)
+		(property "Datasheet" ""
+			(at 172.72 85.09 0)
+			(effects
+				(font
+					(size 1.27 1.27)
+				)
+				(hide yes)
+			)
+		)
+		(property "Description" "Power symbol creates a global label with name \"+3.3V\""
+			(at 172.72 85.09 0)
+			(effects
+				(font
+					(size 1.27 1.27)
+				)
+				(hide yes)
+			)
+		)
+		(pin "1"
+		)
+		(instances
+			(project ""
+				(path "/ce1819b2-f280-40ed-834f-6fe4d12f809d/c1998c4d-3f9a-4761-b447-a813532738a0/b867d855-894b-4aa9-b170-e48a88a70717"
+					(reference "#PWR033")
+					(unit 1)
+				)
+			)
+		)
+	)
+	(symbol
 		(lib_id "#dzdb:g_res/R-15.4k-0603")
 		(at 123.19 81.28 0)
@@
 		(dnp no)
 		(property "Reference" "C21"
-			(at 108.966 86.614 0)
+			(at 105.918 86.614 0)
 			(effects
 				(font
@@
 		)
 		(property "Value" "10uF"
-			(at 108.458 91.186 0)
+			(at 105.41 91.186 0)
 			(effects
 				(font
@@
 		(dnp no)
 		(property "Reference" "C23"
-			(at 117.602 87.122 0)
+			(at 114.554 87.122 0)
 			(effects
 				(font
@@
 		)
 		(property "Value" "100nF"
-			(at 116.078 90.932 0)
-			(effects
-				(font
+			(at 113.03 90.932 0)
+			(effects
+				(font

Commit message: chore: Many routing changes
Connections:
- net +3.3V renamed STM_In_3.3V
Changed lines of the file:
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@@
+		)
+	)
+	(hierarchical_label "STM_In_3.3V"
+		(shape output)
+		(at 172.72 85.09 0)
+		(effects
+			(font
+				(size 1.27 1.27)
+			)
+			(justify left)
 		)
 	)
@@
 					(unit 1)
 				)
-			)
-		)
-	)
-	(symbol
-		(lib_id "power:+3.3V")
-		(at 172.72 85.09 0)
-		(unit 1)
-		(exclude_from_sim no)
-		(in_bom yes)
-		(on_board yes)
-		(dnp no)
-		(fields_autoplaced yes)
-		(property "Reference" "#PWR033"
-			(at 172.72 88.9 0)
-			(effects
-				(font
-					(size 1.27 1.27)
-				)
-				(hide yes)
-			)
-		)
-		(property "Value" "+3.3V"
-			(at 172.72 80.01 0)
-			(effects
-				(font
-					(size 1.27 1.27)
-				)
-			)
-		)
-		(property "Footprint" ""
-			(at 172.72 85.09 0)
-			(effects
-				(font
-					(size 1.27 1.27)
-				)
-				(hide yes)
-			)
-		)
-		(property "Datasheet" ""
-			(at 172.72 85.09 0)
-			(effects
-				(font
-					(size 1.27 1.27)
-				)
-				(hide yes)
-			)
-		)
-		(property "Description" "Power symbol creates a global label with name \"+3.3V\""
-			(at 172.72 85.09 0)
-			(effects
-				(font
-					(size 1.27 1.27)
-				)
-				(hide yes)
-			)
-		)
-		(pin "1"
-		)
-		(instances
-			(project ""
-				(path "/ce1819b2-f280-40ed-834f-6fe4d12f809d/c1998c4d-3f9a-4761-b447-a813532738a0/b867d855-894b-4aa9-b170-e48a88a70717"
-					(reference "#PWR033")
-					(unit 1)
-				)
