File: 3.3V_Logic.kicad_sch (KiCad schematic)
At the start: 13 parts, among them IC3 TPS2121RUXT

Commit message: chore: more cleanup
Parts:
- removed IC3: TPS2121RUXT, dz_dio:TI_Switchover_TPS2121RUXT, symbol #dzdb:s_misc/TEXA-595-TPS2121RUXT
- removed R14: 15.4k, Resistor_SMD:R_0603_1608Metric, symbol #dzdb:g_res/R-15.4k-0603
- removed R16, R18: 4.99k, Resistor_SMD:R_0603_1608Metric, symbol #dzdb:g_res/R-4.99k-0603
- removed R19: 20k, Resistor_SMD:R_0603_1608Metric, symbol #dzdb:g_res/R-20k-0603
- added IC6: TPS2121RUXT, dz_dio:TI_Switchover_TPS2121RUXT, symbol #dzdb:s_misc/TEXA-595-TPS2121RUXT
Connections:
- net Battery_Out_3.3V: now also IC6.6 (PR1), IC6.7 (IN1)
- net GND: now also C25.1, IC6.12 (GND), IC6.3 (CP2), IC6.4 (OV2), IC6.5 (OV1); no longer C25.2
- net STM_In_3.3V: now also IC6.1 (OUT_1), IC6.8 (OUT_2)
- net STM_Plug_3.3V: now also IC6.2 (IN2)
- net at R17.1: now also IC6.10 (ILIM)
- new net: C25.2, IC6.11 (SS)
Other:
- note removed: "100nF CLOSE"
- note removed: "SAME AS IN 5V"
- note removed: "V-div (same ratio as 5V)"
- company: (none) -> Davide
- moved on the sheet: C21, C22, C23, C24, C25, C26, C27, R17

Commit message: chore: Loads of redoing stuff. Added a Changelog
Other:
- title: (none) -> Nautilus_Mainboard
Changed lines of the file:
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@@
 	(paper "A4")
 	(title_block
+		(title "Nautilus_Mainboard")
 		(date "2025-11-19")
 		(rev "0")

Commit message: fix: minor changes, preparations for BOM and gerber, added Stitching
Parts:
- C25: Comment lifecycle=Active; note=Auto-generated -> lifecycle=Active; note: previous part not found.; MPN 885012206098 -> 885012106007; SPN 710-885012206098 -> 710-885012106007; Tolerance 10% -> 20%; Voltage 50V -> 10V
Changed lines of the file:
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@@
+			)
+		)
+		(property "Field16" ""
+			(at 104.14 110.49 0)
+			(effects
+				(font
+					(size 1.27 1.27)
+				)
+				(hide yes)
+			)
+		)
+		(property "Sim.Pins" ""
+			(at 104.14 110.49 0)
+			(effects
+				(font
+					(size 1.27 1.27)
+				)
+				(hide yes)
 			)
 		)
@@
 			)
 		)
+		(property "Field16" ""
+			(at 113.03 110.49 0)
+			(effects
+				(font
+					(size 1.27 1.27)
+				)
+				(hide yes)
+			)
+		)
+		(property "Sim.Pins" ""
+			(at 113.03 110.49 0)
+			(effects
+				(font
+					(size 1.27 1.27)
+				)
+				(hide yes)
+			)
+		)
 		(pin "2"
 		)
@@
 			)
 		)
-		(property "Description" "Cap 330nF 50V 0603 C0G ±10%"
+		(property "Description" "Cap 330nF 10V 0603 C0G ±10%"
 			(at 165.1 106.68 0)
 			(effects
@@
 			)
 		)
-		(property "MPN" "885012206098"
+		(property "MPN" "885012106007"
 			(at 165.1 106.68 0)
 			(effects
@@
 			)
 		)
-		(property "Voltage" "50V"
+		(property "Voltage" "10V"
 			(at 165.1 106.68 0)
 			(effects
@@
 			)
 		)
-		(property "Tolerance" "10%"
+		(property "Tolerance" "20%"
 			(at 165.1 106.68 0)
 			(effects
@@
 			)
 		)
-		(property "SPN" "710-885012206098"
+		(property "SPN" "710-885012106007"
 			(at 165.1 106.68 0)
 			(effects
@@
 			)
 		)
-		(property "Comment" "lifecycle=Active; note=Auto-generated"
+		(property "Comment" "lifecycle=Active; note: previous part not found."
+			(at 165.1 106.68 0)
+			(effects
+				(font
+					(size 1.27 1.27)
+				)
+				(hide yes)
+			)
+		)
+		(property "Field16" ""
+			(at 165.1 106.68 0)
+			(effects
+				(font
+					(size 1.27 1.27)
+				)
+				(hide yes)
+			)
+		)
+		(property "Sim.Pins" ""
 			(at 165.1 106.68 0)
 			(effects
@@
 			)
 		)
+		(property "Field16" ""
+			(at 123.19 87.63 0)
+			(effects
+				(font
+					(size 1.27 1.27)
+				)
+				(hide yes)
+			)
+		)
+		(property "Sim.Pins" ""
+			(at 123.19 87.63 0)
+			(effects
+				(font
+					(size 1.27 1.27)
+				)
+				(hide yes)
+			)
+		)
 		(pin "5"
 		)
@@
 			)
 		)
+		(property "Field16" ""
+			(at 165.1 86.36 0)
+			(effects
+				(font
+					(size 1.27 1.27)
+				)
+				(hide yes)
+			)
+		)
+		(property "Sim.Pins" ""
+			(at 165.1 86.36 0)
+			(effects
+				(font
+					(size 1.27 1.27)
+				)
+				(hide yes)
+			)
+		)
 		(pin "2"
 		)
@@
 			)
 		)
+		(property "Field16" ""
+			(at 158.75 115.57 90)
+			(effects
+				(font
+					(size 1.27 1.27)
+				)
+				(hide yes)
+			)
+		)
+		(property "Sim.Pins" ""
+			(at 158.75 115.57 90)
+			(effects
+				(font
+					(size 1.27 1.27)
+				)
+				(hide yes)
+			)
+		)
 		(pin "2"
 		)
@@
 			)
 		)
+		(property "Field16" ""
+			(at 104.14 85.09 0)
+			(effects
+				(font
+					(size 1.27 1.27)
+				)
+				(hide yes)
+			)
+		)
+		(property "Sim.Pins" ""
+			(at 104.14 85.09 0)
+			(effects
+				(font
+					(size 1.27 1.27)
+				)
+				(hide yes)
+			)
+		)
 		(pin "1"
 		)
@@
 			)
 		)
+		(property "Field16" ""
+			(at 113.03 85.09 0)
+			(effects
+				(font
+					(size 1.27 1.27)
+				)
+				(hide yes)
+			)
+		)
+		(property "Sim.Pins" ""
+			(at 113.03 85.09 0)
+			(effects
+				(font
+					(size 1.27 1.27)
+				)
+				(hide yes)
+			)
+		)
 		(pin "2"
 		)
@@
 			(at 172.72 86.36 0)
 			(effects
+				(font
+					(size 1.27 1.27)
+				)
+				(hide yes)
+			)
+		)
+		(property "Field16" ""
+			(at 172.72 86.36 0)
+			(effects
+				(font
+					(size 1.27 1.27)
+				)
+				(hide yes)
+			)
+		)
+		(property "Sim.Pins" ""
+			(at 172.72 86.36 0)
+			(effects
