File: nautilus_mainboard.kicad_sch (KiCad schematic)
At the start: 7 parts

Commit message: chore: more cleanup
Other:
- sheet STM ports: added Piezzo_Control; removed none
- note removed: "We should consider that we NEVER want the CM4 to power the unpowered STM over the TX pin. Found a neat part for that: https://www.mouser.ch/ProductDetail/Texas-Instruments/SN74LVC1G126DBVR?qs=pajgIaoyDUi3T2WgNNfd3w%3D%3D connections: Pin 5: VCC -> CM4_3V3 Pin 2: A -> CM4 TX (PLTX) Pin 4: Y -> STM_UART_RX Pin 1: OE -> STM_IN_3.3V Pin 3: GND 0.1uF decoupling cap VCC-GND 220 Ohm series at Y (to STM)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"
- company: (none) -> Evan & Davide
Changed lines of the file:
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@@
 	(generator_version "9.0")
 	(paper "A4")
-	(text "We should consider that we NEVER want the CM4 to power the unpowered STM\nover the TX pin. Found a neat part for that:\nhttps://www.mouser.ch/ProductDetail/Texas-Instruments/SN74LVC1G126DBVR?qs=pajgIaoyDUi3T2WgNNfd3w%3D%3D\n\nconnections:\nPin 5: VCC -> CM4_3V3\n\nPin 2: A -> CM4 TX (PLTX)\n\nPin 4: Y -> STM_UART_RX\n\nPin 1: OE -> STM_IN_3.3V\n\nPin 3: GND\n\n0.1uF decoupling cap VCC-GND\n\n220 Ohm series at Y (to STM). (current limiting)\n\n100 kOhm pull-down from OE to GND"
-		(exclude_from_sim no)
-		(at 74.422 180.848 0)
-		(effects
-			(font
-				(size 2 2)
-				(thickness 0.4)
-				(bold yes)
-				(color 44 31 255 1)
-			)
-			(justify left)
-		)
+	(title_block
+		(date "2025-11-18")
+		(company "Evan & Davide")
 	)
 	(text "Standard 5V and 3.3V for the components are sent out as globals."
@@
 	(wire
 		(pts
+			(xy 92.71 154.94) (xy 92.71 59.69)
+		)
+		(stroke
+			(width 0)
+			(type default)
+		)
+	)
+	(wire
+		(pts
 			(xy 163.83 81.28) (xy 163.83 113.03)
 		)
@@
 	(wire
 		(pts
-			(xy 95.25 59.69) (xy 95.25 85.09)
-		)
-		(stroke
-			(width 0)
-			(type default)
-		)
-	)
-	(wire
-		(pts
-			(xy 76.2 59.69) (xy 95.25 59.69)
+			(xy 95.25 57.15) (xy 95.25 85.09)
+		)
+		(stroke
+			(width 0)
+			(type default)
+		)
+	)
+	(wire
+		(pts
+			(xy 76.2 57.15) (xy 95.25 57.15)
+		)
+		(stroke
+			(width 0)
+			(type default)
+		)
+	)
+	(wire
+		(pts
+			(xy 165.1 140.97) (xy 165.1 154.94)
 		)
 		(stroke
@@
 	(wire
 		(pts
+			(xy 165.1 154.94) (xy 92.71 154.94)
+		)
+		(stroke
+			(width 0)
+			(type default)
+		)
+	)
+	(wire
+		(pts
 			(xy 152.4 52.07) (xy 177.8 52.07)
 		)
@@
 	(wire
 		(pts
+			(xy 176.53 140.97) (xy 165.1 140.97)
+		)
+		(stroke
+			(width 0)
+			(type default)
+		)
+	)
+	(wire
+		(pts
 			(xy 177.8 60.96) (xy 163.83 60.96)
 		)
@@
 		(pts
 			(xy 76.2 33.02) (xy 101.6 33.02)
+		)
+		(stroke
+			(width 0)
+			(type default)
+		)
+	)
+	(wire
+		(pts
+			(xy 76.2 59.69) (xy 92.71 59.69)
 		)
 		(stroke
@@
 		)
 		(pin "Battery_Out_3.3V" input
+			(at 76.2 57.15 0)
+			(effects
+				(font
+					(size 1.27 1.27)
+				)
+				(justify right)
+			)
+		)
+		(pin "Piezzo_Control" output
 			(at 76.2 59.69 0)
 			(effects
@@
 		)
 		(pin "Piezo_ctrl" input
-			(at 186.69 93.98 90)
-			(effects
-				(font
-					(size 1.27 1.27)
-				)
-				(justify right)
-			)
-		)
+			(at 176.53 140.97 180)
+			(effects
+				(font
+					(size 1.27 1.27)
+				)
+				(justify left)
+			)
+		)

Commit message: chore: added LED indicators for power and activity status, updated symbold, rerouted some things for better visibility
Parts:
- added TP10, TP11, TP12: TestPoint_Probe, TestPoint:TestPoint_Pad_D1.0mm, symbol Connector:TestPoint_Probe
Connections:
- net GND: now also TP10.1, TP11.1, TP12.1

Commit message: chore: Loads of redoing stuff. Added a Changelog
Parts:
- added TP13, TP14: TestPoint_Probe, TestPoint:TestPoint_Pad_D1.0mm, symbol Connector:TestPoint_Probe
Connections:
- new net +3.3V: TP13.1
- new net +5V: TP14.1
Other:
- sheet LPHS-connector ports: added STM{RX,TX}, ST_CAN{P,N}; removed none
- sheet STM ports: added STM{RX,TX}, ST_CAN{P,N}; removed none
- note added: "All 4 corners should have a testprobe for gnd. plus maybe a lil copper plane for a Krokodilzange :)"
- title: (none) -> Nautilus_Mainboard
- moved on the sheet: TP1, TP10, TP2, TP3, TP8
