File: IMU1.kicad_sch (KiCad schematic)
At the start: 3 parts, among them U4 262-BMI088

Commit message: new outline of board plus first traces
Parts:
- renumbered C48 to C43, C47 to C44, U4 to U2
Changed lines of the file:
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@@
 		(dnp no)
 		(fields_autoplaced yes)
-		(property "Reference" "#PWR043"
+		(property "Reference" "#PWR036"
 			(at 204.47 77.47 0)
 			(effects
@@
 				(path "/ce1819b2-f280-40ed-834f-6fe4d12f809d/bdf8f7d6-a5ee-4741-925d-5019e8cbdfce/0c7afee2-dd12-41f0-a704-0f15387072b0"
 					(reference "#PWR036")
-					(unit 1)
-				)
-				(path "/ce1819b2-f280-40ed-834f-6fe4d12f809d/bdf8f7d6-a5ee-4741-925d-5019e8cbdfce/aa94fdc5-ff6c-4519-87c9-a17e3d5a65da"
-					(reference "#PWR043")
 					(unit 1)
 				)
@@
 		(dnp no)
 		(fields_autoplaced yes)
-		(property "Reference" "#PWR040"
+		(property "Reference" "#PWR035"
 			(at 119.38 119.38 0)
 			(effects
@@
 				(path "/ce1819b2-f280-40ed-834f-6fe4d12f809d/bdf8f7d6-a5ee-4741-925d-5019e8cbdfce/0c7afee2-dd12-41f0-a704-0f15387072b0"
 					(reference "#PWR035")
-					(unit 1)
-				)
-				(path "/ce1819b2-f280-40ed-834f-6fe4d12f809d/bdf8f7d6-a5ee-4741-925d-5019e8cbdfce/aa94fdc5-ff6c-4519-87c9-a17e3d5a65da"
-					(reference "#PWR040")
 					(unit 1)
 				)
@@
 		(dnp no)
 		(fields_autoplaced yes)
-		(property "Reference" "C47"
+		(property "Reference" "C44"
 			(at 175.26 74.9299 0)
 			(effects
@@
 				(path "/ce1819b2-f280-40ed-834f-6fe4d12f809d/bdf8f7d6-a5ee-4741-925d-5019e8cbdfce/0c7afee2-dd12-41f0-a704-0f15387072b0"
 					(reference "C44")
-					(unit 1)
-				)
-				(path "/ce1819b2-f280-40ed-834f-6fe4d12f809d/bdf8f7d6-a5ee-4741-925d-5019e8cbdfce/aa94fdc5-ff6c-4519-87c9-a17e3d5a65da"
-					(reference "C47")
 					(unit 1)
 				)
@@
 		(dnp no)
 		(fields_autoplaced yes)
-		(property "Reference" "#PWR041"
+		(property "Reference" "#PWR023"
 			(at 176.53 119.38 0)
 			(effects
@@
 				(path "/ce1819b2-f280-40ed-834f-6fe4d12f809d/bdf8f7d6-a5ee-4741-925d-5019e8cbdfce/0c7afee2-dd12-41f0-a704-0f15387072b0"
 					(reference "#PWR023")
-					(unit 1)
-				)
-				(path "/ce1819b2-f280-40ed-834f-6fe4d12f809d/bdf8f7d6-a5ee-4741-925d-5019e8cbdfce/aa94fdc5-ff6c-4519-87c9-a17e3d5a65da"
-					(reference "#PWR041")
 					(unit 1)
 				)
@@
 		(dnp no)
 		(fields_autoplaced yes)
-		(property "Reference" "#PWR042"
+		(property "Reference" "#PWR034"
 			(at 185.42 55.88 0)
 			(effects
@@
 				(path "/ce1819b2-f280-40ed-834f-6fe4d12f809d/bdf8f7d6-a5ee-4741-925d-5019e8cbdfce/0c7afee2-dd12-41f0-a704-0f15387072b0"
 					(reference "#PWR034")
-					(unit 1)
-				)
-				(path "/ce1819b2-f280-40ed-834f-6fe4d12f809d/bdf8f7d6-a5ee-4741-925d-5019e8cbdfce/aa94fdc5-ff6c-4519-87c9-a17e3d5a65da"
-					(reference "#PWR042")
 					(unit 1)
 				)
@@
 		(dnp no)
 		(fields_autoplaced yes)
-		(property "Reference" "C48"
+		(property "Reference" "C43"
 			(at 189.23 77.4699 0)
 			(effects
@@
 				(path "/ce1819b2-f280-40ed-834f-6fe4d12f809d/bdf8f7d6-a5ee-4741-925d-5019e8cbdfce/0c7afee2-dd12-41f0-a704-0f15387072b0"
 					(reference "C43")
-					(unit 1)
-				)
-				(path "/ce1819b2-f280-40ed-834f-6fe4d12f809d/bdf8f7d6-a5ee-4741-925d-5019e8cbdfce/aa94fdc5-ff6c-4519-87c9-a17e3d5a65da"
-					(reference "C48")
 					(unit 1)
 				)
@@
 		(dnp no)
 		(fields_autoplaced yes)
-		(property "Reference" "U4"
+		(property "Reference" "U2"
 			(at 148.59 72.39 0)
 			(effects
@@
 					(unit 1)
 				)
-				(path "/ce1819b2-f280-40ed-834f-6fe4d12f809d/bdf8f7d6-a5ee-4741-925d-5019e8cbdfce/aa94fdc5-ff6c-4519-87c9-a17e3d5a65da"
-					(reference "U4")
-					(unit 1)
-				)

Commit message: multiple chainges on PCB
Parts:
- added BMI2, BMI2_SCL1, BMI2_SDA1: 0, Resistor_SMD:R_0603_1608Metric, symbol #dzdb:g_res/R-0-0603
Connections:
- net BMI_IN_3.3V: now also BMI2.1; no longer U2.14 (CSB1), U2.7 (PS)
- net IMU_SCL: now also BMI2_SCL1.1; no longer U2.8 (SCL/SCK)
- net IMU_SDA: now also BMI2_SDA1.1; no longer U2.9 (SDA/SDI)
- new net: BMI2.2, U2.14 (CSB1), U2.7 (PS)
- new net: BMI2_SCL1.2, U2.8 (SCL/SCK)
- new net: BMI2_SDA1.2, U2.9 (SDA/SDI)

Commit message: nearly complete with the PCB
Parts:
- renumbered BMI2 to BMI1, BMI2_SCL1 to BMI1_SCL1, BMI2_SDA1 to BMI1_SDA1, U2 to U1
Changed lines of the file:
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@@
 		(on_board yes)
 		(dnp no)
-		(property "Reference" "BMI2"
+		(property "Reference" "BMI1"
 			(at 124.46 87.63 90)
 			(effects
@@
 			(project "nautilus_mainboard"
 				(path "/ce1819b2-f280-40ed-834f-6fe4d12f809d/bdf8f7d6-a5ee-4741-925d-5019e8cbdfce/0c7afee2-dd12-41f0-a704-0f15387072b0"
-					(reference "BMI2")
+					(reference "BMI1")
 					(unit 1)
 				)
@@
 		(on_board yes)
 		(dnp no)
-		(property "Reference" "BMI2_SCL1"
+		(property "Reference" "BMI1_SCL1"
 			(at 124.46 97.79 90)
 			(effects
@@
 			(project "nautilus_mainboard"
 				(path "/ce1819b2-f280-40ed-834f-6fe4d12f809d/bdf8f7d6-a5ee-4741-925d-5019e8cbdfce/0c7afee2-dd12-41f0-a704-0f15387072b0"
-					(reference "BMI2_SCL1")
+					(reference "BMI1_SCL1")
 					(unit 1)
 				)
@@
 		(on_board yes)
 		(dnp no)
-		(property "Reference" "BMI2_SDA1"
+		(property "Reference" "BMI1_SDA1"
 			(at 124.46 100.33 90)
 			(effects
@@
 			(project "nautilus_mainboard"
 				(path "/ce1819b2-f280-40ed-834f-6fe4d12f809d/bdf8f7d6-a5ee-4741-925d-5019e8cbdfce/0c7afee2-dd12-41f0-a704-0f15387072b0"
-					(reference "BMI2_SDA1")
+					(reference "BMI1_SDA1")
 					(unit 1)
 				)
@@
 		(dnp no)
 		(fields_autoplaced yes)
-		(property "Reference" "U2"
+		(property "Reference" "U1"
 			(at 148.59 72.39 0)
 			(effects
@@
 			(project "nautilus_mainboard"
 				(path "/ce1819b2-f280-40ed-834f-6fe4d12f809d/bdf8f7d6-a5ee-4741-925d-5019e8cbdfce/0c7afee2-dd12-41f0-a704-0f15387072b0"
-					(reference "U2")
+					(reference "U1")
 					(unit 1)
 				)

Commit message: chore: Many routing changes
Parts:
- removed BMI1, BMI1_SCL1, BMI1_SDA1: 0, Resistor_SMD:R_0603_1608Metric, symbol #dzdb:g_res/R-0-0603
- added R50, R51, R53: 0, Resistor_SMD:R_0603_1608Metric, symbol #dzdb:g_res/R-0-0603
Connections:
- net IMU_SCL: now also R50.1
- net IMU_SDA: now also R51.1
- net at U1.14 (CSB1), U1.7 (PS): now also R53.2
- net at U1.8 (SCL/SCK): now also R50.2
- net at U1.9 (SDA/SDI): now also R51.2
- net BMI_IN_3.3V renamed BMI_In_3.3V
- net BMI_In_3.3V: now also R53.1

Commit message: chore: more cleanup
Other:
- company: (none) -> Davide
Changed lines of the file:
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@@
 	(generator_version "9.0")
 	(paper "A4")
+	(title_block
+		(date "2025-11-18")
+		(company "Davide")
+	)
 	(text "Accelerometer\n SD01 pin pulled to GND (0x18)\nSD01 pin pulled to VDDIO: (0x19)\n\nGyroscope:\nSD02 pin pulled to GND: (0x68)\nSDO2 pin pulled to VDDIO: 0x69)"
 		(exclude_from_sim no)

Commit message: chore: Loads of redoing stuff. Added a Changelog
Other:
- title: (none) -> Nautilus_Mainboard
Changed lines of the file:
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@@
 	(paper "A4")
 	(title_block
+		(title "Nautilus_Mainboard")
 		(date "2025-11-19")
 		(rev "0")

Commit message: chore: routed the Jumpers (incomplete) fix: removed all leftover 0Ohm resistors
Parts:
- removed R50, R51, R53: 0, Resistor_SMD:R_0603_1608Metric, symbol #dzdb:g_res/R-0-0603
- added JP19, JP20, JP21: -, Jumper:SolderJumper-2_P1.3mm_Open_RoundedPad1.0x1.5mm, symbol #dzdb:g_mech/Jumper-2P1.3mm_Rounded
Connections:
- net BMI_In_3.3V: now also JP21.1 (A)
- net IMU_SCL: now also JP19.1 (A)
- net IMU_SDA: now also JP20.1 (A)
- net at U1.9 (SDA/SDI): now also JP20.2 (B)
- net at U1.8 (SCL/SCK): now also JP19.2 (B)
- net at U1.14 (CSB1), U1.7 (PS): now also JP21.2 (B)
