File: Presentation/boards/nautilus_mainboard.kicad_pcb (KiCad board)
At the start: 4 copper layers, 125 x 75 mm, 131 parts, among them IC1 STM32H7B0RBT6, IC2 TCAN3414DRBR, IC3 TPS2121RUXT, IC4 TPS2121RUXT, IC5 TPS2121RUXT, J1 FTSH-107-02-L-DV, J18 179-UJ20CHC4SMTTR, J2 61300211121, J4 Header male 1x05, J5 1792876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

Commit message: Deploying to gh-pages from @ Nautilus-UUV/nautilus-mainboard-PCB@e643558b08d37d3a450dbfa2fadeff82d32b99a7 🚀
Parts:
- removed LS1: ~, dz_mech:PT-1140PEQ
- removed Q3: 50V, dz_dio:onsemi_Mosfet_BSS138
- removed R38: 1k, Resistor_SMD:R_0603_1608Metric
- removed R39: 0, Resistor_SMD:R_0603_1608Metric
- removed R40: 100, Resistor_SMD:R_0402_1005Metric
Routing:
- net /STM/PinoutSTM/CAN1_RX: track 22.5 -> 19.1 mm
- net /STM/PinoutSTM/CAN1_TX: track 23.4 -> 25.2 mm
- net /STM/PinoutSTM/USART1_RX: track 44.8 -> 45.9 mm
- net GND: vias 572 -> 595

Commit message: Deploying to gh-pages from @ Nautilus-UUV/nautilus-mainboard-PCB@400426d46daeee198d0eea8645f966723a05ffff 🚀
Parts:
- added TP2: TestPoint_Probe, TestPoint:TestPoint_THTPad_D2.5mm_Drill1.2mm, F.Cu at (170.7, 178.1)
- added TP3: TestPoint_Probe, TestPoint:TestPoint_THTPad_D2.5mm_Drill1.2mm, F.Cu at (170.7, 173.7)
- added TP4: TestPoint_Probe, TestPoint:TestPoint_Pad_D1.0mm, F.Cu at (125.5, 197.5)
- added TP5: TestPoint_Probe, TestPoint:TestPoint_Pad_D1.0mm, F.Cu at (127.5, 199.4)
- added TP6: TestPoint_Probe, TestPoint:TestPoint_THTPad_D2.5mm_Drill1.2mm, F.Cu at (95.9, 216.9)
- added TP7: TestPoint_Probe, TestPoint:TestPoint_THTPad_D2.5mm_Drill1.2mm, F.Cu at (101.1, 217.0)
- moved R4 1.20 mm to (104.0, 219.2), turned to 0 degrees
Routing:
- net /IMU/Pack1_SCL: track 103.4 -> 110.0 mm, vias 7 -> 8
- net GND: track 300.4 -> 295.8 mm, vias 595 -> 587
- net /IMU/Pack1_SDA: track 111.9 -> 116.1 mm
- net /STM/PinoutSTM/CAN1_RX: track 19.1 -> 22.3 mm
- net /STM/PinoutSTM/CAN1_TX: track 25.2 -> 24.0 mm, vias 2 -> 3
- net /CM4/CM4_Module1A/GPIO14: track 23.4 -> 24.6 mm
- net /STM/PinoutSTM/STM_BOOT0: track 27.5 -> 28.2 mm
Other:
- board text added: "11"
- board text added: "13"
- board text added: "3"
- board text added: "5"
- board text added: "7"
- board text added: "9"

Commit message: Deploying to gh-pages from @ Nautilus-UUV/nautilus-mainboard-PCB@ff07aeebf3c2c401dced3247772428d318509d16 🚀
Parts:
- moved TP5 1.33 mm to (126.2, 199.5)
Routing:
- net GND: vias 587 -> 594
Changed lines of the file:
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@@
 			(at 0 -2.148 0)
 			(layer "F.SilkS")
+			(hide yes)
 			(effects
 				(font
@@
 			(at 0 -2.148 0)
 			(layer "F.SilkS")
+			(hide yes)
 			(effects
 				(font
@@
 	(footprint "TestPoint:TestPoint_Pad_D1.0mm"
 		(layer "F.Cu")
-		(at 127.525 199.45)
+		(at 126.2 199.5)
 		(descr "SMD pad as test Point, diameter 1.0mm")
 		(tags "test point SMD pad")
@@
 	)
 	(via
+		(at 141.675 210.875)
+		(size 0.6)
+		(drill 0.3)
+		(layers "F.Cu" "B.Cu")
+		(free yes)
+		(net 2)
+	)
+	(via
 		(at 158.725 197.95)
 		(size 0.6)
@@
 	)
 	(via
+		(at 140.5 204.175)
+		(size 0.6)
+		(drill 0.3)
+		(layers "F.Cu" "B.Cu")
+		(free yes)
+		(net 2)
+	)
+	(via
 		(at 141.175 187.975)
 		(size 0.6)
@@
 	)
 	(via
+		(at 149.05 214.725)
+		(size 0.6)
+		(drill 0.3)
+		(layers "F.Cu" "B.Cu")
+		(free yes)
+		(net 2)
+	)
+	(via
 		(at 186.48 162.42)
 		(size 0.6)
@@
 	)
 	(via
+		(at 143.65 210.875)
+		(size 0.6)
+		(drill 0.3)
+		(layers "F.Cu" "B.Cu")
+		(free yes)
+		(net 2)
+	)
+	(via
 		(at 146.325 215.775)
 		(size 0.6)
@@
 	)
 	(via
+		(at 146.35 223.25)
+		(size 0.6)
+		(drill 0.3)
+		(layers "F.Cu" "B.Cu")
+		(free yes)
+		(net 2)
+	)
+	(via
 		(at 138.725 156.375)
 		(size 0.6)
@@
 	)
 	(via
+		(at 136.75 204.5)
+		(size 0.6)
+		(drill 0.3)
+		(layers "F.Cu" "B.Cu")
+		(free yes)
+		(net 2)
+	)
+	(via
 		(at 173.95 167.275)
 		(size 0.6)
@@
 	)
 	(via
+		(at 131.25 204.45)
+		(size 0.6)
+		(drill 0.3)
+		(layers "F.Cu" "B.Cu")
+		(free yes)
+		(net 2)
+	)
+	(via
 		(at 143.45 195.25)
 		(size 0.6)
@@
 	)
 	(segment
-		(start 128.35 196.288815)
-		(end 128.35 198.4)
-		(width 0.2)
-		(layer "F.Cu")
-		(net 92)
-	)
-	(segment
 		(start 122.999 200.889)
 		(end 123.01 200.9)
@@
 	)
 	(segment
-		(start 129.43 195.208815)
-		(end 128.35 196.288815)
+		(start 126.95 198.55)
+		(end 125.96 199.54)
 		(width 0.2)
 		(layer "F.Cu")
@@
 	)
 	(segment
+		(start 125.96 199.54)
+		(end 124.38 199.54)
+		(width 0.2)
+		(layer "F.Cu")
+		(net 92)
+	)
+	(segment
 		(start 113.27 203.638149)
 		(end 114.538149 202.37)
@@
 	)
 	(segment
-		(start 129.43 194.340001)
-		(end 129.43 195.208815)
+		(start 127.419 196.381)
+		(end 126.95 196.85)
 		(width 0.2)
 		(layer "F.Cu")
@@
 	)
 	(segment
+		(start 128.257814 196.381)
+		(end 127.419 196.381)
+		(width 0.2)
+		(layer "F.Cu")
+		(net 92)
+	)
+	(segment
 		(start 119.95 203.03)
 		(end 122.091 200.889)
@@
 	)
 	(segment
+		(start 129.43 194.340001)
+		(end 129.43 195.208815)
+		(width 0.2)
+		(layer "F.Cu")
+		(net 92)
+	)
+	(segment
 		(start 113.823819 205.740519)
 		(end 113.27 205.1867)
@@
 	)
 	(segment
-		(start 128.35 198.4)
-		(end 127.21 199.54)
+		(start 129.43 195.208815)
+		(end 128.257814 196.381)
 		(width 0.2)
 		(layer "F.Cu")
@@
 	)
 	(segment
-		(start 127.21 199.54)
-		(end 124.38 199.54)
+		(start 126.95 196.85)
+		(end 126.95 198.55)
 		(width 0.2)
 		(layer "F.Cu")
