File: Browse/IMU2.kicad_sch (KiCad schematic)
At the start: 6 parts, among them U2 262-BMI088

Commit message: Deploying to gh-pages from @ Nautilus-UUV/nautilus-mainboard-PCB@f1dd6ce1e57c066b805694b10777c719502cca87 🚀
Parts:
- removed BMI2, BMI2_SCL1, BMI2_SDA1: 0, Resistor_SMD:R_0603_1608Metric, symbol #dzdb:g_res/R-0-0603
- added R48, R49, R52: 0, Resistor_SMD:R_0603_1608Metric, symbol #dzdb:g_res/R-0-0603
Connections:
- net IMU_SCL: now also R48.1
- net IMU_SDA: now also R49.1
- net at U2.8 (SCL/SCK): now also R48.2
- net at U2.14 (CSB1), U2.7 (PS): now also R52.2
- net at U2.9 (SDA/SDI): now also R49.2
- net BMI_IN_3.3V renamed BMI_In_3.3V
- net BMI_In_3.3V: now also R52.1
Other:
- company: (none) -> Davide
- title: (none) -> Nautilus_Mainboard

Commit message: Deploying to gh-pages from @ Nautilus-UUV/nautilus-mainboard-PCB@b731ca7531dd1e48b6b7a45790de08634e79c176 🚀
Parts:
- removed R48, R49, R52: 0, Resistor_SMD:R_0603_1608Metric, symbol #dzdb:g_res/R-0-0603
- added JP22, JP23, JP24: -, Jumper:SolderJumper-2_P1.3mm_Open_RoundedPad1.0x1.5mm, symbol #dzdb:g_mech/Jumper-2P1.3mm_Rounded
Connections:
- net BMI_In_3.3V: now also JP24.1 (A)
- net IMU_SCL: now also JP22.1 (A)
- net IMU_SDA: now also JP23.1 (A)
- net at U2.14 (CSB1), U2.7 (PS): now also JP24.2 (B)
- net at U2.8 (SCL/SCK): now also JP22.2 (B)
- net at U2.9 (SDA/SDI): now also JP23.2 (B)
