File: Browse/CM4.kicad_sch (KiCad schematic)
At the start: 2 parts

Commit message: Deploying to gh-pages from @ Nautilus-UUV/nautilus-mainboard-PCB@8b02e89ade7c168188296ba6f0516f3abec9166b 🚀
Other:
- sheet CM4_Module1B ports: added PCIE_nRST; removed PCIe_nRST
- note added: "5*4.3k / (2.2k+4.3k) = 5*0.6615 = 3.3075"
- note added: "V_{out}= V_{in} * (R_{2}/(R_{1}+R_{2})"
Changed lines of the file:
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@@
   (paper "A4")
   (title_block
-    (date "2025-11-18")
+    (date "2025-11-19")
+    (rev "0")
     (company "Davide")
   )
@@
     (effects (font (size 1.27 1.27)))
   )
+  (text "5*4.3k / (2.2k+4.3k) = 5*0.6615 = 3.3075" (exclude_from_sim no) (at 203.962 139.954 0)
+    (effects (font (size 1.27 1.27)))
+  )
   (text "3.3V out" (exclude_from_sim no) (at 204.47 114.046 90)
+    (effects (font (size 1.27 1.27)))
+  )
+  (text "V_{out}= V_{in} * (R_{2}/(R_{1}+R_{2})" (exclude_from_sim no) (at 194.31 130.81 0)
     (effects (font (size 1.27 1.27)))
   )
@@
       (effects (font (size 1.27 1.27)) (justify left))
     )
-    (pin "PCIe_nRST" input (at 193.04 97.79 270)
-      (effects (font (size 1.27 1.27)) (justify left))
-    )
     (pin "USB_OTG_5V" output (at 196.85 97.79 270)
       (effects (font (size 1.27 1.27)) (justify left))
@@
       (effects (font (size 1.27 1.27)) (justify left))
     )
+    (pin "PCIE_nRST" input (at 193.04 97.79 270)
+      (effects (font (size 1.27 1.27)) (justify left))
+    )

Commit message: Deploying to gh-pages from @ Nautilus-UUV/nautilus-mainboard-PCB@5b07cf6af03655ef9ddad269b1edd5eb03bfa75f 🚀
Other:
- title: (none) -> Nautilus_Mainboard
Changed lines of the file:
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@@
   (paper "A4")
   (title_block
+    (title "Nautilus_Mainboard")
     (date "2025-11-19")
     (rev "0")

Commit message: Deploying to gh-pages from @ Nautilus-UUV/nautilus-mainboard-PCB@5f5fdd9436d408a604bb268d740c0ac7ce1f5af5 🚀
Other:
- sheet CM4_Module1A ports: added none; removed Battery_Out_3.3V, CM4_Out_3.3V, LAN_IN_3.3V
- sheet CM4_Module1B ports: added PCIe_CLK_N, PCIe_CLK_P, PCIe_RX_N, PCIe_RX_P, PCIe_TX_N, PCIe_TX_P, PCIe_nRST; removed PCIE_CLK{_N,_P}, PCIE_RX{_N,_P}, PCIE_TX{_N,_P}, PCIE_nRST, USB_Out_5V
- sheet PCIE_Interface ports: added PCIE_CLK_N, PCIE_CLK_P, PCIE_RX_N, PCIE_RX_P, PCIE_TX_N, PCIE_TX_P; removed Battery_Out_3.3V, PCIE_CLK{_N,_P}, PCIE_RX{_N,_P}, PCIE_TX{_N,_P}
- note added: "do we need BSC master 0 data line and clock line? (for iic)"
- note removed: "5*4.3k / (2.2k+4.3k) = 5*0.6615 = 3.3075"
- note removed: "V_{out}= V_{in} * (R_{2}/(R_{1}+R_{2})"
- company: Davide -> (none)
- title: Nautilus_Mainboard -> (none)

Commit message: Deploying to gh-pages from @ Nautilus-UUV/nautilus-mainboard-PCB@44ad8adb17f33e1aa4439bd10449a9ac7e221a1f 🚀
Changed lines of the file:
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@@
     (stroke (width 0) (type default))
   )
-  (wire (pts (xy 81.28 81.28) (xy 86.36 81.28))
+  (wire (pts (xy 78.74 81.28) (xy 86.36 81.28))
     (stroke (width 0) (type solid))
   )
@@
     (effects (font (size 1.27 1.27)))
   )
-  (global_label "GPIO_VREF_3.3V" (shape input) (at 81.28 81.28 180) (fields_autoplaced)
-    (effects (font (size 1.27 1.27)) (justify right))
-    (property "Intersheetrefs" "${INTERSHEET_REFS}" (at 63.1757 81.28 0)
-      (effects (font (size 1.27 1.27)) (justify right) (hide yes))
-    )
-  )
   (hierarchical_label "PI_RX" (shape input) (at 128.27 104.14 270)
     (effects (font (size 1.27 1.27)) (justify right))
@@
     (effects (font (size 1.27 1.27)) (justify right))
   )
-  (hierarchical_label "PI_TX" (shape input) (at 124.46 104.14 270)
+  (hierarchical_label "PI_TX" (shape output) (at 124.46 104.14 270)
+    (effects (font (size 1.27 1.27)) (justify right))
+  )
+  (hierarchical_label "GPIO_VREF_3.3V" (shape input) (at 78.74 81.28 180)
     (effects (font (size 1.27 1.27)) (justify right))
   )
@@
     (effects (font (size 1.27 1.27)) (justify right))
   )
-  (hierarchical_label "RUN_PG" (shape input) (at 142.24 57.15 0)
+  (hierarchical_label "RUN_PG" (shape output) (at 142.24 57.15 0)
     (effects (font (size 1.27 1.27)) (justify left))
   )
@@
       (effects (font (size 1.27 1.27)) (justify left))
     )
-    (pin "TXD0" input (at 124.46 97.79 270)
+    (pin "TXD0" output (at 124.46 97.79 270)
       (effects (font (size 1.27 1.27)) (justify left))
     )
-    (pin "RUN_PG" input (at 137.16 57.15 0)
+    (pin "RUN_PG" output (at 137.16 57.15 0)
       (effects (font (size 1.27 1.27)) (justify right))
     )

Commit message: Deploying to gh-pages from @ Nautilus-UUV/nautilus-mainboard-PCB@a81f7ffbfc5f9b51f47d7f388c30fcea2673b9ea 🚀
Other:
- sheet CM4_Module1A ports: added Battery_Out_3.3V, CM4_Out_3.3V, LAN_IN_3.3V; removed none
- sheet CM4_Module1B ports: added PCIE_CLK{_N,_P}, PCIE_RX{_N,_P}, PCIE_TX{_N,_P}, USB_Out_5V; removed PCIe_CLK_N, PCIe_CLK_P, PCIe_RX_N, PCIe_RX_P, PCIe_TX_N, PCIe_TX_P
- sheet PCIE_Interface ports: added Battery_Out_3.3V, PCIE_CLK{_N,_P}, PCIE_RX{_N,_P}, PCIE_TX{_N,_P}; removed PCIE_CLK_N, PCIE_CLK_P, PCIE_RX_N, PCIE_RX_P, PCIE_TX_N, PCIE_TX_P
- note removed: "do we need BSC master 0 data line and clock line? (for iic)"
Changed lines of the file:
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@@
 (kicad_sch (version 20250114) (generator "eeschema") (generator_version "9.0")
   (paper "A4")
+  (junction (at 62.23 85.09) (diameter 0) (color 0 0 0 0)
+  )
   (junction (at 203.2 125.73) (diameter 0) (color 0 0 0 0)
   )
-  (wire (pts (xy 158.75 118.11) (xy 135.89 118.11))
-    (stroke (width 0) (type default))
-  )
-  (wire (pts (xy 154.94 72.39) (xy 162.56 72.39))
-    (stroke (width 0) (type default))
-  )
-  (wire (pts (xy 133.35 116.84) (xy 157.48 116.84))
-    (stroke (width 0) (type default))
-  )
-  (wire (pts (xy 153.67 69.85) (xy 153.67 113.03))
-    (stroke (width 0) (type default))
-  )
-  (wire (pts (xy 133.35 127) (xy 133.35 116.84))
+  (wire (pts (xy 62.23 129.54) (xy 86.36 129.54))
+    (stroke (width 0) (type default))
+  )
+  (wire (pts (xy 78.74 77.47) (xy 86.36 77.47))
     (stroke (width 0) (type default))
   )
@@
     (stroke (width 0) (type default))
   )
-  (wire (pts (xy 157.48 116.84) (xy 157.48 77.47))
-    (stroke (width 0) (type default))
-  )
   (bus (pts (xy 78.74 62.23) (xy 86.36 62.23))
     (stroke (width 0) (type default))
   )
-  (wire (pts (xy 156.21 74.93) (xy 156.21 115.57))
-    (stroke (width 0) (type default))
-  )
-  (wire (pts (xy 125.73 113.03) (xy 125.73 127))
+  (wire (pts (xy 213.36 80.01) (xy 218.44 80.01))
     (stroke (width 0) (type default))
   )
@@
     (stroke (width 0) (type solid))
   )
+  (bus (pts (xy 118.11 114.3) (xy 147.32 114.3))
+    (stroke (width 0) (type default))
+  )
+  (wire (pts (xy 78.74 73.66) (xy 86.36 73.66))
+    (stroke (width 0) (type default))
+  )
   (bus (pts (xy 78.74 52.07) (xy 86.36 52.07))
     (stroke (width 0) (type default))
   )
-  (wire (pts (xy 154.94 114.3) (xy 154.94 72.39))
-    (stroke (width 0) (type default))
-  )
   (wire (pts (xy 124.46 97.79) (xy 124.46 104.14))
     (stroke (width 0) (type default))
@@
     (stroke (width 0) (type default))
   )
-  (wire (pts (xy 128.27 127) (xy 128.27 114.3))
-    (stroke (width 0) (type default))
-  )
-  (wire (pts (xy 157.48 77.47) (xy 162.56 77.47))
-    (stroke (width 0) (type default))
-  )
-  (wire (pts (xy 162.56 80.01) (xy 158.75 80.01))
+  (bus (pts (xy 120.65 127) (xy 120.65 116.84))
+    (stroke (width 0) (type default))
+  )
+  (bus (pts (xy 149.86 72.39) (xy 162.56 72.39))
     (stroke (width 0) (type default))
   )
@@
     (stroke (width 0) (type default))
   )
-  (wire (pts (xy 138.43 127) (xy 138.43 119.38))
-    (stroke (width 0) (type default))
-  )
   (wire (pts (xy 203.2 97.79) (xy 203.2 125.73))
     (stroke (width 0) (type default))
   )
+  (bus (pts (xy 123.19 119.38) (xy 152.4 119.38))
+    (stroke (width 0) (type default))
+  )
+  (bus (pts (xy 147.32 114.3) (xy 147.32 69.85))
+    (stroke (width 0) (type default))
+  )
   (wire (pts (xy 193.04 101.6) (xy 193.04 97.79))
     (stroke (width 0) (type default))
   )
+  (bus (pts (xy 118.11 127) (xy 118.11 114.3))
+    (stroke (width 0) (type default))
+  )
+  (wire (pts (xy 59.69 85.09) (xy 62.23 85.09))
+    (stroke (width 0) (type default))
+  )
+  (bus (pts (xy 123.19 127) (xy 123.19 119.38))
+    (stroke (width 0) (type default))
+  )
   (wire (pts (xy 162.56 142.24) (xy 162.56 101.6))
     (stroke (width 0) (type default))
   )
-  (wire (pts (xy 160.02 82.55) (xy 162.56 82.55))
-    (stroke (width 0) (type default))
-  )
   (wire (pts (xy 162.56 101.6) (xy 193.04 101.6))
     (stroke (width 0) (type default))
   )
-  (wire (pts (xy 130.81 115.57) (xy 130.81 127))
-    (stroke (width 0) (type default))
-  )
   (bus (pts (xy 78.74 67.31) (xy 86.36 67.31))
     (stroke (width 0) (type default))
   )
-  (wire (pts (xy 138.43 119.38) (xy 160.02 119.38))
-    (stroke (width 0) (type default))
-  )
-  (wire (pts (xy 160.02 119.38) (xy 160.02 82.55))
+  (wire (pts (xy 62.23 85.09) (xy 86.36 85.09))
     (stroke (width 0) (type default))
   )
@@
     (stroke (width 0) (type default))
   )
-  (wire (pts (xy 162.56 69.85) (xy 153.67 69.85))
-    (stroke (width 0) (type default))
-  )
-  (wire (pts (xy 162.56 74.93) (xy 156.21 74.93))
-    (stroke (width 0) (type default))
-  )
-  (wire (pts (xy 156.21 115.57) (xy 130.81 115.57))
-    (stroke (width 0) (type default))
-  )
-  (wire (pts (xy 135.89 118.11) (xy 135.89 127))
-    (stroke (width 0) (type default))
-  )
-  (wire (pts (xy 153.67 113.03) (xy 125.73 113.03))
+  (bus (pts (xy 152.4 74.93) (xy 162.56 74.93))
+    (stroke (width 0) (type default))
+  )
+  (wire (pts (xy 62.23 85.09) (xy 62.23 129.54))
+    (stroke (width 0) (type default))
+  )
+  (bus (pts (xy 149.86 116.84) (xy 149.86 72.39))
+    (stroke (width 0) (type default))
+  )
+  (bus (pts (xy 147.32 69.85) (xy 162.56 69.85))
     (stroke (width 0) (type default))
   )
@@
     (stroke (width 0) (type default))
   )
-  (wire (pts (xy 128.27 114.3) (xy 154.94 114.3))
-    (stroke (width 0) (type default))
-  )
   (wire (pts (xy 203.2 125.73) (xy 209.55 125.73))
     (stroke (width 0) (type default))
   )
+  (bus (pts (xy 152.4 119.38) (xy 152.4 74.93))
+    (stroke (width 0) (type default))
+  )
   (wire (pts (xy 139.7 142.24) (xy 162.56 142.24))
     (stroke (width 0) (type default))
   )
-  (wire (pts (xy 158.75 80.01) (xy 158.75 118.11))
+  (bus (pts (xy 120.65 116.84) (xy 149.86 116.84))
     (stroke (width 0) (type default))
   )
@@
     (stroke (width 0) (type default))
     (fill (type none))
-  )
-  (text "do we need BSC master 0 data line and clock line? (for iic)" (exclude_from_sim no) (at 53.594 89.662 0)
-    (effects (font (size 1.27 1.27)))
   )
   (text "5V in\n" (exclude_from_sim no) (at 197.866 112.776 90)
@@
     (effects (font (size 1.27 1.27)) (justify right))
   )
+  (hierarchical_label "USB_Out_5V" (shape output) (at 218.44 80.01 0)
+    (effects (font (size 1.27 1.27)) (justify left))
+  )
+  (hierarchical_label "LAN_IN_3.3V" (shape input) (at 78.74 77.47 180)
+    (effects (font (size 1.27 1.27)) (justify right))
+  )
+  (hierarchical_label "CM4_Out_3.3V" (shape output) (at 78.74 73.66 180)
+    (effects (font (size 1.27 1.27)) (justify right))
+  )
   (hierarchical_label "GPIO_VREF_3.3V" (shape input) (at 78.74 81.28 180)
     (effects (font (size 1.27 1.27)) (justify right))
@@
   (hierarchical_label "RUN_PG" (shape output) (at 142.24 57.15 0)
     (effects (font (size 1.27 1.27)) (justify left))
+  )
+  (hierarchical_label "Battery_Out_3.3V" (shape input) (at 59.69 85.09 180)
+    (effects (font (size 1.27 1.27)) (justify right))
   )
   (symbol (lib_id "#dzdb:g_res/R-4.3k-0603") (at 213.36 125.73 90) (unit 1)
@@
       (effects (font (size 1.27 1.27)) (justify left))
     )
+    (pin "LAN_IN_3.3V" input (at 86.36 77.47 180)
+      (effects (font (size 1.27 1.27)) (justify left))
+    )
+    (pin "Battery_Out_3.3V" input (at 86.36 85.09 180)
+      (effects (font (size 1.27 1.27)) (justify left))
+    )
+    (pin "CM4_Out_3.3V" output (at 86.36 73.66 180)
+      (effects (font (size 1.27 1.27)) (justify left))
+    )
     (instances
       (project "nautilus_mainboard"
@@
       (effects (font (size 1.27 1.27)) (justify left))
     )
-    (pin "PCIe_CLK_N" bidirectional (at 162.56 69.85 180)
-      (effects (font (size 1.27 1.27)) (justify left))
-    )
-    (pin "PCIe_CLK_P" bidirectional (at 162.56 72.39 180)
-      (effects (font (size 1.27 1.27)) (justify left))
-    )
-    (pin "PCIe_RX_N" bidirectional (at 162.56 74.93 180)
-      (effects (font (size 1.27 1.27)) (justify left))
-    )
-    (pin "PCIe_RX_P" bidirectional (at 162.56 77.47 180)
-      (effects (font (size 1.27 1.27)) (justify left))
-    )
-    (pin "PCIe_TX_N" bidirectional (at 162.56 80.01 180)
-      (effects (font (size 1.27 1.27)) (justify left))
-    )
-    (pin "PCIe_TX_P" bidirectional (at 162.56 82.55 180)
-      (effects (font (size 1.27 1.27)) (justify left))
-    )
     (pin "PCIe_nRST" input (at 193.04 97.79 270)
       (effects (font (size 1.27 1.27)) (justify left))
     )
-    (pin "USB_OTG_5V" input (at 196.85 97.79 270)
+    (pin "USB_OTG_5V" output (at 196.85 97.79 270)
+      (effects (font (size 1.27 1.27)) (justify left))
+    )
+    (pin "USB_Out_5V" output (at 213.36 80.01 0)
+      (effects (font (size 1.27 1.27)) (justify right))
+    )
+    (pin "PCIE_CLK{_N,_P}" bidirectional (at 162.56 69.85 180)
+      (effects (font (size 1.27 1.27)) (justify left))
+    )
+    (pin "PCIE_RX{_N,_P}" bidirectional (at 162.56 72.39 180)
+      (effects (font (size 1.27 1.27)) (justify left))
+    )
+    (pin "PCIE_TX{_N,_P}" bidirectional (at 162.56 74.93 180)
       (effects (font (size 1.27 1.27)) (justify left))
     )
@@
       (effects (font (size 1.27 1.27)) (justify left top))
     )
-    (pin "PCIE_CLK_N" bidirectional (at 125.73 127 90)
-      (effects (font (size 1.27 1.27)) (justify right))
-    )
-    (pin "PCIE_CLK_P" bidirectional (at 128.27 127 90)
-      (effects (font (size 1.27 1.27)) (justify right))
-    )
-    (pin "PCIE_RX_N" bidirectional (at 130.81 127 90)
-      (effects (font (size 1.27 1.27)) (justify right))
-    )
-    (pin "PCIE_RX_P" bidirectional (at 133.35 127 90)
-      (effects (font (size 1.27 1.27)) (justify right))
-    )
-    (pin "PCIE_TX_N" bidirectional (at 135.89 127 90)
-      (effects (font (size 1.27 1.27)) (justify right))
-    )
-    (pin "PCIE_TX_P" bidirectional (at 138.43 127 90)
-      (effects (font (size 1.27 1.27)) (justify right))
-    )
     (pin "PCIE_nRST" input (at 139.7 142.24 0)
       (effects (font (size 1.27 1.27)) (justify right))
     )
+    (pin "Battery_Out_3.3V" input (at 86.36 129.54 180)
+      (effects (font (size 1.27 1.27)) (justify left))
+    )
+    (pin "PCIE_CLK{_N,_P}" bidirectional (at 118.11 127 90)
+      (effects (font (size 1.27 1.27)) (justify right))
+    )
+    (pin "PCIE_RX{_N,_P}" bidirectional (at 120.65 127 90)
+      (effects (font (size 1.27 1.27)) (justify right))
+    )
+    (pin "PCIE_TX{_N,_P}" bidirectional (at 123.19 127 90)
+      (effects (font (size 1.27 1.27)) (justify right))
+    )

Commit message: Deploying to gh-pages from @ Nautilus-UUV/nautilus-mainboard-PCB@2d3890115fd9d3c0bb909c9898aa64801bed9e67 🚀
Other:
- company: (none) -> Davide
Changed lines of the file:
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@@
 (kicad_sch (version 20250114) (generator "eeschema") (generator_version "9.0")
   (paper "A4")
+  (title_block
+    (date "2025-11-18")
+    (company "Davide")
+  )
   (junction (at 62.23 85.09) (diameter 0) (color 0 0 0 0)
   )
