File: Browse/CM4.kicad_sch (KiCad schematic)
At the start: 2 parts

Commit message: Deploying to gh-pages from @ Nautilus-UUV/nautilus-mainboard-PCB@b62834b88bb3e2a9413bcb4ea8e223af403e20ba 🚀
Other:
- sheet CM4_Module1A ports: added TRD0{D+ D-}, TRD1{D+ D-}, TRD2{D+ D-}, TRD3{D+ D-}; removed ET1, ET2, ET3, ET4, ET5, ET6, ET7, ET8
Changed lines of the file:
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@@
-    (stroke (width 0) (type default))
-  )
-  (wire (pts (xy 83.82 59.69) (xy 86.36 59.69))
     (stroke (width 0) (type default))
   )
@@
   )
   (wire (pts (xy 157.48 116.84) (xy 157.48 77.47))
+    (stroke (width 0) (type default))
+  )
+  (bus (pts (xy 78.74 62.23) (xy 86.36 62.23))
     (stroke (width 0) (type default))
   )
@@
     (stroke (width 0) (type solid))
   )
-  (wire (pts (xy 83.82 62.23) (xy 86.36 62.23))
+  (bus (pts (xy 78.74 52.07) (xy 86.36 52.07))
     (stroke (width 0) (type default))
   )
@@
     (stroke (width 0) (type default))
   )
+  (bus (pts (xy 78.74 57.15) (xy 86.36 57.15))
+    (stroke (width 0) (type default))
+  )
   (wire (pts (xy 138.43 127) (xy 138.43 119.38))
     (stroke (width 0) (type default))
   )
-  (wire (pts (xy 83.82 54.61) (xy 86.36 54.61))
-    (stroke (width 0) (type default))
-  )
   (wire (pts (xy 203.2 97.79) (xy 203.2 125.73))
     (stroke (width 0) (type default))
   )
-  (wire (pts (xy 83.82 64.77) (xy 86.36 64.77))
-    (stroke (width 0) (type default))
-  )
   (wire (pts (xy 193.04 101.6) (xy 193.04 97.79))
     (stroke (width 0) (type default))
   )
-  (wire (pts (xy 83.82 57.15) (xy 86.36 57.15))
-    (stroke (width 0) (type default))
-  )
   (wire (pts (xy 162.56 142.24) (xy 162.56 101.6))
     (stroke (width 0) (type default))
@@
     (stroke (width 0) (type default))
   )
+  (bus (pts (xy 78.74 67.31) (xy 86.36 67.31))
+    (stroke (width 0) (type default))
+  )
   (wire (pts (xy 138.43 119.38) (xy 160.02 119.38))
     (stroke (width 0) (type default))
@@
     (stroke (width 0) (type default))
   )
-  (wire (pts (xy 83.82 67.31) (xy 86.36 67.31))
-    (stroke (width 0) (type default))
-  )
   (wire (pts (xy 82.55 93.98) (xy 86.36 93.98))
     (stroke (width 0) (type default))
@@
   )
   (wire (pts (xy 158.75 80.01) (xy 158.75 118.11))
-    (stroke (width 0) (type default))
-  )
-  (wire (pts (xy 83.82 72.39) (xy 86.36 72.39))
-    (stroke (width 0) (type default))
-  )
-  (wire (pts (xy 83.82 69.85) (xy 86.36 69.85))
     (stroke (width 0) (type default))
   )
@@
     )
   )
-  (hierarchical_label "ET5" (shape input) (at 83.82 64.77 180)
-    (effects (font (size 1.27 1.27)) (justify right))
-  )
-  (hierarchical_label "ET2" (shape input) (at 83.82 57.15 180)
-    (effects (font (size 1.27 1.27)) (justify right))
-  )
   (hierarchical_label "PI_RX" (shape input) (at 128.27 104.14 270)
     (effects (font (size 1.27 1.27)) (justify right))
   )
-  (hierarchical_label "ET1" (shape input) (at 83.82 54.61 180)
-    (effects (font (size 1.27 1.27)) (justify right))
-  )
-  (hierarchical_label "ET6" (shape input) (at 83.82 67.31 180)
-    (effects (font (size 1.27 1.27)) (justify right))
-  )
-  (hierarchical_label "ET4" (shape input) (at 83.82 62.23 180)
-    (effects (font (size 1.27 1.27)) (justify right))
-  )
-  (hierarchical_label "ET8" (shape input) (at 83.82 72.39 180)
+  (hierarchical_label "TRD0{D+ D-}" (shape bidirectional) (at 78.74 52.07 180)
+    (effects (font (size 1.27 1.27)) (justify right))
+  )
+  (hierarchical_label "TRD1{D+ D-}" (shape bidirectional) (at 78.74 57.15 180)
     (effects (font (size 1.27 1.27)) (justify right))
   )
@@
     (effects (font (size 1.27 1.27)) (justify right))
   )
+  (hierarchical_label "TRD3{D+ D-}" (shape bidirectional) (at 78.74 67.31 180)
+    (effects (font (size 1.27 1.27)) (justify right))
+  )
   (hierarchical_label "PI_TX" (shape input) (at 124.46 104.14 270)
     (effects (font (size 1.27 1.27)) (justify right))
   )
-  (hierarchical_label "ET7" (shape input) (at 83.82 69.85 180)
-    (effects (font (size 1.27 1.27)) (justify right))
-  )
-  (hierarchical_label "ET3" (shape input) (at 83.82 59.69 180)
+  (hierarchical_label "TRD2{D+ D-}" (shape bidirectional) (at 78.74 62.23 180)
     (effects (font (size 1.27 1.27)) (justify right))
   )
@@
       (effects (font (size 1.27 1.27)) (justify left top))
     )
-    (pin "ET1" input (at 86.36 54.61 180)
-      (effects (font (size 1.27 1.27)) (justify left))
-    )
-    (pin "ET2" input (at 86.36 57.15 180)
-      (effects (font (size 1.27 1.27)) (justify left))
-    )
-    (pin "ET3" input (at 86.36 59.69 180)
-      (effects (font (size 1.27 1.27)) (justify left))
-    )
-    (pin "ET4" input (at 86.36 62.23 180)
-      (effects (font (size 1.27 1.27)) (justify left))
-    )
-    (pin "ET5" input (at 86.36 64.77 180)
-      (effects (font (size 1.27 1.27)) (justify left))
-    )
-    (pin "ET6" input (at 86.36 67.31 180)
-      (effects (font (size 1.27 1.27)) (justify left))
-    )
-    (pin "ET7" input (at 86.36 69.85 180)
-      (effects (font (size 1.27 1.27)) (justify left))
-    )
-    (pin "ET8" input (at 86.36 72.39 180)
-      (effects (font (size 1.27 1.27)) (justify left))
-    )
     (pin "GPIO_VREF" input (at 86.36 81.28 180)
       (effects (font (size 1.27 1.27)) (justify left))
@@
       (effects (font (size 1.27 1.27)) (justify left))
     )
+    (pin "TRD0{D+ D-}" bidirectional (at 86.36 52.07 180)
+      (effects (font (size 1.27 1.27)) (justify left))
+    )
+    (pin "TRD1{D+ D-}" bidirectional (at 86.36 57.15 180)
+      (effects (font (size 1.27 1.27)) (justify left))
+    )
+    (pin "TRD2{D+ D-}" bidirectional (at 86.36 62.23 180)
+      (effects (font (size 1.27 1.27)) (justify left))
+    )
+    (pin "TRD3{D+ D-}" bidirectional (at 86.36 67.31 180)
+      (effects (font (size 1.27 1.27)) (justify left))
+    )

Commit message: Deploying to gh-pages from @ Nautilus-UUV/nautilus-mainboard-PCB@a20f16cf7e6ebba0b5127d7f7acbd1e63379e186 🚀
Changed lines of the file:
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@@
     (effects (font (size 1.27 1.27)) (justify right))
   )
-  (hierarchical_label "PI_TX" (shape input) (at 124.46 104.14 270)
+  (hierarchical_label "PI_TX" (shape output) (at 124.46 104.14 270)
     (effects (font (size 1.27 1.27)) (justify right))
   )
@@
       (effects (font (size 1.27 1.27)) (justify left))
     )
-    (pin "TXD0" input (at 124.46 97.79 270)
+    (pin "TXD0" output (at 124.46 97.79 270)
       (effects (font (size 1.27 1.27)) (justify left))
     )

Commit message: Deploying to gh-pages from @ Nautilus-UUV/nautilus-mainboard-PCB@f1dd6ce1e57c066b805694b10777c719502cca87 🚀
Other:
- sheet CM4_Module1A ports: added Battery_Out_3.3V, CM4_Out_3.3V, LAN_IN_3.3V; removed none
- sheet CM4_Module1B ports: added PCIE_CLK{_N,_P}, PCIE_RX{_N,_P}, PCIE_TX{_N,_P}, PCIE_nRST, USB_Out_5V; removed PCIe_CLK_N, PCIe_CLK_P, PCIe_RX_N, PCIe_RX_P, PCIe_TX_N, PCIe_TX_P, PCIe_nRST
- sheet PCIE_Interface ports: added Battery_Out_3.3V, PCIE_CLK{_N,_P}, PCIE_RX{_N,_P}, PCIE_TX{_N,_P}; removed PCIE_CLK_N, PCIE_CLK_P, PCIE_RX_N, PCIE_RX_P, PCIE_TX_N, PCIE_TX_P
- note added: "5*4.3k / (2.2k+4.3k) = 5*0.6615 = 3.3075"
- note added: "V_{out}= V_{in} * (R_{2}/(R_{1}+R_{2})"
- note removed: "do we need BSC master 0 data line and clock line? (for iic)"
- company: (none) -> Davide
- title: (none) -> Nautilus_Mainboard

Commit message: Deploying to gh-pages from @ Nautilus-UUV/nautilus-mainboard-PCB@03be77246175febedc852bdb83cb4e2df1ae0c88 🚀
Other:
- moved on the sheet: R1, R2
