File: Browse/CM4_LED2.kicad_sch (KiCad schematic)
At the start: 2 parts

Commit message: Deploying to gh-pages from @ Nautilus-UUV/nautilus-mainboard-PCB@8b02e89ade7c168188296ba6f0516f3abec9166b 🚀
Parts:
- removed D2: APHHS1005LZGCK-V, LED_SMD:LED_0402_1005Metric, symbol #dzdb:s_dio/D-KIN-APHHS1005LZGCK-V
- added LED7: 710-150060YS83000, dz_dio:Wuerth_LED_150060RS83000, symbol #dzdb:s_dio/D-WURT-710-150060YS83000
Connections:
- net Battery_Out_3.3V: now also LED7.2 (A)
- net at R6.2: now also LED7.1 (K)
Changed lines of the file:
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@@
   (paper "A4")
   (title_block
-    (date "2025-11-18")
+    (date "2025-11-19")
+    (rev "0")
     (company "Davide")
   )
@@
     (effects (font (size 1.27 1.27)))
   )
-  (hierarchical_label "PI_nLED_Activity" (shape input) (at 139.7 62.23 0)
+  (hierarchical_label "PI_nLED_Activity" (shape output) (at 139.7 62.23 0)
     (effects (font (size 1.27 1.27)) (justify left))
   )
@@
     )
   )
-  (symbol (lib_id "#dzdb:s_dio/D-KIN-APHHS1005LZGCK-V") (at 91.44 62.23 0) (mirror y) (unit 1)
+  (symbol (lib_id "#dzdb:s_dio/D-WURT-710-150060YS83000") (at 91.44 62.23 0) (unit 1)
     (exclude_from_sim no) (in_bom yes) (on_board yes) (dnp no) (fields_autoplaced)
-    (property "Reference" "D2" (at 93.0275 55.88 0)
+    (property "Reference" "LED7" (at 97.79 52.07 0)
       (effects (font (size 1.27 1.27)))
     )
-    (property "Value" "APHHS1005LZGCK-V" (at 93.0275 58.42 0)
+    (property "Value" "710-150060YS83000" (at 97.79 54.61 0)
       (effects (font (size 1.27 1.27)))
     )
-    (property "Footprint" "LED_SMD:LED_0402_1005Metric" (at 91.44 62.23 0)
+    (property "Footprint" "dz_dio:Wuerth_LED_150060RS83000" (at 104.14 155.88 0)
+      (effects (font (size 1.27 1.27)) (justify left bottom) (hide yes))
+    )
+    (property "Datasheet" "https://www.we-online.com/catalog/datasheet/150060SY83000.pdf" (at 104.14 255.88 0)
+      (effects (font (size 1.27 1.27)) (justify left bottom) (hide yes))
+    )
+    (property "Description" "Einfarbige LEDs leds WL-SMCW SMT 0603 Dome Yellow Typ 650mcd 2V" (at 91.44 62.23 0)
       (effects (font (size 1.27 1.27)) (hide yes))
     )
-    (property "Datasheet" "https://www.kingbrightusa.com/images/catalog/SPEC/APHHS1005LZGCK-V.pdf" (at 91.44 62.23 0)
+    (property "Height" "0.95" (at 104.14 455.88 0)
+      (effects (font (size 1.27 1.27)) (justify left bottom) (hide yes))
+    )
+    (property "Mouser Part Number" "" (at 104.14 555.88 0)
+      (effects (font (size 1.27 1.27)) (justify left bottom) (hide yes))
+    )
+    (property "Mouser Price/Stock" "" (at 104.14 655.88 0)
+      (effects (font (size 1.27 1.27)) (justify left bottom) (hide yes))
+    )
+    (property "Manufacturer_Name" "Wurth Elektronik" (at 104.14 755.88 0)
+      (effects (font (size 1.27 1.27)) (justify left bottom) (hide yes))
+    )
+    (property "Manufacturer_Part_Number" "150060RS83000" (at 104.14 855.88 0)
+      (effects (font (size 1.27 1.27)) (justify left bottom) (hide yes))
+    )
+    (property "IPN" "D-WURT-710-150060YS83000" (at 91.44 62.23 0)
       (effects (font (size 1.27 1.27)) (hide yes))
     )
-    (property "Description" "LED EMERALD GREEN 525nm 180mcd@2mA 40mcd@0.44mA 2.54V" (at 91.44 62.23 0)
+    (property "MPN" "710-150060YS83000" (at 91.44 62.23 0)
       (effects (font (size 1.27 1.27)) (hide yes))
     )
-    (property "Sim.Pins" "1=K 2=A" (at 91.44 62.23 0)
+    (property "Manufacturer" "Wurth Elektronik" (at 91.44 62.23 0)
       (effects (font (size 1.27 1.27)) (hide yes))
     )
-    (property "IPN" "D-KIN-APHHS1005LZGCK-V" (at 91.44 62.23 0)
+    (property "Type" "Einfarbige LEDs leds" (at 91.44 62.23 0)
       (effects (font (size 1.27 1.27)) (hide yes))
     )
-    (property "MPN" "APHHS1005LZGCK-V" (at 91.44 62.23 0)
+    (property "Vf" "2V" (at 91.44 62.23 0)
       (effects (font (size 1.27 1.27)) (hide yes))
     )
-    (property "Manufacturer" "Kingbright" (at 91.44 62.23 0)
-      (effects (font (size 1.27 1.27)) (hide yes))
-    )
-    (property "Type" "LED GREEN" (at 91.44 62.23 0)
-      (effects (font (size 1.27 1.27)) (hide yes))
-    )
-    (property "Vf" "2.65V" (at 91.44 62.23 0)
-      (effects (font (size 1.27 1.27)) (hide yes))
-    )
-    (property "If" "2mA" (at 91.44 62.23 0)
+    (property "If" "20 mA" (at 91.44 62.23 0)
       (effects (font (size 1.27 1.27)) (hide yes))
     )
@@
       (effects (font (size 1.27 1.27)) (hide yes))
     )
-    (property "SPN" "604-APHHS1005LZGCK-V" (at 91.44 62.23 0)
+    (property "SPN" "710-150060YS83000" (at 91.44 62.23 0)
       (effects (font (size 1.27 1.27)) (hide yes))
     )
-    (property "LCSC" "C5875752" (at 91.44 62.23 0)
+    (property "LCSC" "" (at 91.44 62.23 0)
       (effects (font (size 1.27 1.27)) (hide yes))
     )
-    (property "Comment" "lifecycle=Active" (at 91.44 62.23 0)
+    (property "Comment" "lifecycle=New Product" (at 91.44 62.23 0)
       (effects (font (size 1.27 1.27)) (hide yes))
     )
+    (pin "2")
     (pin "1")
-    (pin "2")
     (instances
-      (project "nautilus_mainboard"
+      (project ""
         (path "/ce1819b2-f280-40ed-834f-6fe4d12f809d/c2b6dac3-d6fd-4d5d-bd17-0cff91db88eb/0837dad1-ec16-488a-a684-981e55247089/b50f6d86-4325-4d05-931a-73973954b099"
-          (reference "D2") (unit 1)
+          (reference "LED7") (unit 1)
         )
       )

Commit message: Deploying to gh-pages from @ Nautilus-UUV/nautilus-mainboard-PCB@5b07cf6af03655ef9ddad269b1edd5eb03bfa75f 🚀
Other:
- title: (none) -> Nautilus_Mainboard
Changed lines of the file:
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@@
   (paper "A4")
   (title_block
+    (title "Nautilus_Mainboard")
     (date "2025-11-19")
     (rev "0")

Commit message: Deploying to gh-pages from @ Nautilus-UUV/nautilus-mainboard-PCB@5f5fdd9436d408a604bb268d740c0ac7ce1f5af5 🚀
Parts:
- removed LED7: 710-150060YS83000, dz_dio:Wuerth_LED_150060RS83000, symbol #dzdb:s_dio/D-WURT-710-150060YS83000
- added D2: APHHS1005LZGCK-V, LED_SMD:LED_0402_1005Metric, symbol #dzdb:s_dio/D-KIN-APHHS1005LZGCK-V
Connections:
- net at R6.2: now also D2.1 (K)
- new net CM4_LED_IN_3.3V: D2.2 (A)
Other:
- company: Davide -> (none)
- title: Nautilus_Mainboard -> (none)
- moved on the sheet: R6
Changed lines of the file:
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@@
 (kicad_sch (version 20250114) (generator "eeschema") (generator_version "9.0")
   (paper "A4")
-  (title_block
-    (title "Nautilus_Mainboard")
-    (date "2025-11-19")
-    (rev "0")
-    (company "Davide")
-  )
-  (wire (pts (xy 120.65 62.23) (xy 95.25 62.23))
+  (wire (pts (xy 90.17 62.23) (xy 115.57 62.23))
     (stroke (width 0) (type default))
   )
-  (wire (pts (xy 139.7 62.23) (xy 128.27 62.23))
+  (wire (pts (xy 71.12 62.23) (xy 82.55 62.23))
     (stroke (width 0) (type default))
   )
-  (wire (pts (xy 87.63 62.23) (xy 74.93 62.23))
+  (wire (pts (xy 123.19 62.23) (xy 135.89 62.23))
     (stroke (width 0) (type default))
   )
@@
     (effects (font (size 1.27 1.27)))
   )
-  (text "Activity LED" (exclude_from_sim no) (at 91.694 69.088 0)
+  (text "Activity LED" (exclude_from_sim no) (at 119.126 69.088 0)
     (effects (font (size 1.27 1.27)))
   )
-  (hierarchical_label "PI_nLED_Activity" (shape output) (at 139.7 62.23 0)
+  (global_label "CM4_LED_IN_3.3V" (shape input) (at 135.89 62.23 0) (fields_autoplaced)
     (effects (font (size 1.27 1.27)) (justify left))
+    (property "Intersheetrefs" "${INTERSHEET_REFS}" (at 155.2037 62.23 0)
+      (effects (font (size 1.27 1.27)) (justify left) (hide yes))
+    )
   )
-  (hierarchical_label "Battery_Out_3.3V" (shape input) (at 74.93 62.23 180)
+  (hierarchical_label "PI_nLED_Activity" (shape input) (at 71.12 62.23 180)
     (effects (font (size 1.27 1.27)) (justify right))
   )
-  (symbol (lib_id "#dzdb:g_res/R-1k-0603") (at 124.46 62.23 270) (mirror x) (unit 1)
+  (symbol (lib_id "#dzdb:g_res/R-1k-0603") (at 86.36 62.23 90) (unit 1)
     (exclude_from_sim no) (in_bom yes) (on_board yes) (dnp no) (fields_autoplaced)
-    (property "Reference" "R6" (at 124.46 55.88 90)
+    (property "Reference" "R6" (at 86.36 55.88 90)
       (effects (font (size 1.27 1.27)))
     )
-    (property "Value" "1k" (at 124.46 58.42 90)
+    (property "Value" "1k" (at 86.36 58.42 90)
       (effects (font (size 1.27 1.27)))
     )
-    (property "Footprint" "Resistor_SMD:R_0603_1608Metric" (at 124.46 64.008 90)
+    (property "Footprint" "Resistor_SMD:R_0603_1608Metric" (at 86.36 64.008 90)
       (effects (font (size 1.27 1.27)) (hide yes))
     )
-    (property "Datasheet" "https://www.we-online.com/components/products/datasheet/560112116014.pdf" (at 124.46 62.23 0)
+    (property "Datasheet" "https://www.we-online.com/components/products/datasheet/560112116014.pdf" (at 86.36 62.23 0)
       (effects (font (size 1.27 1.27)) (hide yes))
     )
-    (property "Description" "Thick Film Resistors - SMD WRIS-RSKS 1 kOhms 1 % 0.1 W 0603" (at 124.46 62.23 0)
+    (property "Description" "Thick Film Resistors - SMD WRIS-RSKS 1 kOhms 1 % 0.1 W 0603" (at 86.36 62.23 0)
       (effects (font (size 1.27 1.27)) (hide yes))
     )
-    (property "IPN" "R-1k-0603" (at 124.46 62.23 0)
+    (property "IPN" "R-1k-0603" (at 86.36 62.23 0)
       (effects (font (size 1.27 1.27)) (hide yes))
     )
-    (property "MPN" "560112116014" (at 124.46 62.23 0)
+    (property "MPN" "560112116014" (at 86.36 62.23 0)
       (effects (font (size 1.27 1.27)) (hide yes))
     )
-    (property "Manufacturer" "Wurth Elektronik" (at 124.46 62.23 0)
+    (property "Manufacturer" "Wurth Elektronik" (at 86.36 62.23 0)
       (effects (font (size 1.27 1.27)) (hide yes))
     )
-    (property "Resistance" "1k" (at 124.46 62.23 0)
+    (property "Resistance" "1k" (at 86.36 62.23 0)
       (effects (font (size 1.27 1.27)) (hide yes))
     )
-    (property "Power" "0.1 W" (at 124.46 62.23 0)
+    (property "Power" "0.1 W" (at 86.36 62.23 0)
       (effects (font (size 1.27 1.27)) (hide yes))
     )
-    (property "Material" "Thick film" (at 124.46 62.23 0)
+    (property "Material" "Thick film" (at 86.36 62.23 0)
       (effects (font (size 1.27 1.27)) (hide yes))
     )
-    (property "Tolerance" "1 %" (at 124.46 62.23 0)
+    (property "Tolerance" "1 %" (at 86.36 62.23 0)
       (effects (font (size 1.27 1.27)) (hide yes))
     )
-    (property "Supplier" "Mouser" (at 124.46 62.23 0)
+    (property "Supplier" "Mouser" (at 86.36 62.23 0)
       (effects (font (size 1.27 1.27)) (hide yes))
     )
-    (property "SPN" "710-560112116014" (at 124.46 62.23 0)
+    (property "SPN" "710-560112116014" (at 86.36 62.23 0)
       (effects (font (size 1.27 1.27)) (hide yes))
     )
-    (property "LCSC" "CXXXXX" (at 124.46 62.23 0)
+    (property "LCSC" "CXXXXX" (at 86.36 62.23 0)
       (effects (font (size 1.27 1.27)) (hide yes))
     )
-    (property "Comment" "lifecycle=Active; note=Auto-generated" (at 124.46 62.23 0)
+    (property "Comment" "lifecycle=Active; note=Auto-generated" (at 86.36 62.23 0)
       (effects (font (size 1.27 1.27)) (hide yes))
     )
@@
     )
   )
-  (symbol (lib_id "#dzdb:s_dio/D-WURT-710-150060YS83000") (at 91.44 62.23 0) (unit 1)
+  (symbol (lib_id "#dzdb:s_dio/D-KIN-APHHS1005LZGCK-V") (at 119.38 62.23 0) (unit 1)
     (exclude_from_sim no) (in_bom yes) (on_board yes) (dnp no) (fields_autoplaced)
-    (property "Reference" "LED7" (at 97.79 52.07 0)
+    (property "Reference" "D2" (at 117.7925 55.88 0)
       (effects (font (size 1.27 1.27)))
     )
-    (property "Value" "710-150060YS83000" (at 97.79 54.61 0)
+    (property "Value" "APHHS1005LZGCK-V" (at 117.7925 58.42 0)
       (effects (font (size 1.27 1.27)))
     )
-    (property "Footprint" "dz_dio:Wuerth_LED_150060RS83000" (at 104.14 155.88 0)
-      (effects (font (size 1.27 1.27)) (justify left bottom) (hide yes))
-    )
-    (property "Datasheet" "https://www.we-online.com/catalog/datasheet/150060SY83000.pdf" (at 104.14 255.88 0)
-      (effects (font (size 1.27 1.27)) (justify left bottom) (hide yes))
-    )
-    (property "Description" "Einfarbige LEDs leds WL-SMCW SMT 0603 Dome Yellow Typ 650mcd 2V" (at 91.44 62.23 0)
+    (property "Footprint" "LED_SMD:LED_0402_1005Metric" (at 119.38 62.23 0)
       (effects (font (size 1.27 1.27)) (hide yes))
     )
-    (property "Height" "0.95" (at 104.14 455.88 0)
-      (effects (font (size 1.27 1.27)) (justify left bottom) (hide yes))
-    )
-    (property "Mouser Part Number" "" (at 104.14 555.88 0)
-      (effects (font (size 1.27 1.27)) (justify left bottom) (hide yes))
-    )
-    (property "Mouser Price/Stock" "" (at 104.14 655.88 0)
-      (effects (font (size 1.27 1.27)) (justify left bottom) (hide yes))
-    )
-    (property "Manufacturer_Name" "Wurth Elektronik" (at 104.14 755.88 0)
-      (effects (font (size 1.27 1.27)) (justify left bottom) (hide yes))
-    )
-    (property "Manufacturer_Part_Number" "150060RS83000" (at 104.14 855.88 0)
-      (effects (font (size 1.27 1.27)) (justify left bottom) (hide yes))
-    )
-    (property "IPN" "D-WURT-710-150060YS83000" (at 91.44 62.23 0)
+    (property "Datasheet" "https://www.kingbrightusa.com/images/catalog/SPEC/APHHS1005LZGCK-V.pdf" (at 119.38 62.23 0)
       (effects (font (size 1.27 1.27)) (hide yes))
     )
-    (property "MPN" "710-150060YS83000" (at 91.44 62.23 0)
+    (property "Description" "LED EMERALD GREEN 525nm 180mcd@2mA 40mcd@0.44mA 2.54V" (at 119.38 62.23 0)
       (effects (font (size 1.27 1.27)) (hide yes))
     )
-    (property "Manufacturer" "Wurth Elektronik" (at 91.44 62.23 0)
+    (property "Sim.Pins" "1=K 2=A" (at 119.38 62.23 0)
       (effects (font (size 1.27 1.27)) (hide yes))
     )
-    (property "Type" "Einfarbige LEDs leds" (at 91.44 62.23 0)
+    (property "IPN" "D-KIN-APHHS1005LZGCK-V" (at 119.38 62.23 0)
       (effects (font (size 1.27 1.27)) (hide yes))
     )
-    (property "Vf" "2V" (at 91.44 62.23 0)
+    (property "MPN" "APHHS1005LZGCK-V" (at 119.38 62.23 0)
       (effects (font (size 1.27 1.27)) (hide yes))
     )
-    (property "If" "20 mA" (at 91.44 62.23 0)
+    (property "Manufacturer" "Kingbright" (at 119.38 62.23 0)
       (effects (font (size 1.27 1.27)) (hide yes))
     )
-    (property "Supplier" "Mouser" (at 91.44 62.23 0)
+    (property "Type" "LED GREEN" (at 119.38 62.23 0)
       (effects (font (size 1.27 1.27)) (hide yes))
     )
-    (property "SPN" "710-150060YS83000" (at 91.44 62.23 0)
+    (property "Vf" "2.65V" (at 119.38 62.23 0)
       (effects (font (size 1.27 1.27)) (hide yes))
     )
-    (property "LCSC" "" (at 91.44 62.23 0)
+    (property "If" "2mA" (at 119.38 62.23 0)
       (effects (font (size 1.27 1.27)) (hide yes))
     )
-    (property "Comment" "lifecycle=New Product" (at 91.44 62.23 0)
+    (property "Supplier" "Mouser" (at 119.38 62.23 0)
       (effects (font (size 1.27 1.27)) (hide yes))
     )
+    (property "SPN" "604-APHHS1005LZGCK-V" (at 119.38 62.23 0)
+      (effects (font (size 1.27 1.27)) (hide yes))
+    )
+    (property "LCSC" "C5875752" (at 119.38 62.23 0)
+      (effects (font (size 1.27 1.27)) (hide yes))
+    )
+    (property "Comment" "lifecycle=Active" (at 119.38 62.23 0)
+      (effects (font (size 1.27 1.27)) (hide yes))
+    )
+    (pin "1")
     (pin "2")
-    (pin "1")
     (instances
-      (project ""
+      (project "nautilus_mainboard"
         (path "/ce1819b2-f280-40ed-834f-6fe4d12f809d/c2b6dac3-d6fd-4d5d-bd17-0cff91db88eb/0837dad1-ec16-488a-a684-981e55247089/b50f6d86-4325-4d05-931a-73973954b099"
-          (reference "LED7") (unit 1)
+          (reference "D2") (unit 1)
         )
       )

Commit message: Deploying to gh-pages from @ Nautilus-UUV/nautilus-mainboard-PCB@44ad8adb17f33e1aa4439bd10449a9ac7e221a1f 🚀
Connections:
- net CM4_LED_IN_3.3V renamed Battery_Out_3.3V
Changed lines of the file:
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@@
     (effects (font (size 1.27 1.27)))
   )
-  (global_label "CM4_LED_IN_3.3V" (shape input) (at 135.89 62.23 0) (fields_autoplaced)
+  (global_label "Battery_Out_3.3V" (shape input) (at 135.89 62.23 0) (fields_autoplaced)
     (effects (font (size 1.27 1.27)) (justify left))
-    (property "Intersheetrefs" "${INTERSHEET_REFS}" (at 155.2037 62.23 0)
+    (property "Intersheetrefs" "${INTERSHEET_REFS}" (at 154.8408 62.23 0)
       (effects (font (size 1.27 1.27)) (justify left) (hide yes))
     )
