File: Browse/CM4_Ethernet.kicad_sch (KiCad schematic)
At the start: 6 parts

Commit message: Deploying to gh-pages from @ Nautilus-UUV/nautilus-mainboard-PCB@b62834b88bb3e2a9413bcb4ea8e223af403e20ba 🚀
Connections:
- net TRD0_N renamed TRD0.D-
- net TRD0_P renamed TRD0.D+
- net TRD1_N renamed TRD1.D-
- net TRD1_P renamed TRD1.D+
- net TRD2_N renamed TRD2.D-
- net TRD2_P renamed TRD2.D+
- net TRD3_N renamed TRD3.D-
- net TRD3_P renamed TRD3.D+
Other:
- moved on the sheet: D3, D4, R7, R8

Commit message: Deploying to gh-pages from @ Nautilus-UUV/nautilus-mainboard-PCB@f1dd6ce1e57c066b805694b10777c719502cca87 🚀
Parts:
- removed D3: APHHS1005LSYCK/J3-PF, LED_SMD:LED_0402_1005Metric, symbol #dzdb:s_dio/D-KIN-APHHS1005LSYCK/J3-PF
- removed D4: APHHS1005LZGCK-V, LED_SMD:LED_0402_1005Metric, symbol #dzdb:s_dio/D-KIN-APHHS1005LZGCK-V
- added LED5: 710-150060VS83000, dz_dio:Wuerth_LED_150060RS83000, symbol #dzdb:s_dio/D-WURT-710-150060VS83000
- added LED6: 710-150060YS83000, dz_dio:Wuerth_LED_150060RS83000, symbol #dzdb:s_dio/D-WURT-710-150060YS83000
Connections:
- net ETH_LED_G: now also LED5.1 (K)
- net ETH_LED_Y: now also LED6.1 (K)
- net at R7.1: now also LED5.2 (A)
- net at R8.1: now also LED6.2 (A)
Other:
- note removed: "Optimal: Green: 325 Ohm (3.3-2.65)/0.002"
- note removed: "Optimal: Yellow: 725 Ohm (3.3-1.85)/0.002"
- company: (none) -> Davide
- title: (none) -> Nautilus_Mainboard
- moved on the sheet: R7, R8

Commit message: Deploying to gh-pages from @ Nautilus-UUV/nautilus-mainboard-PCB@5f5fdd9436d408a604bb268d740c0ac7ce1f5af5 🚀
Parts:
- removed LED5: 710-150060VS83000, dz_dio:Wuerth_LED_150060RS83000, symbol #dzdb:s_dio/D-WURT-710-150060VS83000
- removed LED6: 710-150060YS83000, dz_dio:Wuerth_LED_150060RS83000, symbol #dzdb:s_dio/D-WURT-710-150060YS83000
- added D3: APHHS1005LSYCK/J3-PF, LED_SMD:LED_0402_1005Metric, symbol #dzdb:s_dio/D-KIN-APHHS1005LSYCK/J3-PF
- added D4: APHHS1005LZGCK-V, LED_SMD:LED_0402_1005Metric, symbol #dzdb:s_dio/D-KIN-APHHS1005LZGCK-V
Connections:
- net ETH_LED_G: now also D4.1 (K)
- net ETH_LED_Y: now also D3.1 (K)
- net at R7.1: now also D4.2 (A)
- net at R8.1: now also D3.2 (A)
Other:
- note added: "Optimal: Green: 325 Ohm (3.3-2.65)/0.002"
- note added: "Optimal: Yellow: 725 Ohm (3.3-1.85)/0.002"
- company: Davide -> (none)
- title: Nautilus_Mainboard -> (none)
- moved on the sheet: R7, R8

Commit message: Deploying to gh-pages from @ Nautilus-UUV/nautilus-mainboard-PCB@44ad8adb17f33e1aa4439bd10449a9ac7e221a1f 🚀
Changed lines of the file:
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@@
 (kicad_sch (version 20250114) (generator "eeschema") (generator_version "9.0")
   (paper "A4")
-  (junction (at 134.62 57.15) (diameter 0) (color 0 0 0 0)
+  (junction (at 134.62 54.61) (diameter 0) (color 0 0 0 0)
+  )
+  (junction (at 134.62 100.33) (diameter 0) (color 0 0 0 0)
   )
   (junction (at 224.79 43.18) (diameter 0) (color 0 0 0 0)
   )
-  (junction (at 134.62 102.87) (diameter 0) (color 0 0 0 0)
-  )
   (bus_entry (at 146.05 44.45) (size -2.54 2.54)
     (stroke (width 0) (type default))
@@
     (stroke (width 0) (type default))
   )
-  (wire (pts (xy 134.62 57.15) (xy 138.43 57.15))
+  (wire (pts (xy 134.62 54.61) (xy 138.43 54.61))
     (stroke (width 0) (type default))
   )
@@
     (stroke (width 0) (type default))
   )
-  (wire (pts (xy 134.62 102.87) (xy 138.43 102.87))
-    (stroke (width 0) (type default))
-  )
   (wire (pts (xy 179.07 44.45) (xy 186.69 44.45))
     (stroke (width 0) (type default))
@@
   )
   (bus (pts (xy 146.05 59.69) (xy 146.05 62.23))
+    (stroke (width 0) (type default))
+  )
+  (wire (pts (xy 134.62 100.33) (xy 140.97 100.33))
     (stroke (width 0) (type default))
   )
@@
     (effects (font (size 1.27 1.27)) (justify right))
   )
-  (symbol (lib_id "power:GND") (at 138.43 57.15 0) (unit 1)
+  (symbol (lib_id "power:GND") (at 138.43 54.61 0) (unit 1)
     (exclude_from_sim no) (in_bom yes) (on_board yes) (dnp no)
-    (property "Reference" "#PWR019" (at 138.43 63.5 0)
-      (effects (font (size 1.27 1.27)) (hide yes))
-    )
-    (property "Value" "GND" (at 141.986 57.912 0)
-      (effects (font (size 1.27 1.27)))
-    )
-    (property "Footprint" "" (at 138.43 57.15 0)
-      (effects (font (size 1.27 1.27)) (hide yes))
-    )
-    (property "Datasheet" "" (at 138.43 57.15 0)
-      (effects (font (size 1.27 1.27)) (hide yes))
-    )
-    (property "Description" "Power symbol creates a global label with name \"GND\" , ground" (at 138.43 57.15 0)
+    (property "Reference" "#PWR019" (at 138.43 60.96 0)
+      (effects (font (size 1.27 1.27)) (hide yes))
+    )
+    (property "Value" "GND" (at 141.986 55.372 0)
+      (effects (font (size 1.27 1.27)))
+    )
+    (property "Footprint" "" (at 138.43 54.61 0)
+      (effects (font (size 1.27 1.27)) (hide yes))
+    )
+    (property "Datasheet" "" (at 138.43 54.61 0)
+      (effects (font (size 1.27 1.27)) (hide yes))
+    )
+    (property "Description" "Power symbol creates a global label with name \"GND\" , ground" (at 138.43 54.61 0)
       (effects (font (size 1.27 1.27)) (hide yes))
     )
@@
     )
   )
-  (symbol (lib_id "power:GND") (at 138.43 102.87 0) (unit 1)
+  (symbol (lib_id "power:GND") (at 140.97 100.33 0) (unit 1)
     (exclude_from_sim no) (in_bom yes) (on_board yes) (dnp no) (fields_autoplaced)
-    (property "Reference" "#PWR020" (at 138.43 109.22 0)
-      (effects (font (size 1.27 1.27)) (hide yes))
-    )
-    (property "Value" "GND" (at 138.43 107.95 0)
-      (effects (font (size 1.27 1.27)))
-    )
-    (property "Footprint" "" (at 138.43 102.87 0)
-      (effects (font (size 1.27 1.27)) (hide yes))
-    )
-    (property "Datasheet" "" (at 138.43 102.87 0)
-      (effects (font (size 1.27 1.27)) (hide yes))
-    )
-    (property "Description" "Power symbol creates a global label with name \"GND\" , ground" (at 138.43 102.87 0)
-      (effects (font (size 1.27 1.27)) (hide yes))
-    )
+    (property "Reference" "#PWR020" (at 140.97 106.68 0)
+      (effects (font (size 1.27 1.27)) (hide yes))
+    )
+    (property "Value" "GND" (at 140.97 105.41 0)
+      (effects (font (size 1.27 1.27)))
+    )
+    (property "Footprint" "" (at 140.97 100.33 0)
+      (effects (font (size 1.27 1.27)) (hide yes))
+    )
+    (property "Datasheet" "" (at 140.97 100.33 0)
+      (effects (font (size 1.27 1.27)) (hide yes))
+    )
+    (property "Description" "Power symbol creates a global label with name \"GND\" , ground" (at 140.97 100.33 0)
+      (effects (font (size 1.27 1.27)) (hide yes))
+    )

Commit message: Deploying to gh-pages from @ Nautilus-UUV/nautilus-mainboard-PCB@a81f7ffbfc5f9b51f47d7f388c30fcea2673b9ea 🚀
Other:
- moved on the sheet: D3, D4, R7, R8

Commit message: Deploying to gh-pages from @ Nautilus-UUV/nautilus-mainboard-PCB@2d3890115fd9d3c0bb909c9898aa64801bed9e67 🚀
Other:
- company: (none) -> Davide
Changed lines of the file:
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@@
 (kicad_sch (version 20250114) (generator "eeschema") (generator_version "9.0")
   (paper "A4")
+  (title_block
+    (date "2025-11-18")
+    (company "Davide")
+  )
   (junction (at 134.62 54.61) (diameter 0) (color 0 0 0 0)
   )

Commit message: Deploying to gh-pages from @ Nautilus-UUV/nautilus-mainboard-PCB@8b02e89ade7c168188296ba6f0516f3abec9166b 🚀
Parts:
- removed D3: APHHS1005LSYCK/J3-PF, LED_SMD:LED_0402_1005Metric, symbol #dzdb:s_dio/D-KIN-APHHS1005LSYCK/J3-PF
- removed D4: APHHS1005LZGCK-V, LED_SMD:LED_0402_1005Metric, symbol #dzdb:s_dio/D-KIN-APHHS1005LZGCK-V
- added LED5: 710-150060VS83000, dz_dio:Wuerth_LED_150060RS83000, symbol #dzdb:s_dio/D-WURT-710-150060VS83000
- added LED6: 710-150060YS83000, dz_dio:Wuerth_LED_150060RS83000, symbol #dzdb:s_dio/D-WURT-710-150060YS83000
Connections:
- net ETH_LED_G: now also LED5.1 (K)
- net ETH_LED_Y: now also LED6.1 (K)
- net at R7.1: now also LED5.2 (A)
- net at R8.1: now also LED6.2 (A)
Other:
- note removed: "Optimal: Green: 325 Ohm (3.3-2.65)/0.002"
- note removed: "Optimal: Yellow: 725 Ohm (3.3-1.85)/0.002"

Commit message: Deploying to gh-pages from @ Nautilus-UUV/nautilus-mainboard-PCB@5b07cf6af03655ef9ddad269b1edd5eb03bfa75f 🚀
Other:
- title: (none) -> Nautilus_Mainboard
Changed lines of the file:
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@@
   (paper "A4")
   (title_block
+    (title "Nautilus_Mainboard")
     (date "2025-11-19")
     (rev "0")
