File: Browse/LPHT-connector.kicad_sch (KiCad schematic)
At the start: 1 part, among them J7 LPHT-04-16-L-RT1-GP

Commit message: Deploying to gh-pages from @ Nautilus-UUV/nautilus-mainboard-PCB@b62834b88bb3e2a9413bcb4ea8e223af403e20ba 🚀
Connections:
- net ET1 renamed TRD0.D-
- net ET2 renamed TRD0.D+
- net ET3 renamed TRD1.D-
- net ET4 renamed TRD1.D+
- net ET5 renamed TRD2.D-
- net ET6 renamed TRD2.D+
- net ET7 renamed TRD3.D-
- net ET8 renamed TRD3.D+
Changed lines of the file:
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@@
   (no_connect (at 242.57 102.87))
   (no_connect (at 217.17 120.65))
+  (bus_entry (at 260.35 72.39) (size -2.54 2.54)
+    (stroke (width 0) (type default))
+  )
+  (bus_entry (at 260.35 85.09) (size -2.54 2.54)
+    (stroke (width 0) (type default))
+  )
+  (bus_entry (at 260.35 80.01) (size -2.54 2.54)
+    (stroke (width 0) (type default))
+  )
+  (bus_entry (at 260.35 77.47) (size -2.54 2.54)
+    (stroke (width 0) (type default))
+  )
+  (bus_entry (at 260.35 87.63) (size -2.54 2.54)
+    (stroke (width 0) (type default))
+  )
+  (bus_entry (at 260.35 90.17) (size -2.54 2.54)
+    (stroke (width 0) (type default))
+  )
+  (bus_entry (at 260.35 74.93) (size -2.54 2.54)
+    (stroke (width 0) (type default))
+  )
+  (bus_entry (at 260.35 82.55) (size -2.54 2.54)
+    (stroke (width 0) (type default))
+  )
   (wire (pts (xy 205.74 87.63) (xy 217.17 87.63))
     (stroke (width 0) (type default))
   )
-  (wire (pts (xy 242.57 85.09) (xy 250.19 85.09))
+  (wire (pts (xy 242.57 85.09) (xy 257.81 85.09))
     (stroke (width 0) (type default))
   )
@@
     (stroke (width 0) (type default))
   )
-  (wire (pts (xy 242.57 80.01) (xy 250.19 80.01))
+  (wire (pts (xy 242.57 80.01) (xy 257.81 80.01))
     (stroke (width 0) (type default))
   )
@@
     (stroke (width 0) (type default))
   )
+  (bus (pts (xy 260.35 72.39) (xy 260.35 74.93))
+    (stroke (width 0) (type default))
+  )
   (wire (pts (xy 217.17 105.41) (xy 217.17 107.95))
     (stroke (width 0) (type default))
   )
+  (bus (pts (xy 261.62 82.55) (xy 260.35 82.55))
+    (stroke (width 0) (type default))
+  )
   (wire (pts (xy 205.74 76.2) (xy 217.17 76.2))
     (stroke (width 0) (type default))
@@
     (stroke (width 0) (type default))
   )
+  (bus (pts (xy 260.35 82.55) (xy 260.35 85.09))
+    (stroke (width 0) (type default))
+  )
+  (bus (pts (xy 260.35 87.63) (xy 260.35 90.17))
+    (stroke (width 0) (type default))
+  )
   (wire (pts (xy 242.57 115.57) (xy 242.57 118.11))
     (stroke (width 0) (type default))
   )
-  (wire (pts (xy 242.57 87.63) (xy 250.19 87.63))
-    (stroke (width 0) (type default))
-  )
-  (wire (pts (xy 242.57 90.17) (xy 250.19 90.17))
-    (stroke (width 0) (type default))
-  )
-  (wire (pts (xy 242.57 82.55) (xy 250.19 82.55))
+  (wire (pts (xy 242.57 87.63) (xy 257.81 87.63))
+    (stroke (width 0) (type default))
+  )
+  (wire (pts (xy 242.57 90.17) (xy 257.81 90.17))
+    (stroke (width 0) (type default))
+  )
+  (wire (pts (xy 242.57 82.55) (xy 257.81 82.55))
     (stroke (width 0) (type default))
   )
@@
     (stroke (width 0) (type default))
   )
+  (bus (pts (xy 261.62 87.63) (xy 260.35 87.63))
+    (stroke (width 0) (type default))
+  )
   (wire (pts (xy 217.17 76.2) (xy 217.17 77.47))
     (stroke (width 0) (type default))
@@
     (stroke (width 0) (type default))
   )
-  (wire (pts (xy 242.57 77.47) (xy 250.19 77.47))
-    (stroke (width 0) (type default))
-  )
-  (wire (pts (xy 242.57 74.93) (xy 250.19 74.93))
+  (wire (pts (xy 242.57 77.47) (xy 257.81 77.47))
+    (stroke (width 0) (type default))
+  )
+  (wire (pts (xy 242.57 74.93) (xy 257.81 74.93))
+    (stroke (width 0) (type default))
+  )
+  (bus (pts (xy 261.62 72.39) (xy 260.35 72.39))
     (stroke (width 0) (type default))
   )
@@
     (stroke (width 0) (type default))
   )
+  (bus (pts (xy 261.62 77.47) (xy 260.35 77.47))
+    (stroke (width 0) (type default))
+  )
   (wire (pts (xy 217.17 102.87) (xy 217.17 105.41))
     (stroke (width 0) (type default))
@@
     (stroke (width 0) (type default))
   )
+  (bus (pts (xy 260.35 77.47) (xy 260.35 80.01))
+    (stroke (width 0) (type default))
+  )
   (wire (pts (xy 217.17 100.33) (xy 217.17 102.87))
     (stroke (width 0) (type default))
@@
     (stroke (width 0) (type default))
   )
-  (wire (pts (xy 242.57 92.71) (xy 250.19 92.71))
+  (wire (pts (xy 242.57 92.71) (xy 257.81 92.71))
     (stroke (width 0) (type default))
   )
@@
   )
   (text_box "Counterpiece to  LPHS-04-16-L-VP1-GP"
-    (exclude_from_sim no) (at 185.42 60.96 0) (size 83.82 71.12)
+    (exclude_from_sim no) (at 185.42 60.96 0) (size 93.98 71.12)
     (margins 0.9525 0.9525 0.9525 0.9525) (stroke (width 0) (type solid))
     (fill (type none))
     (effects (font (size 1.27 1.27)) (justify left top))
   )
-  (text "9-16 lan\n" (exclude_from_sim no) (at 261.62 83.566 0)
+  (text "9-16 lan\n" (exclude_from_sim no) (at 256.54 94.742 0)
     (effects (font (size 1.27 1.27)))
   )
@@
     (effects (font (size 1.27 1.27)) (justify left bottom))
   )
+  (label "TRD2.D+" (at 254 87.63 180)
+    (effects (font (size 1.27 1.27)) (justify right bottom))
+  )
+  (label "TRD1.D+" (at 254 82.55 180)
+    (effects (font (size 1.27 1.27)) (justify right bottom))
+  )
+  (label "TRD3.D-" (at 254 90.17 180)
+    (effects (font (size 1.27 1.27)) (justify right bottom))
+  )
+  (label "TRD2.D-" (at 254 85.09 180)
+    (effects (font (size 1.27 1.27)) (justify right bottom))
+  )
   (label "RX_STM" (at 205.74 87.63 0)
     (effects (font (size 1.27 1.27)) (justify left bottom))
@@
   (label "RX_PI" (at 205.74 82.55 0)
     (effects (font (size 1.27 1.27)) (justify left bottom))
+  )
+  (label "TRD3.D+" (at 254 92.71 180)
+    (effects (font (size 1.27 1.27)) (justify right bottom))
+  )
+  (label "TRD0.D+" (at 254 77.47 180)
+    (effects (font (size 1.27 1.27)) (justify right bottom))
+  )
+  (label "TRD1.D-" (at 254 80.01 180)
+    (effects (font (size 1.27 1.27)) (justify right bottom))
+  )
+  (label "TRD0.D-" (at 254 74.93 180)
+    (effects (font (size 1.27 1.27)) (justify right bottom))
   )
   (global_label "Battery_Out_3.3V" (shape output) (at 205.74 76.2 180) (fields_autoplaced)
@@
     )
   )
-  (hierarchical_label "ET2" (shape input) (at 250.19 77.47 0)
+  (hierarchical_label "TRD3{D+ D-}" (shape bidirectional) (at 261.62 87.63 0)
     (effects (font (size 1.27 1.27)) (justify left))
   )
-  (hierarchical_label "ET5" (shape input) (at 250.19 85.09 0)
+  (hierarchical_label "TRD1{D+ D-}" (shape bidirectional) (at 261.62 77.47 0)
     (effects (font (size 1.27 1.27)) (justify left))
   )
-  (hierarchical_label "ET8" (shape input) (at 250.19 92.71 0)
+  (hierarchical_label "TRD2{D+ D-}" (shape bidirectional) (at 261.62 82.55 0)
     (effects (font (size 1.27 1.27)) (justify left))
   )
-  (hierarchical_label "ET3" (shape input) (at 250.19 80.01 0)
+  (hierarchical_label "TRD0{D+ D-}" (shape bidirectional) (at 261.62 72.39 0)
     (effects (font (size 1.27 1.27)) (justify left))
   )
-  (hierarchical_label "ET6" (shape input) (at 250.19 87.63 0)
-    (effects (font (size 1.27 1.27)) (justify left))
-  )
-  (hierarchical_label "ET7" (shape input) (at 250.19 90.17 0)
-    (effects (font (size 1.27 1.27)) (justify left))
-  )
-  (hierarchical_label "ET4" (shape input) (at 250.19 82.55 0)
-    (effects (font (size 1.27 1.27)) (justify left))
-  )
-  (hierarchical_label "ET1" (shape input) (at 250.19 74.93 0)
-    (effects (font (size 1.27 1.27)) (justify left))
-  )

Commit message: Deploying to gh-pages from @ Nautilus-UUV/nautilus-mainboard-PCB@a20f16cf7e6ebba0b5127d7f7acbd1e63379e186 🚀
Changed lines of the file:
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@@
     )
   )
-  (global_label "STM_RX" (shape input) (at 205.74 87.63 180) (fields_autoplaced)
+  (global_label "STM_RX" (shape output) (at 205.74 87.63 180) (fields_autoplaced)
     (effects (font (size 1.27 1.27)) (justify right))
     (property "Intersheetrefs" "${INTERSHEET_REFS}" (at 195.6792 87.63 0)
@@
     )
   )
-  (global_label "ST_CAN_N" (shape input) (at 205.74 92.71 180) (fields_autoplaced)
+  (global_label "ST_CAN_N" (shape bidirectional) (at 205.74 92.71 180) (fields_autoplaced)
     (effects (font (size 1.27 1.27)) (justify right))
-    (property "Intersheetrefs" "${INTERSHEET_REFS}" (at 193.6229 92.71 0)
+    (property "Intersheetrefs" "${INTERSHEET_REFS}" (at 192.5116 92.71 0)
       (effects (font (size 1.27 1.27)) (justify right) (hide yes))
     )
@@
     )
   )
-  (global_label "ST_CAN_P" (shape input) (at 205.74 90.17 180) (fields_autoplaced)
+  (global_label "ST_CAN_P" (shape bidirectional) (at 205.74 90.17 180) (fields_autoplaced)
     (effects (font (size 1.27 1.27)) (justify right))
-    (property "Intersheetrefs" "${INTERSHEET_REFS}" (at 193.6834 90.17 0)
+    (property "Intersheetrefs" "${INTERSHEET_REFS}" (at 192.5721 90.17 0)
       (effects (font (size 1.27 1.27)) (justify right) (hide yes))
     )

Commit message: Deploying to gh-pages from @ Nautilus-UUV/nautilus-mainboard-PCB@f1dd6ce1e57c066b805694b10777c719502cca87 🚀
Parts:
- added D1: 710-82402374, Package_TO_SOT_SMD:SOT-23-5, symbol #dzdb:s_dio/WURT-710-82402374
- added LED1, LED2: 710-150060RS83000, dz_dio:Wuerth_LED_150060RS83000, symbol #dzdb:s_dio/D-WURT-710-150060RS83000
- added R16: 1k, Resistor_SMD:R_0603_1608Metric, symbol #dzdb:g_res/R-1k-0603
- added R18: 2.2k, Resistor_SMD:R_0603_1608Metric, symbol #dzdb:g_res/R-2.2k-0603
Connections:
- net Battery_Out_3.3V: now also D1.3 (K), R16.2
- net Battery_Out_5V: now also D1.1 (K), R18.1
- net GND: now also D1.2 (A), LED1.1 (K), LED2.1 (K)
- net RX_PI: no longer names the net of J7.04
- net STM_RX renamed STM.RX
- net STM_TX renamed STM.TX
- net ST_CAN_N renamed ST_CAN.N
- net ST_CAN_P renamed ST_CAN.P
- net TX_PI: no longer names the net of J7.03
- new net: LED2.2 (A), R18.2
- new net: LED1.2 (A), R16.1
- no-connect marks 10 -> 14
Other:
- note added: "I_{F} = 20mA V_{in} = 3.3V V_{F} ≈ 2.0V"
- note added: "I_{F} = 20mA V_{in} = 5V V_{F} ≈ 2.0V"
- note added: "R= (V_{in} - V_{F}) / I_{F}"
- note added: "So min R is 150Ω"
- note added: "So min R is 68Ω"
- company: (none) -> Davide, Evan
- title: (none) -> Nautilus_Mainboard
- moved on the sheet: J7

Commit message: Deploying to gh-pages from @ Nautilus-UUV/nautilus-mainboard-PCB@5f5fdd9436d408a604bb268d740c0ac7ce1f5af5 🚀
Parts:
- removed D1: 710-82402374, Package_TO_SOT_SMD:SOT-23-5, symbol #dzdb:s_dio/WURT-710-82402374
- removed LED1, LED2: 710-150060RS83000, dz_dio:Wuerth_LED_150060RS83000, symbol #dzdb:s_dio/D-WURT-710-150060RS83000
- removed R16: 1k, Resistor_SMD:R_0603_1608Metric, symbol #dzdb:g_res/R-1k-0603
- removed R18: 2.2k, Resistor_SMD:R_0603_1608Metric, symbol #dzdb:g_res/R-2.2k-0603
Connections:
- net TX_PI: now reaches J7.03
- net RX_PI: now reaches J7.04
- net STM.RX renamed STM_RX
- net STM.TX renamed STM_TX
- net ST_CAN.N renamed ST_CAN_N
- net ST_CAN.P renamed ST_CAN_P
- no-connect marks 14 -> 10
Other:
- note removed: "I_{F} = 20mA V_{in} = 3.3V V_{F} ≈ 2.0V"
- note removed: "I_{F} = 20mA V_{in} = 5V V_{F} ≈ 2.0V"
- note removed: "R= (V_{in} - V_{F}) / I_{F}"
- note removed: "So min R is 150Ω"
- note removed: "So min R is 68Ω"
- company: Davide, Evan -> (none)
- title: Nautilus_Mainboard -> (none)
- moved on the sheet: J7

Commit message: Deploying to gh-pages from @ Nautilus-UUV/nautilus-mainboard-PCB@a81f7ffbfc5f9b51f47d7f388c30fcea2673b9ea 🚀
Connections:
- net RX_PI: no longer names the net of J7.04
- net TX_PI: no longer names the net of J7.03
- no-connect marks 10 -> 12
Changed lines of the file:
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@@
   (no_connect (at 217.17 113.03))
   (no_connect (at 217.17 118.11))
+  (no_connect (at 217.17 82.55))
   (no_connect (at 217.17 115.57))
   (no_connect (at 242.57 107.95))
@@
   (no_connect (at 217.17 110.49))
   (no_connect (at 242.57 102.87))
+  (no_connect (at 217.17 80.01))
   (no_connect (at 217.17 120.65))
   (bus_entry (at 260.35 72.39) (size -2.54 2.54)
@@
     (stroke (width 0) (type default))
   )
-  (wire (pts (xy 205.74 82.55) (xy 217.17 82.55))
-    (stroke (width 0) (type default))
-  )
   (wire (pts (xy 242.57 113.03) (xy 242.57 115.57))
     (stroke (width 0) (type default))
   )
   (wire (pts (xy 242.57 80.01) (xy 257.81 80.01))
-    (stroke (width 0) (type default))
-  )
-  (wire (pts (xy 205.74 80.01) (xy 217.17 80.01))
     (stroke (width 0) (type default))
   )
@@
     (effects (font (size 1.27 1.27)) (justify left bottom))
   )
-  (label "TX_PI" (at 205.74 80.01 0)
-    (effects (font (size 1.27 1.27)) (justify left bottom))
-  )
   (label "ST_CAN_P" (at 205.74 90.17 0)
     (effects (font (size 1.27 1.27)) (justify left bottom))
   )
   (label "ST_CAN_N" (at 205.74 92.71 0)
-    (effects (font (size 1.27 1.27)) (justify left bottom))
-  )
-  (label "RX_PI" (at 205.74 82.55 0)
     (effects (font (size 1.27 1.27)) (justify left bottom))
   )
@@
     )
   )
-  (global_label "STM_TX" (shape input) (at 205.74 85.09 180) (fields_autoplaced)
+  (global_label "STM_TX" (shape output) (at 205.74 85.09 180) (fields_autoplaced)
     (effects (font (size 1.27 1.27)) (justify right))
     (property "Intersheetrefs" "${INTERSHEET_REFS}" (at 195.9816 85.09 0)
@@
     )
   )
-  (global_label "ST_CAN_N" (shape input) (at 205.74 92.71 180) (fields_autoplaced)
+  (global_label "ST_CAN_N" (shape bidirectional) (at 205.74 92.71 180) (fields_autoplaced)
     (effects (font (size 1.27 1.27)) (justify right))
-    (property "Intersheetrefs" "${INTERSHEET_REFS}" (at 193.6229 92.71 0)
+    (property "Intersheetrefs" "${INTERSHEET_REFS}" (at 192.5116 92.71 0)
       (effects (font (size 1.27 1.27)) (justify right) (hide yes))
     )
   )
-  (global_label "Battery_Out_5V" (shape output) (at 205.74 100.33 180) (fields_autoplaced)
+  (global_label "ST_CAN_P" (shape bidirectional) (at 205.74 90.17 180) (fields_autoplaced)
     (effects (font (size 1.27 1.27)) (justify right))
-    (property "Intersheetrefs" "${INTERSHEET_REFS}" (at 188.6035 100.33 0)
+    (property "Intersheetrefs" "${INTERSHEET_REFS}" (at 192.5721 90.17 0)
       (effects (font (size 1.27 1.27)) (justify right) (hide yes))
     )
   )
-  (global_label "ST_CAN_P" (shape input) (at 205.74 90.17 180) (fields_autoplaced)
-    (effects (font (size 1.27 1.27)) (justify right))
-    (property "Intersheetrefs" "${INTERSHEET_REFS}" (at 193.6834 90.17 0)
-      (effects (font (size 1.27 1.27)) (justify right) (hide yes))
-    )
-  )
   (hierarchical_label "TRD3{D+ D-}" (shape bidirectional) (at 261.62 87.63 0)
     (effects (font (size 1.27 1.27)) (justify left))
   )
+  (hierarchical_label "Battery_Out_3.3V" (shape output) (at 205.74 73.66 180)
+    (effects (font (size 1.27 1.27)) (justify right))
+  )
   (hierarchical_label "TRD1{D+ D-}" (shape bidirectional) (at 261.62 77.47 0)
     (effects (font (size 1.27 1.27)) (justify left))
   )
+  (hierarchical_label "Battery_Out_5V" (shape output) (at 205.74 100.33 180)
+    (effects (font (size 1.27 1.27)) (justify right))
+  )
   (hierarchical_label "TRD2{D+ D-}" (shape bidirectional) (at 261.62 82.55 0)

Commit message: Deploying to gh-pages from @ Nautilus-UUV/nautilus-mainboard-PCB@2d3890115fd9d3c0bb909c9898aa64801bed9e67 🚀
Other:
- company: (none) -> Davide, Evan
Changed lines of the file:
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@@
 (kicad_sch (version 20250114) (generator "eeschema") (generator_version "9.0")
   (paper "A4")
+  (title_block
+    (date "2025-11-18")
+    (company "Davide, Evan")
+  )
   (junction (at 242.57 115.57) (diameter 0) (color 0 0 0 0)
   )
@@
     (effects (font (size 1.27 1.27)) (justify right bottom))
   )
-  (global_label "Battery_Out_3.3V" (shape output) (at 205.74 76.2 180) (fields_autoplaced)
-    (effects (font (size 1.27 1.27)) (justify right))
-    (property "Intersheetrefs" "${INTERSHEET_REFS}" (at 186.7892 76.2 0)
-      (effects (font (size 1.27 1.27)) (justify right) (hide yes))
-    )
-  )
   (global_label "STM_TX" (shape output) (at 205.74 85.09 180) (fields_autoplaced)
     (effects (font (size 1.27 1.27)) (justify right))
@@
     (effects (font (size 1.27 1.27)) (justify left))
   )
-  (hierarchical_label "Battery_Out_3.3V" (shape output) (at 205.74 73.66 180)
+  (hierarchical_label "Battery_Out_3.3V" (shape output) (at 205.74 76.2 180)
     (effects (font (size 1.27 1.27)) (justify right))
   )

Commit message: Deploying to gh-pages from @ Nautilus-UUV/nautilus-mainboard-PCB@8b02e89ade7c168188296ba6f0516f3abec9166b 🚀
Parts:
- added LED1, LED2: 710-150060RS83000, dz_dio:Wuerth_LED_150060RS83000, symbol #dzdb:s_dio/D-WURT-710-150060RS83000
- added R16, R18: 1k, Resistor_SMD:R_0603_1608Metric, symbol #dzdb:g_res/R-1k-0603
Connections:
- net Battery_Out_3.3V: now also R16.2
- net Battery_Out_5V: now also R18.2
- net GND: now also LED1.1 (K), LED2.1 (K)
- new net: LED2.2 (A), R18.1
- new net: LED1.2 (A), R16.1
Other:
- note added: "I_{F} = 20mA V_{in} = 3.3V V_{F} ≈ 2.0V"
- note added: "I_{F} = 20mA V_{in} = 5V V_{F} ≈ 2.0V"
- note added: "R= (V_{in} - V_{F}) / I_{F}"
- note added: "So min R is 150Ω"
- note added: "So min R is 68Ω"

Commit message: Deploying to gh-pages from @ Nautilus-UUV/nautilus-mainboard-PCB@5b07cf6af03655ef9ddad269b1edd5eb03bfa75f 🚀
Parts:
- added D1: 710-82402374, Package_TO_SOT_SMD:SOT-23-5, symbol #dzdb:s_dio/WURT-710-82402374
Connections:
- net Battery_Out_3.3V: now also D1.3 (K)
- net Battery_Out_5V: now also D1.1 (K)
- net GND: now also D1.2 (A)
- net STM_RX renamed STM.RX
- net STM_TX renamed STM.TX
- net ST_CAN_N renamed ST_CAN.N
- net ST_CAN_P renamed ST_CAN.P
- no-connect marks 12 -> 14
Other:
- title: (none) -> Nautilus_Mainboard
- moved on the sheet: J7, LED1, LED2, R16, R18
