File: Browse/Power_logic.kicad_sch (KiCad schematic)
At the start: 6 parts

Commit message: Deploying to gh-pages from @ Nautilus-UUV/nautilus-mainboard-PCB@4372544f9d98c8c318df3aa79b1ddc615587ee00 🚀
Parts:
- removed Bat_3.3V_direct1, Bat_5V_direct1, Plug_3.3V_direct1, USB_5V_direct1, Vref_3.3V_CM41, Vref_3.3V_STM1: DNP, Resistor_SMD:R_0603_1608Metric, symbol #dzdb:g_res/R-0-0603
- added R34, R35, R36, R37, R38, R41, R42, R43, R44, R45, R46, R47: 0, Resistor_SMD:R_0603_1608Metric, symbol #dzdb:g_res/R-0-0603
Connections:
- net Battery_Out_3.3V: now also R44.1, R47.1
- net Battery_Out_5V: now also R35.1, R36.1
- net CM4_LED_IN_3.3V: now also R38.1, R43.1
- net GPIO_VREF_3.3V: now also R38.2, R41.2
- net STM_Plug_3.3V: now also R45.1, R46.1
- net USB_Out_5V: now also R34.1, R37.1
- new net +3.3V: R41.1, R42.1, R46.2, R47.2
- new net +5V: R34.2, R35.2
- new net 3.3V_Logic/Battery_Out_3.3V: R44.2
- new net 3.3V_Logic/STM_Plug_3.3V: R45.2
- new net 5V_Logic/Battery_Out_5V: R36.2
- new net 5V_Logic/USB_Out_5V: R37.2
- new net GPIO_REF3.3V/CM4_OUT_3.3V: R43.2
- new net GPIO_REF3.3V/STM_IN_3.3V: R42.2
Other:
- note added: "Directly connected if plug is in"
- note added: "place to activate"
- note added: "place to deactivate"
- note removed: "If STM has power, power the gyro and accelerometer"
- note removed: "LED APHHS1005LSECK/J3-PF"
- note removed: "R 1.6k"
- note removed: "Wont work... diodes are not perfect..."
- note removed: "if there is a battery connected, the LED will light up and you should not plug in your USB cable/STM connector."
- note removed: "maybe scrap this?"

Commit message: Deploying to gh-pages from @ Nautilus-UUV/nautilus-mainboard-PCB@f1dd6ce1e57c066b805694b10777c719502cca87 🚀
Parts:
- added LED10, LED9: 710-150060RS83000, dz_dio:Wuerth_LED_150060RS83000, symbol #dzdb:s_dio/D-WURT-710-150060RS83000
- added R24, R25: 1k, Resistor_SMD:R_0603_1608Metric, symbol #dzdb:g_res/R-1k-0603
Connections:
- net +3.3V: now also R24.2
- net +5V: now also R25.2
- net CM4_LED_IN_3.3V renamed CM4_Out_3.3V
- new net: LED10.2 (A), R25.1
- new net: LED9.2 (A), R24.1
- new net GND: LED10.1 (K), LED9.1 (K)
Other:
- sheet 3.3V_Logic ports: added STM_In_3.3V; removed STM_IN_3.3V
- note added: "Different Power Sources."
- note added: "I_{F} = 20mA V_{in} = 3.3V V_{F} ≈ 2.0V"
- note added: "I_{F} = 20mA V_{in} = 5V V_{F} ≈ 2.0V"
- note added: "R= (V_{in} - V_{F}) / I_{F}"
- note added: "Reference power sources"
- note added: "So min R is 150Ω"
- note added: "So min R is 68Ω"
- note added: "Whenever the CM4 runs, also run the LED signals AND the SSD voltage. all "core" tasks tied to the CM4."
- note removed: "Directly connected if plug is in"
- note removed: "Whenever the CM4 runs, also run the LED signals AND the SSD voltage. all "core" tasks tied to the CM4. If I forgot something please let me know."
- company: (none) -> Davide
- title: (none) -> Nautilus_Mainboard

Commit message: Deploying to gh-pages from @ Nautilus-UUV/nautilus-mainboard-PCB@5f5fdd9436d408a604bb268d740c0ac7ce1f5af5 🚀
Parts:
- removed LED10, LED9: 710-150060RS83000, dz_dio:Wuerth_LED_150060RS83000, symbol #dzdb:s_dio/D-WURT-710-150060RS83000
- removed R24, R25: 1k, Resistor_SMD:R_0603_1608Metric, symbol #dzdb:g_res/R-1k-0603
Connections:
- net CM4_Out_3.3V renamed CM4_LED_IN_3.3V
Other:
- sheet 3.3V_Logic ports: added STM_IN_3.3V; removed STM_In_3.3V
- note added: "Directly connected if plug is in"
- note added: "Whenever the CM4 runs, also run the LED signals AND the SSD voltage. all "core" tasks tied to the CM4. If I forgot something please let me know."
- note removed: "Different Power Sources."
- note removed: "I_{F} = 20mA V_{in} = 3.3V V_{F} ≈ 2.0V"
- note removed: "I_{F} = 20mA V_{in} = 5V V_{F} ≈ 2.0V"
- note removed: "R= (V_{in} - V_{F}) / I_{F}"
- note removed: "Reference power sources"
- note removed: "So min R is 150Ω"
- note removed: "So min R is 68Ω"
- note removed: "Whenever the CM4 runs, also run the LED signals AND the SSD voltage. all "core" tasks tied to the CM4."
- company: Davide -> (none)
- title: Nautilus_Mainboard -> (none)

Commit message: Deploying to gh-pages from @ Nautilus-UUV/nautilus-mainboard-PCB@44ad8adb17f33e1aa4439bd10449a9ac7e221a1f 🚀
Connections:
- net CM4_LED_IN_3.3V renamed CM4_OUT_3.3V
Other:
- note removed: "Directly connected if plug is in"

Commit message: Deploying to gh-pages from @ Nautilus-UUV/nautilus-mainboard-PCB@a81f7ffbfc5f9b51f47d7f388c30fcea2673b9ea 🚀
Other:
- note added: "Different Power Sources."
- note added: "Reference power sources"
- note added: "Whenever the CM4 runs, also run the LED signals AND the SSD voltage. all "core" tasks tied to the CM4."
- note removed: "Whenever the CM4 runs, also run the LED signals AND the SSD voltage. all "core" tasks tied to the CM4. If I forgot something please let me know."
- company: (none) -> dcarocci

Commit message: Deploying to gh-pages from @ Nautilus-UUV/nautilus-mainboard-PCB@2d3890115fd9d3c0bb909c9898aa64801bed9e67 🚀
Connections:
- net CM4_OUT_3.3V is gone; now on net CM4_Out_3.3V: R38.1, R43.1
Other:
- sheet 3.3V_Logic ports: added STM_In_3.3V; removed STM_IN_3.3V
- company: dcarocci -> Davide
Changed lines of the file:
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@@
   (title_block
     (date "2025-11-18")
-    (company "dcarocci")
+    (company "Davide")
   )
   (junction (at 142.24 109.22) (diameter 0) (color 0 0 0 0)
@@
     (effects (font (size 1.27 1.27)))
   )
-  (global_label "CM4_OUT_3.3V" (shape input) (at 73.66 127 180) (fields_autoplaced)
-    (effects (font (size 1.27 1.27)) (justify right))
-    (property "Intersheetrefs" "${INTERSHEET_REFS}" (at 57.0677 127 0)
-      (effects (font (size 1.27 1.27)) (justify right) (hide yes))
-    )
-  )
   (hierarchical_label "STM_Plug_3.3V" (shape input) (at 40.64 106.68 180)
     (effects (font (size 1.27 1.27)) (justify right))
@@
     (effects (font (size 1.27 1.27)) (justify right))
   )
-  (hierarchical_label "CM4_Out_3.3V" (shape input) (at 73.66 124.46 180)
+  (hierarchical_label "CM4_Out_3.3V" (shape input) (at 73.66 127 180)
     (effects (font (size 1.27 1.27)) (justify right))
   )
@@
       (effects (font (size 1.27 1.27)) (justify left top))
     )
-    (pin "Battery_Out_3.3V" output (at 119.38 85.09 180)
+    (pin "Battery_Out_3.3V" input (at 119.38 85.09 180)
       (effects (font (size 1.27 1.27)) (justify left))
     )
-    (pin "STM_IN_3.3V" output (at 149.86 87.63 0)
+    (pin "STM_Plug_3.3V" input (at 119.38 90.17 180)
+      (effects (font (size 1.27 1.27)) (justify left))
+    )
+    (pin "STM_In_3.3V" output (at 149.86 87.63 0)
       (effects (font (size 1.27 1.27)) (justify right))
-    )
-    (pin "STM_Plug_3.3V" output (at 119.38 90.17 180)
-      (effects (font (size 1.27 1.27)) (justify left))
     )
     (instances
@@
       (effects (font (size 1.27 1.27)) (justify left top))
     )
-    (pin "CM4_OUT_3.3V" output (at 119.38 127 180)
-      (effects (font (size 1.27 1.27)) (justify left))
-    )
     (pin "GPIO_VREF_3.3V" output (at 149.86 124.46 0)
       (effects (font (size 1.27 1.27)) (justify right))
     )
-    (pin "STM_IN_3.3V" output (at 119.38 121.92 180)
+    (pin "STM_IN_3.3V" input (at 119.38 121.92 180)
       (effects (font (size 1.27 1.27)) (justify left))
     )
+    (pin "CM4_OUT_3.3V" input (at 119.38 127 180)
+      (effects (font (size 1.27 1.27)) (justify left))
+    )

Commit message: Deploying to gh-pages from @ Nautilus-UUV/nautilus-mainboard-PCB@8b02e89ade7c168188296ba6f0516f3abec9166b 🚀
Changed lines of the file:
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@@
   (paper "A4")
   (title_block
-    (date "2025-11-18")
+    (date "2025-11-19")
+    (rev "1")
     (company "Davide")
   )
@@
     (effects (font (size 1.27 1.27)))
   )
-  (text "Whenever the CM4 runs, also run the LED signals AND the\nSSD voltage. all \"core\" tasks tied to the CM4." (exclude_from_sim no) (at 223.52 33.528 0)
+  (text "Whenever the CM4 runs, also run the LED signals AND the\nSSD voltage. all \"core\" tasks tied to the CM4." (exclude_from_sim no) (at 101.6 41.91 0)
     (effects (font (size 1.27 1.27)) (justify left))
   )
@@
     (effects (font (size 1.27 1.27)))
   )
-  (text "some rules:\nUSB wont power the STM32.\nSTM_Plug wont power the CM4\nThe GPIO_VREF of the CM4 needs to be STM32's 3.3V\nThe Lan Vin is only powered when running on Battery\nBattery preferrably powers everything." (exclude_from_sim no) (at 223.266 24.638 0)
+  (text "some rules:\nUSB wont power the STM32.\nSTM_Plug wont power the CM4\nThe GPIO_VREF of the CM4 needs to be STM32's 3.3V\nThe Lan Vin is only powered when running on Battery\nBattery preferrably powers everything." (exclude_from_sim no) (at 101.346 33.02 0)
     (effects (font (size 1.27 1.27)) (justify left))
   )

Commit message: Deploying to gh-pages from @ Nautilus-UUV/nautilus-mainboard-PCB@5b07cf6af03655ef9ddad269b1edd5eb03bfa75f 🚀
Parts:
- added LED10, LED9: 710-150060RS83000, dz_dio:Wuerth_LED_150060RS83000, symbol #dzdb:s_dio/D-WURT-710-150060RS83000
- added R24, R25: 1k, Resistor_SMD:R_0603_1608Metric, symbol #dzdb:g_res/R-1k-0603
Connections:
- net +3.3V: now also R24.2
- net +5V: now also R25.2
- new net: LED10.2 (A), R25.1
- new net: LED9.2 (A), R24.1
- new net GND: LED10.1 (K), LED9.1 (K)
Other:
- note added: "I_{F} = 20mA V_{in} = 3.3V V_{F} ≈ 2.0V"
- note added: "I_{F} = 20mA V_{in} = 5V V_{F} ≈ 2.0V"
- note added: "R= (V_{in} - V_{F}) / I_{F}"
- note added: "So min R is 150Ω"
- note added: "So min R is 68Ω"
- title: (none) -> Nautilus_Mainboard
