File: Browse/Power_logic.kicad_sch (KiCad schematic)
At the start: 16 parts

Commit message: Deploying to gh-pages from @ Nautilus-UUV/nautilus-mainboard-PCB@7cbe43864a66a110f5cd8f57d0dac694c5d0b0c8 🚀
Parts:
- removed R34, R35, R36, R37, R38, R41, R42, R43, R44, R45, R46, R47: 0, Resistor_SMD:R_0603_1608Metric, symbol #dzdb:g_res/R-0-0603
- added JP1, JP10, JP11, JP12, JP2, JP3, JP4, JP5, JP6, JP7, JP8, JP9: -, Jumper:SolderJumper-2_P1.3mm_Open_RoundedPad1.0x1.5mm, symbol #dzdb:g_mech/Jumper-2P1.3mm_Rounded
Connections:
- net +3.3V: now also JP2.1 (A), JP3.2 (B), JP4.2 (B), JP9.1 (A)
- net +5V: now also JP5.2 (B), JP6.2 (B)
- net 3.3V_Logic/Battery_Out_3.3V: now also JP11.2 (B)
- net 3.3V_Logic/STM_Plug_3.3V: now also JP12.2 (B)
- net 5V_Logic/Battery_Out_5V: now also JP7.2 (B)
- net 5V_Logic/USB_Out_5V: now also JP8.2 (B)
- net Battery_Out_3.3V: now also JP11.1 (A), JP4.1 (A)
- net Battery_Out_5V: now also JP6.1 (A), JP7.1 (A)
- net CM4_Out_3.3V: now also JP1.1 (A), JP10.1 (A)
- net GPIO_REF3.3V/CM4_OUT_3.3V: now also JP10.2 (B)
- net GPIO_REF3.3V/STM_IN_3.3V: now also JP9.2 (B)
- net GPIO_VREF_3.3V: now also JP1.2 (B), JP2.2 (B)
- net STM_Plug_3.3V: now also JP12.1 (A), JP3.1 (A)
- net USB_Out_5V: now also JP5.1 (A), JP8.1 (A)

Commit message: Deploying to gh-pages from @ Nautilus-UUV/nautilus-mainboard-PCB@b731ca7531dd1e48b6b7a45790de08634e79c176 🚀
Changed lines of the file:
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@@
       (effects (font (size 1.27 1.27)))
     )
-    (property "Value" "-" (at 133.35 76.962 0)
+    (property "Value" "-" (at 133.35 69.85 0)
       (effects (font (size 1.27 1.27)))
     )
@@
       (effects (font (size 1.27 1.27)))
     )
-    (property "Value" "-" (at 133.35 69.85 0)
-      (effects (font (size 1.27 1.27)))
-    )
+    (property "Value" "-" (at 133.35 74.93 0)
+      (effects (font (size 1.27 1.27)))
+    )
