File: Browse/nautilus_mainboard.kicad_sch (KiCad schematic)
At the start: 0 parts

Commit message: Deploying to gh-pages from @ Nautilus-UUV/nautilus-mainboard-PCB@400426d46daeee198d0eea8645f966723a05ffff 🚀
Parts:
- added TP2, TP3: TestPoint_Probe, TestPoint:TestPoint_THTPad_D2.5mm_Drill1.2mm, symbol Connector:TestPoint_Probe
- added TP4, TP5: TestPoint_Probe, TestPoint:TestPoint_Pad_D1.0mm, symbol Connector:TestPoint_Probe
Connections:
- net CM4/PI_RX: now also TP4.1
- net CM4/PI_TX: now also TP5.1
- net IMU/Pack1_SCL: now also TP3.1
- net IMU/Pack1_SDA: now also TP2.1
Changed lines of the file:
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@@
 (kicad_sch (version 20250114) (generator "eeschema") (generator_version "9.0")
   (paper "A4")
+  (junction (at 78.74 52.07) (diameter 0) (color 0 0 0 0)
+  )
+  (junction (at 80.01 45.72) (diameter 0) (color 0 0 0 0)
+  )
+  (junction (at 83.82 90.17) (diameter 0) (color 0 0 0 0)
+  )
+  (junction (at 83.82 87.63) (diameter 0) (color 0 0 0 0)
+  )
   (wire (pts (xy 134.62 76.2) (xy 134.62 92.71))
     (stroke (width 0) (type default))
@@
     (stroke (width 0) (type default))
   )
-  (wire (pts (xy 76.2 45.72) (xy 101.6 45.72))
+  (wire (pts (xy 121.92 76.2) (xy 121.92 92.71))
     (stroke (width 0) (type default))
   )
-  (wire (pts (xy 121.92 76.2) (xy 121.92 92.71))
+  (wire (pts (xy 76.2 45.72) (xy 80.01 45.72))
     (stroke (width 0) (type default))
   )
@@
     (stroke (width 0) (type default))
   )
+  (wire (pts (xy 76.2 52.07) (xy 78.74 52.07))
+    (stroke (width 0) (type default))
+  )
   (wire (pts (xy 184.15 93.98) (xy 184.15 90.17))
     (stroke (width 0) (type default))
   )
-  (wire (pts (xy 184.15 90.17) (xy 55.88 90.17))
+  (wire (pts (xy 78.74 52.07) (xy 101.6 52.07))
+    (stroke (width 0) (type default))
+  )
+  (wire (pts (xy 55.88 90.17) (xy 83.82 90.17))
     (stroke (width 0) (type default))
   )
   (wire (pts (xy 76.2 59.69) (xy 101.6 59.69))
-    (stroke (width 0) (type default))
-  )
-  (wire (pts (xy 76.2 52.07) (xy 101.6 52.07))
     (stroke (width 0) (type default))
   )
@@
     (stroke (width 0) (type default))
   )
-  (wire (pts (xy 186.69 87.63) (xy 59.69 87.63))
+  (wire (pts (xy 186.69 87.63) (xy 83.82 87.63))
+    (stroke (width 0) (type default))
+  )
+  (wire (pts (xy 83.82 90.17) (xy 184.15 90.17))
     (stroke (width 0) (type default))
   )
@@
     (stroke (width 0) (type default))
   )
+  (wire (pts (xy 83.82 87.63) (xy 59.69 87.63))
+    (stroke (width 0) (type default))
+  )
   (wire (pts (xy 186.69 93.98) (xy 186.69 87.63))
+    (stroke (width 0) (type default))
+  )
+  (wire (pts (xy 80.01 45.72) (xy 101.6 45.72))
     (stroke (width 0) (type default))
   )
@@
     (effects (font (size 2 2) (thickness 0.4) (bold yes) (color 44 31 255 1)) (justify left))
   )
+  (symbol (lib_id "Connector:TestPoint_Probe") (at 80.01 45.72 0) (unit 1)
+    (exclude_from_sim no) (in_bom yes) (on_board yes) (dnp no) (fields_autoplaced)
+    (property "Reference" "TP4" (at 83.82 42.8624 0)
+      (effects (font (size 1.27 1.27)) (justify left))
+    )
+    (property "Value" "TestPoint_Probe" (at 83.82 45.4024 0)
+      (effects (font (size 1.27 1.27)) (justify left))
+    )
+    (property "Footprint" "TestPoint:TestPoint_Pad_D1.0mm" (at 85.09 45.72 0)
+      (effects (font (size 1.27 1.27)) (hide yes))
+    )
+    (property "Datasheet" "~" (at 85.09 45.72 0)
+      (effects (font (size 1.27 1.27)) (hide yes))
+    )
+    (property "Description" "test point (alternative probe-style design)" (at 80.01 45.72 0)
+      (effects (font (size 1.27 1.27)) (hide yes))
+    )
+    (pin "1")
+    (instances
+      (project "nautilus_mainboard"
+        (path "/ce1819b2-f280-40ed-834f-6fe4d12f809d"
+          (reference "TP4") (unit 1)
+        )
+      )
+    )
+  )
+  (symbol (lib_id "Connector:TestPoint_Probe") (at 83.82 87.63 0) (unit 1)
+    (exclude_from_sim no) (in_bom yes) (on_board yes) (dnp no) (fields_autoplaced)
+    (property "Reference" "TP2" (at 87.63 84.7724 0)
+      (effects (font (size 1.27 1.27)) (justify left))
+    )
+    (property "Value" "TestPoint_Probe" (at 87.63 87.3124 0)
+      (effects (font (size 1.27 1.27)) (justify left))
+    )
+    (property "Footprint" "TestPoint:TestPoint_THTPad_D2.5mm_Drill1.2mm" (at 88.9 87.63 0)
+      (effects (font (size 1.27 1.27)) (hide yes))
+    )
+    (property "Datasheet" "~" (at 88.9 87.63 0)
+      (effects (font (size 1.27 1.27)) (hide yes))
+    )
+    (property "Description" "test point (alternative probe-style design)" (at 83.82 87.63 0)
+      (effects (font (size 1.27 1.27)) (hide yes))
+    )
+    (pin "1")
+    (instances
+      (project ""
+        (path "/ce1819b2-f280-40ed-834f-6fe4d12f809d"
+          (reference "TP2") (unit 1)
+        )
+      )
+    )
+  )
+  (symbol (lib_id "Connector:TestPoint_Probe") (at 83.82 90.17 0) (unit 1)
+    (exclude_from_sim no) (in_bom yes) (on_board yes) (dnp no) (fields_autoplaced)
+    (property "Reference" "TP3" (at 87.63 87.3124 0)
+      (effects (font (size 1.27 1.27)) (justify left))
+    )
+    (property "Value" "TestPoint_Probe" (at 87.63 89.8524 0)
+      (effects (font (size 1.27 1.27)) (justify left))
+    )
+    (property "Footprint" "TestPoint:TestPoint_THTPad_D2.5mm_Drill1.2mm" (at 88.9 90.17 0)
+      (effects (font (size 1.27 1.27)) (hide yes))
+    )
+    (property "Datasheet" "~" (at 88.9 90.17 0)
+      (effects (font (size 1.27 1.27)) (hide yes))
+    )
+    (property "Description" "test point (alternative probe-style design)" (at 83.82 90.17 0)
+      (effects (font (size 1.27 1.27)) (hide yes))
+    )
+    (pin "1")
+    (instances
+      (project "nautilus_mainboard"
+        (path "/ce1819b2-f280-40ed-834f-6fe4d12f809d"
+          (reference "TP3") (unit 1)
+        )
+      )
+    )
+  )
+  (symbol (lib_id "Connector:TestPoint_Probe") (at 78.74 52.07 0) (unit 1)
+    (exclude_from_sim no) (in_bom yes) (on_board yes) (dnp no) (fields_autoplaced)
+    (property "Reference" "TP5" (at 82.55 49.2124 0)
+      (effects (font (size 1.27 1.27)) (justify left))
+    )
+    (property "Value" "TestPoint_Probe" (at 82.55 51.7524 0)
+      (effects (font (size 1.27 1.27)) (justify left))
+    )
+    (property "Footprint" "TestPoint:TestPoint_Pad_D1.0mm" (at 83.82 52.07 0)
+      (effects (font (size 1.27 1.27)) (hide yes))
+    )
+    (property "Datasheet" "~" (at 83.82 52.07 0)
+      (effects (font (size 1.27 1.27)) (hide yes))
+    )
+    (property "Description" "test point (alternative probe-style design)" (at 78.74 52.07 0)
+      (effects (font (size 1.27 1.27)) (hide yes))
+    )
+    (pin "1")
+    (instances
+      (project "nautilus_mainboard"
+        (path "/ce1819b2-f280-40ed-834f-6fe4d12f809d"
+          (reference "TP5") (unit 1)
+        )
+      )
+    )
+  )
   (sheet (at 25.4 25.4) (size 50.8 50.8) (exclude_from_sim no) (in_bom yes) (on_board yes) (dnp no) (fields_autoplaced)

Commit message: Deploying to gh-pages from @ Nautilus-UUV/nautilus-mainboard-PCB@b62834b88bb3e2a9413bcb4ea8e223af403e20ba 🚀
Other:
- sheet CM4 ports: added TRD0{D+ D-}, TRD1{D+ D-}, TRD2{D+ D-}, TRD3{D+ D-}; removed ET1, ET2, ET3, ET4, ET5, ET6, ET7, ET8
- sheet LPHS-connector ports: added TRD0{D+ D-}, TRD1{D+ D-}, TRD2{D+ D-}, TRD3{D+ D-}; removed ET1, ET2, ET3, ET4, ET5, ET6, ET7, ET8
Changed lines of the file:
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@@
   (junction (at 83.82 87.63) (diameter 0) (color 0 0 0 0)
   )
-  (wire (pts (xy 134.62 76.2) (xy 134.62 92.71))
-    (stroke (width 0) (type default))
-  )
-  (wire (pts (xy 129.54 76.2) (xy 129.54 92.71))
-    (stroke (width 0) (type default))
-  )
-  (wire (pts (xy 121.92 76.2) (xy 121.92 92.71))
+  (bus (pts (xy 132.08 76.2) (xy 132.08 92.71))
+    (stroke (width 0) (type default))
+  )
+  (bus (pts (xy 127 76.2) (xy 127 92.71))
     (stroke (width 0) (type default))
   )
@@
     (stroke (width 0) (type default))
   )
-  (wire (pts (xy 127 76.2) (xy 127 92.71))
-    (stroke (width 0) (type default))
-  )
   (wire (pts (xy 76.2 52.07) (xy 78.74 52.07))
     (stroke (width 0) (type default))
@@
     (stroke (width 0) (type default))
   )
-  (wire (pts (xy 132.08 76.2) (xy 132.08 92.71))
-    (stroke (width 0) (type default))
-  )
-  (wire (pts (xy 139.7 76.2) (xy 139.7 92.71))
+  (bus (pts (xy 116.84 76.2) (xy 116.84 92.71))
     (stroke (width 0) (type default))
   )
@@
     (stroke (width 0) (type default))
   )
-  (wire (pts (xy 137.16 76.2) (xy 137.16 92.71))
+  (bus (pts (xy 121.92 76.2) (xy 121.92 92.71))
     (stroke (width 0) (type default))
   )
@@
   )
   (wire (pts (xy 76.2 40.64) (xy 101.6 40.64))
-    (stroke (width 0) (type default))
-  )
-  (wire (pts (xy 124.46 76.2) (xy 124.46 92.71))
     (stroke (width 0) (type default))
   )
@@
       (effects (font (size 1.27 1.27)) (justify left top))
     )
-    (pin "ET1" input (at 121.92 92.71 90)
-      (effects (font (size 1.27 1.27)) (justify right))
-    )
-    (pin "ET2" input (at 124.46 92.71 90)
-      (effects (font (size 1.27 1.27)) (justify right))
-    )
-    (pin "ET3" input (at 127 92.71 90)
-      (effects (font (size 1.27 1.27)) (justify right))
-    )
-    (pin "ET4" input (at 129.54 92.71 90)
-      (effects (font (size 1.27 1.27)) (justify right))
-    )
-    (pin "ET5" input (at 132.08 92.71 90)
-      (effects (font (size 1.27 1.27)) (justify right))
-    )
-    (pin "ET6" input (at 134.62 92.71 90)
-      (effects (font (size 1.27 1.27)) (justify right))
-    )
-    (pin "ET7" input (at 137.16 92.71 90)
-      (effects (font (size 1.27 1.27)) (justify right))
-    )
-    (pin "ET8" input (at 139.7 92.71 90)
+    (pin "TRD0{D+ D-}" bidirectional (at 116.84 92.71 90)
+      (effects (font (size 1.27 1.27)) (justify right))
+    )
+    (pin "TRD1{D+ D-}" bidirectional (at 121.92 92.71 90)
+      (effects (font (size 1.27 1.27)) (justify right))
+    )
+    (pin "TRD2{D+ D-}" bidirectional (at 127 92.71 90)
+      (effects (font (size 1.27 1.27)) (justify right))
+    )
+    (pin "TRD3{D+ D-}" bidirectional (at 132.08 92.71 90)
       (effects (font (size 1.27 1.27)) (justify right))
     )
@@
       (effects (font (size 1.27 1.27)) (justify left top))
     )
-    (pin "ET1" input (at 121.92 76.2 270)
-      (effects (font (size 1.27 1.27)) (justify left))
-    )
-    (pin "ET2" input (at 124.46 76.2 270)
-      (effects (font (size 1.27 1.27)) (justify left))
-    )
-    (pin "ET3" input (at 127 76.2 270)
-      (effects (font (size 1.27 1.27)) (justify left))
-    )
-    (pin "ET4" input (at 129.54 76.2 270)
-      (effects (font (size 1.27 1.27)) (justify left))
-    )
-    (pin "ET5" input (at 132.08 76.2 270)
-      (effects (font (size 1.27 1.27)) (justify left))
-    )
-    (pin "ET6" input (at 134.62 76.2 270)
-      (effects (font (size 1.27 1.27)) (justify left))
-    )
-    (pin "ET7" input (at 137.16 76.2 270)
-      (effects (font (size 1.27 1.27)) (justify left))
-    )
-    (pin "ET8" input (at 139.7 76.2 270)
-      (effects (font (size 1.27 1.27)) (justify left))
-    )
     (pin "PI_RX" input (at 101.6 45.72 180)
       (effects (font (size 1.27 1.27)) (justify left))
@@
       (effects (font (size 1.27 1.27)) (justify left))
     )
+    (pin "TRD0{D+ D-}" bidirectional (at 116.84 76.2 270)
+      (effects (font (size 1.27 1.27)) (justify left))
+    )
+    (pin "TRD1{D+ D-}" bidirectional (at 121.92 76.2 270)
+      (effects (font (size 1.27 1.27)) (justify left))
+    )
+    (pin "TRD2{D+ D-}" bidirectional (at 127 76.2 270)
+      (effects (font (size 1.27 1.27)) (justify left))
+    )
+    (pin "TRD3{D+ D-}" bidirectional (at 132.08 76.2 270)
+      (effects (font (size 1.27 1.27)) (justify left))
+    )

Commit message: Deploying to gh-pages from @ Nautilus-UUV/nautilus-mainboard-PCB@44ad8adb17f33e1aa4439bd10449a9ac7e221a1f 🚀
Other:
- sheet CM4 ports: added GPIO_VREF_3.3V; removed none
- sheet Power_logic ports: added GPIO_VREF_3.3V; removed none
- moved on the sheet: TP2, TP3

Commit message: Deploying to gh-pages from @ Nautilus-UUV/nautilus-mainboard-PCB@a81f7ffbfc5f9b51f47d7f388c30fcea2673b9ea 🚀
Parts:
- added TP1, TP8, TP9: TestPoint_Probe, TestPoint:TestPoint_Pad_D1.0mm, symbol Connector:TestPoint_Probe
Connections:
- new net CM4/Battery_Out_3.3V: TP8.1
- new net GND: TP9.1
- new net LPHS-connector/Battery_Out_5V: TP1.1
Other:
- sheet CM4 ports: added Battery_Out_3.3V, CM4_Out_3.3V, LAN_IN_3.3V, USB_Out_5V; removed none
- sheet LPHS-connector ports: added Battery_Out_3.3V, Battery_Out_5V; removed none
- sheet Piezzo ports: added Piezo_ctrl; removed none
- sheet Power_logic ports: added Battery_Out_3.3V, Battery_Out_5V, CM4_Out_3.3V, LAN_IN_3.3V, STM_Plug_3.3V, USB_Out_5V; removed none
- sheet STM ports: added Battery_Out_3.3V, STM_Plug_3.3V; removed none
- note added: "Standard 5V and 3.3V for the components are sent out as globals."
- moved on the sheet: TP2, TP3, TP4, TP5

Commit message: Deploying to gh-pages from @ Nautilus-UUV/nautilus-mainboard-PCB@2d3890115fd9d3c0bb909c9898aa64801bed9e67 🚀
Other:
- sheet STM ports: added Piezzo_Control; removed none
- note removed: "We should consider that we NEVER want the CM4 to power the unpowered STM over the TX pin. Found a neat part for that: https://www.mouser.ch/ProductDetail/Texas-Instruments/SN74LVC1G126DBVR?qs=pajgIaoyDUi3T2WgNNfd3w%3D%3D connections: Pin 5: VCC -> CM4_3V3 Pin 2: A -> CM4 TX (PLTX) Pin 4: Y -> STM_UART_RX Pin 1: OE -> STM_IN_3.3V Pin 3: GND 0.1uF decoupling cap VCC-GND 220 Ohm series at Y (to STM)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"
- company: (none) -> Evan & Davide
Changed lines of the file:
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@@
 (kicad_sch (version 20250114) (generator "eeschema") (generator_version "9.0")
   (paper "A4")
+  (title_block
+    (date "2025-11-18")
+    (company "Evan & Davide")
+  )
   (junction (at 78.74 44.45) (diameter 0) (color 0 0 0 0)
   )
@@
     (stroke (width 0) (type default))
   )
+  (wire (pts (xy 92.71 154.94) (xy 92.71 59.69))
+    (stroke (width 0) (type default))
+  )
   (wire (pts (xy 163.83 81.28) (xy 163.83 113.03))
     (stroke (width 0) (type default))
@@
     (stroke (width 0) (type default))
   )
-  (wire (pts (xy 95.25 59.69) (xy 95.25 85.09))
-    (stroke (width 0) (type default))
-  )
-  (wire (pts (xy 76.2 59.69) (xy 95.25 59.69))
+  (wire (pts (xy 95.25 57.15) (xy 95.25 85.09))
+    (stroke (width 0) (type default))
+  )
+  (wire (pts (xy 76.2 57.15) (xy 95.25 57.15))
+    (stroke (width 0) (type default))
+  )
+  (wire (pts (xy 165.1 140.97) (xy 165.1 154.94))
     (stroke (width 0) (type default))
   )
@@
     (stroke (width 0) (type default))
   )
+  (wire (pts (xy 165.1 154.94) (xy 92.71 154.94))
+    (stroke (width 0) (type default))
+  )
   (wire (pts (xy 152.4 52.07) (xy 177.8 52.07))
     (stroke (width 0) (type default))
@@
     (stroke (width 0) (type default))
   )
+  (wire (pts (xy 176.53 140.97) (xy 165.1 140.97))
+    (stroke (width 0) (type default))
+  )
   (wire (pts (xy 177.8 60.96) (xy 163.83 60.96))
     (stroke (width 0) (type default))
@@
     (stroke (width 0) (type default))
   )
-  (text "We should consider that we NEVER want the CM4 to power the unpowered STM\nover the TX pin. Found a neat part for that:\nhttps://www.mouser.ch/ProductDetail/Texas-Instruments/SN74LVC1G126DBVR?qs=pajgIaoyDUi3T2WgNNfd3w%3D%3D\n\nconnections:\nPin 5: VCC -> CM4_3V3\n\nPin 2: A -> CM4 TX (PLTX)\n\nPin 4: Y -> STM_UART_RX\n\nPin 1: OE -> STM_IN_3.3V\n\nPin 3: GND\n\n0.1uF decoupling cap VCC-GND\n\n220 Ohm series at Y (to STM). (current limiting)\n\n100 kOhm pull-down from OE to GND" (exclude_from_sim no) (at 74.422 180.848 0)
-    (effects (font (size 2 2) (thickness 0.4) (bold yes) (color 44 31 255 1)) (justify left))
+  (wire (pts (xy 76.2 59.69) (xy 92.71 59.69))
+    (stroke (width 0) (type default))
   )
   (text "Standard 5V and 3.3V for the components are sent out as globals." (exclude_from_sim no) (at 203.962 20.32 0)
@@
       (effects (font (size 1.27 1.27)) (justify right))
     )
-    (pin "Battery_Out_3.3V" input (at 76.2 59.69 0)
+    (pin "Battery_Out_3.3V" input (at 76.2 57.15 0)
+      (effects (font (size 1.27 1.27)) (justify right))
+    )
+    (pin "Piezzo_Control" output (at 76.2 59.69 0)
       (effects (font (size 1.27 1.27)) (justify right))
     )
@@
       (effects (font (size 1.27 1.27)) (justify left top))
     )
-    (pin "Piezo_ctrl" input (at 186.69 93.98 90)
-      (effects (font (size 1.27 1.27)) (justify right))
-    )
-    (instances
+    (pin "Piezo_ctrl" input (at 176.53 140.97 180)
+      (effects (font (size 1.27 1.27)) (justify left))
+    )
+    (instances

Commit message: Deploying to gh-pages from @ Nautilus-UUV/nautilus-mainboard-PCB@8b02e89ade7c168188296ba6f0516f3abec9166b 🚀
Parts:
- added TP10, TP11, TP12: TestPoint_Probe, TestPoint:TestPoint_Pad_D1.0mm, symbol Connector:TestPoint_Probe
Connections:
- net GND: now also TP10.1, TP11.1, TP12.1
Changed lines of the file:
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@@
   (paper "A4")
   (title_block
-    (date "2025-11-18")
+    (date "2025-11-19")
+    (rev "0")
     (company "Evan & Davide")
   )
@@
     (effects (font (size 1.27 1.27)))
   )
+  (symbol (lib_id "power:GND") (at 236.22 93.98 0) (unit 1)
+    (exclude_from_sim no) (in_bom yes) (on_board yes) (dnp no) (fields_autoplaced)
+    (property "Reference" "#PWR061" (at 236.22 100.33 0)
+      (effects (font (size 1.27 1.27)) (hide yes))
+    )
+    (property "Value" "GND" (at 236.22 99.06 0)
+      (effects (font (size 1.27 1.27)))
+    )
+    (property "Footprint" "" (at 236.22 93.98 0)
+      (effects (font (size 1.27 1.27)) (hide yes))
+    )
+    (property "Datasheet" "" (at 236.22 93.98 0)
+      (effects (font (size 1.27 1.27)) (hide yes))
+    )
+    (property "Description" "Power symbol creates a global label with name \"GND\" , ground" (at 236.22 93.98 0)
+      (effects (font (size 1.27 1.27)) (hide yes))
+    )
+    (pin "1")
+    (instances
+      (project "nautilus_mainboard"
+        (path "/ce1819b2-f280-40ed-834f-6fe4d12f809d"
+          (reference "#PWR061") (unit 1)
+        )
+      )
+    )
+  )
   (symbol (lib_id "Connector:TestPoint_Probe") (at 80.01 38.1 0) (unit 1)
     (exclude_from_sim no) (in_bom yes) (on_board yes) (dnp no)
@@
         (path "/ce1819b2-f280-40ed-834f-6fe4d12f809d"
           (reference "TP4") (unit 1)
+        )
+      )
+    )
+  )
+  (symbol (lib_id "power:GND") (at 256.54 82.55 0) (unit 1)
+    (exclude_from_sim no) (in_bom yes) (on_board yes) (dnp no) (fields_autoplaced)
+    (property "Reference" "#PWR017" (at 256.54 88.9 0)
+      (effects (font (size 1.27 1.27)) (hide yes))
+    )
+    (property "Value" "GND" (at 256.54 87.63 0)
+      (effects (font (size 1.27 1.27)))
+    )
+    (property "Footprint" "" (at 256.54 82.55 0)
+      (effects (font (size 1.27 1.27)) (hide yes))
+    )
+    (property "Datasheet" "" (at 256.54 82.55 0)
+      (effects (font (size 1.27 1.27)) (hide yes))
+    )
+    (property "Description" "Power symbol creates a global label with name \"GND\" , ground" (at 256.54 82.55 0)
+      (effects (font (size 1.27 1.27)) (hide yes))
+    )
+    (pin "1")
+    (instances
+      (project "nautilus_mainboard"
+        (path "/ce1819b2-f280-40ed-834f-6fe4d12f809d"
+          (reference "#PWR017") (unit 1)
+        )
+      )
+    )
+  )
+  (symbol (lib_id "Connector:TestPoint_Probe") (at 256.54 93.98 0) (unit 1)
+    (exclude_from_sim no) (in_bom yes) (on_board yes) (dnp no)
+    (property "Reference" "TP12" (at 260.096 90.17 0)
+      (effects (font (size 1.27 1.27)) (justify left))
+    )
+    (property "Value" "TestPoint_Probe" (at 260.096 92.71 0)
+      (effects (font (size 1.27 1.27)) (justify left))
+    )
+    (property "Footprint" "TestPoint:TestPoint_Pad_D1.0mm" (at 261.62 93.98 0)
+      (effects (font (size 1.27 1.27)) (hide yes))
+    )
+    (property "Datasheet" "~" (at 261.62 93.98 0)
+      (effects (font (size 1.27 1.27)) (hide yes))
+    )
+    (property "Description" "test point (alternative probe-style design)" (at 256.54 93.98 0)
+      (effects (font (size 1.27 1.27)) (hide yes))
+    )
+    (pin "1")
+    (instances
+      (project "nautilus_mainboard"
+        (path "/ce1819b2-f280-40ed-834f-6fe4d12f809d"
+          (reference "TP12") (unit 1)
+        )
+      )
+    )
+  )
+  (symbol (lib_id "power:GND") (at 256.54 93.98 0) (unit 1)
+    (exclude_from_sim no) (in_bom yes) (on_board yes) (dnp no) (fields_autoplaced)
+    (property "Reference" "#PWR062" (at 256.54 100.33 0)
+      (effects (font (size 1.27 1.27)) (hide yes))
+    )
+    (property "Value" "GND" (at 256.54 99.06 0)
+      (effects (font (size 1.27 1.27)))
+    )
+    (property "Footprint" "" (at 256.54 93.98 0)
+      (effects (font (size 1.27 1.27)) (hide yes))
+    )
+    (property "Datasheet" "" (at 256.54 93.98 0)
+      (effects (font (size 1.27 1.27)) (hide yes))
+    )
+    (property "Description" "Power symbol creates a global label with name \"GND\" , ground" (at 256.54 93.98 0)
+      (effects (font (size 1.27 1.27)) (hide yes))
+    )
+    (pin "1")
+    (instances
+      (project "nautilus_mainboard"
+        (path "/ce1819b2-f280-40ed-834f-6fe4d12f809d"
+          (reference "#PWR062") (unit 1)
         )
       )
@@
     )
   )
+  (symbol (lib_id "Connector:TestPoint_Probe") (at 256.54 82.55 0) (unit 1)
+    (exclude_from_sim no) (in_bom yes) (on_board yes) (dnp no)
+    (property "Reference" "TP10" (at 260.096 78.74 0)
+      (effects (font (size 1.27 1.27)) (justify left))
+    )
+    (property "Value" "TestPoint_Probe" (at 260.096 81.28 0)
+      (effects (font (size 1.27 1.27)) (justify left))
+    )
+    (property "Footprint" "TestPoint:TestPoint_Pad_D1.0mm" (at 261.62 82.55 0)
+      (effects (font (size 1.27 1.27)) (hide yes))
+    )
+    (property "Datasheet" "~" (at 261.62 82.55 0)
+      (effects (font (size 1.27 1.27)) (hide yes))
+    )
+    (property "Description" "test point (alternative probe-style design)" (at 256.54 82.55 0)
+      (effects (font (size 1.27 1.27)) (hide yes))
+    )
+    (pin "1")
+    (instances
+      (project "nautilus_mainboard"
+        (path "/ce1819b2-f280-40ed-834f-6fe4d12f809d"
+          (reference "TP10") (unit 1)
+        )
+      )
+    )
+  )
   (symbol (lib_id "Connector:TestPoint_Probe") (at 49.53 86.36 0) (unit 1)
     (exclude_from_sim no) (in_bom yes) (on_board yes) (dnp no) (fields_autoplaced)
@@
         )
       )
+    )
+  )
+  (symbol (lib_id "Connector:TestPoint_Probe") (at 236.22 93.98 0) (unit 1)
+    (exclude_from_sim no) (in_bom yes) (on_board yes) (dnp no)
+    (property "Reference" "TP11" (at 239.776 90.17 0)
+      (effects (font (size 1.27 1.27)) (justify left))
+    )
+    (property "Value" "TestPoint_Probe" (at 239.776 92.71 0)
+      (effects (font (size 1.27 1.27)) (justify left))
+    )
+    (property "Footprint" "TestPoint:TestPoint_Pad_D1.0mm" (at 241.3 93.98 0)
+      (effects (font (size 1.27 1.27)) (hide yes))
+    )
+    (property "Datasheet" "~" (at 241.3 93.98 0)
+      (effects (font (size 1.27 1.27)) (hide yes))
+    )
+    (property "Description" "test point (alternative probe-style design)" (at 236.22 93.98 0)
+      (effects (font (size 1.27 1.27)) (hide yes))
+    )
+    (pin "1")
+    (instances
+      (project "nautilus_mainboard"
+        (path "/ce1819b2-f280-40ed-834f-6fe4d12f809d"
+          (reference "TP11") (unit 1)
+        )
+      )
