File: Browse/nautilus_mainboard.kicad_sch (KiCad schematic)
At the start: 12 parts

Commit message: Deploying to gh-pages from @ Nautilus-UUV/nautilus-mainboard-PCB@2b5265db7706a31505c0a0411337a4a604b5fb21 🚀
Changed lines of the file:
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@@
     (stroke (width 0) (type default))
+  )
+  (text_box "20.11.2025\nSwitched R18 from 1k to 2.2k for equal led strength\n\n+ Added more routing in PCB."
+    (exclude_from_sim no) (at 93.98 147.32 0) (size 58.42 50.8)
+    (margins 0.9525 0.9525 0.9525 0.9525) (stroke (width 0) (type solid))
+    (fill (type none))
+    (effects (font (size 1.27 1.27)) (justify left top))
   )
   (text_box "Changelog:\n\n+ Added Bus where it seems reasonable.\n+ Added unified LED symbol (Red power, Yellow data)\n+ Added Buzzer logic and Buzzer\n+ Added Sheet titles, Authors, Date, Revision\n+ Added ESD protection on all Plugs (not sure if 3.3V is correct like that)\n\n- Removed Overengineered Power distribution system\n+ Implemented simpler Power distribution system\n- Reduced Globals to a minimum, used +3.3V and +5V for voltage of parts\n+ Introduced a lot of TestPoints with symbol that catches the eye fast.\n\n* Redesigned some Symbols\n* Cleaned up rubbish and wiring sphagetti\n\n- Removed PCB for new layout. (WIP)\n\nNotes:\n-> Fan not yet updated, still a screw terminal.\n-> Piezzo randomly connected to an STM Pin. Evan should check this.\n-> PCB in the making.\nIssue: Footprint and Model for SSD holder not present anymore @evan\n"

Commit message: Deploying to gh-pages from @ Nautilus-UUV/nautilus-mainboard-PCB@e232027359a390dc54348e0f0abbe6a5df208f5c 🚀
Parts:
- removed TP1, TP10, TP11, TP12, TP13, TP14, TP4, TP5, TP8, TP9: TestPoint_Probe, TestPoint:TestPoint_Pad_D1.0mm, symbol Connector:TestPoint_Probe
- removed TP2, TP3: TestPoint_Probe, TestPoint:TestPoint_THTPad_D2.5mm_Drill1.2mm, symbol Connector:TestPoint_Probe
- added TP1, TP10, TP11, TP12, TP15, TP16, TP2, TP3, TP4, TP5, TP8, TP9: Test Point, TestPoint:TestPoint_Pad_D1.5mm, symbol #dzdb:g_mech/M-TEST-SMT_1.5mm_round
Connections:
- net +3.3V: now also TP5.1
- net +5V: now also TP8.1
- net CM4/Battery_Out_3.3V: now also TP15.1
- net CM4/PI_RX: now also TP4.1
- net CM4/PI_TX: now also TP3.1
- net GND: now also TP10.1, TP12.1, TP9.1
- net IMU/Pack1_SCL: now also TP2.1
- net IMU/Pack1_SDA: now also TP1.1
- net LPHS-connector/Battery_Out_5V: now also TP16.1

Commit message: Deploying to gh-pages from @ Nautilus-UUV/nautilus-mainboard-PCB@62d9beca31554f779583bfc3c938b3f82a581309 🚀
Connections:
- net GND: now also TP11.1
Other:
- moved on the sheet: TP11
Changed lines of the file:
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@@
     )
   )
-  (symbol (lib_id "#dzdb:g_mech/M-TEST-SMT_1.5mm_round") (at 236.22 92.71 0) (unit 1)
+  (symbol (lib_id "#dzdb:g_mech/M-TEST-SMT_1.5mm_round") (at 236.22 93.98 0) (unit 1)
     (exclude_from_sim no) (in_bom yes) (on_board yes) (dnp no) (fields_autoplaced)
-    (property "Reference" "TP11" (at 238.76 88.1379 0)
+    (property "Reference" "TP11" (at 238.76 89.4079 0)
       (effects (font (size 1.27 1.27)) (justify left))
     )
-    (property "Value" "Test Point" (at 238.76 90.6779 0)
+    (property "Value" "Test Point" (at 238.76 91.9479 0)
       (effects (font (size 1.27 1.27)) (justify left))
     )
-    (property "Footprint" "TestPoint:TestPoint_Pad_D1.5mm" (at 241.3 92.71 0)
+    (property "Footprint" "TestPoint:TestPoint_Pad_D1.5mm" (at 241.3 93.98 0)
       (effects (font (size 1.27 1.27)) (hide yes))
     )
-    (property "Datasheet" "~" (at 241.3 92.71 0)
+    (property "Datasheet" "~" (at 241.3 93.98 0)
       (effects (font (size 1.27 1.27)) (hide yes))
     )
-    (property "Description" "SMT Test Point 1.5mm round" (at 236.22 92.71 0)
+    (property "Description" "SMT Test Point 1.5mm round" (at 236.22 93.98 0)
       (effects (font (size 1.27 1.27)) (hide yes))
     )
-    (property "IPN" "M-TEST-SMT_1.5mm_round" (at 236.22 92.71 0)
+    (property "IPN" "M-TEST-SMT_1.5mm_round" (at 236.22 93.98 0)
       (effects (font (size 1.27 1.27)) (hide yes))
     )
-    (property "Comments" "TestPoint 1.5mm" (at 236.22 92.71 0)
+    (property "Comments" "TestPoint 1.5mm" (at 236.22 93.98 0)
       (effects (font (size 1.27 1.27)) (hide yes))
     )

Commit message: Deploying to gh-pages from @ Nautilus-UUV/nautilus-mainboard-PCB@03be77246175febedc852bdb83cb4e2df1ae0c88 🚀
Other:
- note added: "logo sync doesnt work?"
Changed lines of the file:
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@@
     (effects (font (size 1.27 1.27)))
+  )
+  (text "logo sync doesnt work?" (exclude_from_sim no) (at 257.81 155.702 0)
+    (effects (font (size 1.27 1.27)))
+  )
+  (symbol (lib_id "#dzdb:g_art/ART-LOGO-Davide-silkscreen") (at 259.08 170.18 0) (unit 1)
+    (exclude_from_sim no) (in_bom no) (on_board yes) (dnp no) (fields_autoplaced)
+    (property "Reference" "#G1" (at 259.08 156.972 0)
+      (effects (font (size 1.27 1.27)) (hide yes))
+    )
+    (property "Value" "Davide's Logo silkscreen" (at 259.0252 158.75 0)
+      (effects (font (size 1.27 1.27)))
+    )
+    (property "Footprint" "dz_art:davide_logo" (at 259.08 170.18 0)
+      (effects (font (size 1.27 1.27)) (hide yes))
+    )
+    (property "Datasheet" "" (at 259.08 170.18 0)
+      (effects (font (size 1.27 1.27)) (hide yes))
+    )
+    (property "Description" "Davide's Logo silkscreen" (at 259.08 170.18 0)
+      (effects (font (size 1.27 1.27)) (hide yes))
+    )
+    (property "IPN" "ART-LOGO-Davide-silkscreen" (at 259.08 170.18 0)
+      (effects (font (size 1.27 1.27)) (hide yes))
+    )
+    (property "Comments" "Davide Logo" (at 259.08 170.18 0)
+      (effects (font (size 1.27 1.27)) (hide yes))
+    )
+    (instances
+      (project ""
+        (path "/ce1819b2-f280-40ed-834f-6fe4d12f809d"
+          (reference "#G1") (unit 1)
+        )
+      )
+    )
   )
   (symbol (lib_id "power:+3.3V") (at 237.49 63.5 0) (unit 1)
