File: Browse/GPIO_REF3.3V.kicad_sch (KiCad schematic)
At the start: 14 parts, among them IC4 TPS2121RUXT

Commit message: Deploying to gh-pages from @ Nautilus-UUV/nautilus-mainboard-PCB@4372544f9d98c8c318df3aa79b1ddc615587ee00 🚀
Parts:
- renumbered IC4 to IC5, R14 to R25
Changed lines of the file:
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@@
     (pin "2")
     (instances
-      (project ""
-        (path "/ce1819b2-f280-40ed-834f-6fe4d12f809d/c1998c4d-3f9a-4761-b447-a813532738a0/e46d3b44-477e-48ec-b385-9b4870813d66"
+      (project "nautilus_mainboard"
+        (path "/ce1819b2-f280-40ed-834f-6fe4d12f809d/c1998c4d-3f9a-4761-b447-a813532738a0/b9b676f4-45ad-4d4b-96a9-894c1f9d02cb"
           (reference "C39") (unit 1)
         )
@@
     (instances
       (project "nautilus_mainboard"
-        (path "/ce1819b2-f280-40ed-834f-6fe4d12f809d/c1998c4d-3f9a-4761-b447-a813532738a0/e46d3b44-477e-48ec-b385-9b4870813d66"
+        (path "/ce1819b2-f280-40ed-834f-6fe4d12f809d/c1998c4d-3f9a-4761-b447-a813532738a0/b9b676f4-45ad-4d4b-96a9-894c1f9d02cb"
           (reference "C40") (unit 1)
         )
@@
     (instances
       (project "nautilus_mainboard"
-        (path "/ce1819b2-f280-40ed-834f-6fe4d12f809d/c1998c4d-3f9a-4761-b447-a813532738a0/e46d3b44-477e-48ec-b385-9b4870813d66"
+        (path "/ce1819b2-f280-40ed-834f-6fe4d12f809d/c1998c4d-3f9a-4761-b447-a813532738a0/b9b676f4-45ad-4d4b-96a9-894c1f9d02cb"
           (reference "R26") (unit 1)
         )
@@
   (symbol (lib_id "#dzdb:g_res/R-15.4k-0603") (at 129.54 85.09 0) (unit 1)
     (exclude_from_sim no) (in_bom yes) (on_board yes) (dnp no)
-    (property "Reference" "R14" (at 129.54 87.122 90)
+    (property "Reference" "R25" (at 129.54 87.122 90)
       (effects (font (size 1.27 1.27)) (justify left))
     )
@@
     (instances
       (project "nautilus_mainboard"
-        (path "/ce1819b2-f280-40ed-834f-6fe4d12f809d/c1998c4d-3f9a-4761-b447-a813532738a0/e46d3b44-477e-48ec-b385-9b4870813d66"
-          (reference "R14") (unit 1)
+        (path "/ce1819b2-f280-40ed-834f-6fe4d12f809d/c1998c4d-3f9a-4761-b447-a813532738a0/b9b676f4-45ad-4d4b-96a9-894c1f9d02cb"
+          (reference "R25") (unit 1)
         )
       )
@@
     (instances
       (project "nautilus_mainboard"
-        (path "/ce1819b2-f280-40ed-834f-6fe4d12f809d/c1998c4d-3f9a-4761-b447-a813532738a0/e46d3b44-477e-48ec-b385-9b4870813d66"
+        (path "/ce1819b2-f280-40ed-834f-6fe4d12f809d/c1998c4d-3f9a-4761-b447-a813532738a0/b9b676f4-45ad-4d4b-96a9-894c1f9d02cb"
           (reference "R28") (unit 1)
         )
@@
     (instances
       (project "nautilus_mainboard"
-        (path "/ce1819b2-f280-40ed-834f-6fe4d12f809d/c1998c4d-3f9a-4761-b447-a813532738a0/e46d3b44-477e-48ec-b385-9b4870813d66"
+        (path "/ce1819b2-f280-40ed-834f-6fe4d12f809d/c1998c4d-3f9a-4761-b447-a813532738a0/b9b676f4-45ad-4d4b-96a9-894c1f9d02cb"
           (reference "C37") (unit 1)
         )
@@
   (symbol (lib_id "power:GND") (at 168.91 123.19 0) (unit 1)
     (exclude_from_sim no) (in_bom yes) (on_board yes) (dnp no) (fields_autoplaced)
-    (property "Reference" "#PWR033" (at 168.91 129.54 0)
+    (property "Reference" "#PWR030" (at 168.91 129.54 0)
       (effects (font (size 1.27 1.27)) (hide yes))
     )
@@
     (instances
       (project "nautilus_mainboard"
-        (path "/ce1819b2-f280-40ed-834f-6fe4d12f809d/c1998c4d-3f9a-4761-b447-a813532738a0/e46d3b44-477e-48ec-b385-9b4870813d66"
-          (reference "#PWR033") (unit 1)
+        (path "/ce1819b2-f280-40ed-834f-6fe4d12f809d/c1998c4d-3f9a-4761-b447-a813532738a0/b9b676f4-45ad-4d4b-96a9-894c1f9d02cb"
+          (reference "#PWR030") (unit 1)
         )
       )
@@
     (instances
       (project "nautilus_mainboard"
-        (path "/ce1819b2-f280-40ed-834f-6fe4d12f809d/c1998c4d-3f9a-4761-b447-a813532738a0/e46d3b44-477e-48ec-b385-9b4870813d66"
+        (path "/ce1819b2-f280-40ed-834f-6fe4d12f809d/c1998c4d-3f9a-4761-b447-a813532738a0/b9b676f4-45ad-4d4b-96a9-894c1f9d02cb"
           (reference "C41") (unit 1)
         )
@@
     (instances
       (project "nautilus_mainboard"
-        (path "/ce1819b2-f280-40ed-834f-6fe4d12f809d/c1998c4d-3f9a-4761-b447-a813532738a0/e46d3b44-477e-48ec-b385-9b4870813d66"
+        (path "/ce1819b2-f280-40ed-834f-6fe4d12f809d/c1998c4d-3f9a-4761-b447-a813532738a0/b9b676f4-45ad-4d4b-96a9-894c1f9d02cb"
           (reference "C35") (unit 1)
         )
@@
     (instances
       (project "nautilus_mainboard"
-        (path "/ce1819b2-f280-40ed-834f-6fe4d12f809d/c1998c4d-3f9a-4761-b447-a813532738a0/e46d3b44-477e-48ec-b385-9b4870813d66"
+        (path "/ce1819b2-f280-40ed-834f-6fe4d12f809d/c1998c4d-3f9a-4761-b447-a813532738a0/b9b676f4-45ad-4d4b-96a9-894c1f9d02cb"
           (reference "R29") (unit 1)
         )
@@
     (pin "1")
     (instances
-      (project ""
-        (path "/ce1819b2-f280-40ed-834f-6fe4d12f809d/c1998c4d-3f9a-4761-b447-a813532738a0/e46d3b44-477e-48ec-b385-9b4870813d66"
+      (project "nautilus_mainboard"
+        (path "/ce1819b2-f280-40ed-834f-6fe4d12f809d/c1998c4d-3f9a-4761-b447-a813532738a0/b9b676f4-45ad-4d4b-96a9-894c1f9d02cb"
           (reference "R30") (unit 1)
         )
@@
     (instances
       (project "nautilus_mainboard"
-        (path "/ce1819b2-f280-40ed-834f-6fe4d12f809d/c1998c4d-3f9a-4761-b447-a813532738a0/e46d3b44-477e-48ec-b385-9b4870813d66"
+        (path "/ce1819b2-f280-40ed-834f-6fe4d12f809d/c1998c4d-3f9a-4761-b447-a813532738a0/b9b676f4-45ad-4d4b-96a9-894c1f9d02cb"
           (reference "C38") (unit 1)
         )
@@
     (instances
       (project "nautilus_mainboard"
-        (path "/ce1819b2-f280-40ed-834f-6fe4d12f809d/c1998c4d-3f9a-4761-b447-a813532738a0/e46d3b44-477e-48ec-b385-9b4870813d66"
+        (path "/ce1819b2-f280-40ed-834f-6fe4d12f809d/c1998c4d-3f9a-4761-b447-a813532738a0/b9b676f4-45ad-4d4b-96a9-894c1f9d02cb"
           (reference "R27") (unit 1)
         )
@@
   (symbol (lib_id "#dzdb:s_misc/TEXA-595-TPS2121RUXT") (at 132.08 88.9 0) (unit 1)
     (exclude_from_sim no) (in_bom yes) (on_board yes) (dnp no) (fields_autoplaced)
-    (property "Reference" "IC4" (at 146.05 119.38 0)
+    (property "Reference" "IC5" (at 146.05 119.38 0)
       (effects (font (size 1.27 1.27)))
     )
@@
     (instances
       (project "nautilus_mainboard"
-        (path "/ce1819b2-f280-40ed-834f-6fe4d12f809d/c1998c4d-3f9a-4761-b447-a813532738a0/e46d3b44-477e-48ec-b385-9b4870813d66"
-          (reference "IC4") (unit 1)
+        (path "/ce1819b2-f280-40ed-834f-6fe4d12f809d/c1998c4d-3f9a-4761-b447-a813532738a0/b9b676f4-45ad-4d4b-96a9-894c1f9d02cb"
+          (reference "IC5") (unit 1)
         )
       )
@@
     (instances
       (project "nautilus_mainboard"
-        (path "/ce1819b2-f280-40ed-834f-6fe4d12f809d/c1998c4d-3f9a-4761-b447-a813532738a0/e46d3b44-477e-48ec-b385-9b4870813d66"
+        (path "/ce1819b2-f280-40ed-834f-6fe4d12f809d/c1998c4d-3f9a-4761-b447-a813532738a0/b9b676f4-45ad-4d4b-96a9-894c1f9d02cb"
           (reference "C36") (unit 1)
         )

Commit message: Deploying to gh-pages from @ Nautilus-UUV/nautilus-mainboard-PCB@f1dd6ce1e57c066b805694b10777c719502cca87 🚀
Parts:
- removed C35, C36: 10uF, Capacitor_SMD:C_1210_3225Metric, symbol #dzdb:s_cap/C-MUR-GRM32EC72A106KE05
- removed C37, C38, C40: 100nF, Capacitor_SMD:C_0603_1608Metric, symbol #dzdb:g_cap/C-100n-0603
- removed C41: 47uF, Capacitor_SMD:C_0805_2012Metric, symbol #dzdb:s_cap/C-MUR-GRM21BR61A476ME15
- removed IC5: TPS2121RUXT, dz_dio:TI_Switchover_TPS2121RUXT, symbol #dzdb:s_misc/TEXA-595-TPS2121RUXT
- removed R25: 15.4k, Resistor_SMD:R_0603_1608Metric, symbol #dzdb:g_res/R-15.4k-0603
- removed R26, R28: 4.99k, Resistor_SMD:R_0603_1608Metric, symbol #dzdb:g_res/R-4.99k-0603
- removed R29: 20k, Resistor_SMD:R_0603_1608Metric, symbol #dzdb:g_res/R-20k-0603
- removed R30: 100k, Resistor_SMD:R_0603_1608Metric, symbol #dzdb:g_res/R-100k-0603
- added C48, C49: 10uF, Capacitor_SMD:C_1210_3225Metric, symbol #dzdb:s_cap/C-MUR-GRM32EC72A106KE05
- added C50, C51, C52: 100nF, Capacitor_SMD:C_0603_1608Metric, symbol #dzdb:g_cap/C-100n-0603
- added C54: 47uF, Capacitor_SMD:C_0805_2012Metric, symbol #dzdb:s_cap/C-MUR-GRM21BR61A476ME15
- added IC3: TPS2121RUXT, dz_dio:TI_Switchover_TPS2121RUXT, symbol #dzdb:s_misc/TEXA-595-TPS2121RUXT
- added R14: 100k, Resistor_SMD:R_0603_1608Metric, symbol #dzdb:g_res/R-100k-0603
- added TP13: Test Point, TestPoint:TestPoint_Pad_D1.5mm, symbol #dzdb:g_mech/M-TEST-SMT_1.5mm_round
Connections:
- net CM4_OUT_3.3V: now also C49.1, C51.1, IC3.2 (IN2)
- net GND: now also C39.1, R27.1, C48.2, C49.2, C50.2, C51.2, C52.2, C54.2, IC3.12 (GND), IC3.3 (CP2), IC3.4 (OV2), IC3.5 (OV1), R14.2; no longer C39.2, R27.2
- net GPIO_VREF_3.3V: now also C52.1, C54.1, IC3.1 (OUT_1), IC3.8 (OUT_2), R14.1, TP13.1
- net STM_IN_3.3V: now also C48.1, C50.1, IC3.6 (PR1), IC3.7 (IN1)
- new net: C39.2, IC3.11 (SS)
- new net: IC3.10 (ILIM), R27.2
Other:
- note removed: "100nF CLOSE"
- note removed: "SAME AS IN 5V"
- note removed: "V-div (same ratio as 5V)"
- company: (none) -> Davide
- title: (none) -> Nautilus_Mainboard
- moved on the sheet: C39, R27

Commit message: Deploying to gh-pages from @ Nautilus-UUV/nautilus-mainboard-PCB@5f5fdd9436d408a604bb268d740c0ac7ce1f5af5 🚀
Parts:
- removed C48, C49: 10uF, Capacitor_SMD:C_1210_3225Metric, symbol #dzdb:s_cap/C-MUR-GRM32EC72A106KE05
- removed C50, C51, C52: 100nF, Capacitor_SMD:C_0603_1608Metric, symbol #dzdb:g_cap/C-100n-0603
- removed C54: 47uF, Capacitor_SMD:C_0805_2012Metric, symbol #dzdb:s_cap/C-MUR-GRM21BR61A476ME15
- removed IC3: TPS2121RUXT, dz_dio:TI_Switchover_TPS2121RUXT, symbol #dzdb:s_misc/TEXA-595-TPS2121RUXT
- removed R14: 100k, Resistor_SMD:R_0603_1608Metric, symbol #dzdb:g_res/R-100k-0603
- removed TP13: Test Point, TestPoint:TestPoint_Pad_D1.5mm, symbol #dzdb:g_mech/M-TEST-SMT_1.5mm_round
- added C35, C36: 10uF, Capacitor_SMD:C_1210_3225Metric, symbol #dzdb:s_cap/C-MUR-GRM32EC72A106KE05
- added C37, C38, C40: 100nF, Capacitor_SMD:C_0603_1608Metric, symbol #dzdb:g_cap/C-100n-0603
- added C41: 47uF, Capacitor_SMD:C_0805_2012Metric, symbol #dzdb:s_cap/C-MUR-GRM21BR61A476ME15
- added IC5: TPS2121RUXT, dz_dio:TI_Switchover_TPS2121RUXT, symbol #dzdb:s_misc/TEXA-595-TPS2121RUXT
- added R25: 15.4k, Resistor_SMD:R_0603_1608Metric, symbol #dzdb:g_res/R-15.4k-0603
- added R26, R28: 4.99k, Resistor_SMD:R_0603_1608Metric, symbol #dzdb:g_res/R-4.99k-0603
- added R29: 20k, Resistor_SMD:R_0603_1608Metric, symbol #dzdb:g_res/R-20k-0603
- added R30: 100k, Resistor_SMD:R_0603_1608Metric, symbol #dzdb:g_res/R-100k-0603
Connections:
- net CM4_OUT_3.3V: now also C36.1, C38.1, IC5.2 (IN2), R29.2
- net GND: now also C39.2, R27.2, C35.2, C36.2, C37.2, C38.2, C40.2, C41.2, IC5.12 (GND), IC5.4 (OV2), IC5.5 (OV1), R26.1, R28.1, R30.2; no longer C39.1, R27.1
- net GPIO_VREF_3.3V: now also C40.1, C41.1, IC5.1 (OUT_1), IC5.8 (OUT_2), R30.1
- net STM_IN_3.3V: now also C35.1, C37.1, IC5.7 (IN1), R25.2
- new net: C39.1, IC5.11 (SS)
- new net: IC5.6 (PR1), R25.1, R26.2
- new net: IC5.3 (CP2), R28.2, R29.1
- new net: IC5.10 (ILIM), R27.1
Other:
- note added: "100nF CLOSE"
- note added: "SAME AS IN 5V"
- note added: "V-div (same ratio as 5V)"
- company: Davide -> (none)
- title: Nautilus_Mainboard -> (none)
- moved on the sheet: C39, R27

Commit message: Deploying to gh-pages from @ Nautilus-UUV/nautilus-mainboard-PCB@2d3890115fd9d3c0bb909c9898aa64801bed9e67 🚀
Parts:
- removed C35, C36: 10uF, Capacitor_SMD:C_1210_3225Metric, symbol #dzdb:s_cap/C-MUR-GRM32EC72A106KE05
- removed C37, C38, C40: 100nF, Capacitor_SMD:C_0603_1608Metric, symbol #dzdb:g_cap/C-100n-0603
- removed C41: 47uF, Capacitor_SMD:C_0805_2012Metric, symbol #dzdb:s_cap/C-MUR-GRM21BR61A476ME15
- removed IC5: TPS2121RUXT, dz_dio:TI_Switchover_TPS2121RUXT, symbol #dzdb:s_misc/TEXA-595-TPS2121RUXT
- removed R25: 15.4k, Resistor_SMD:R_0603_1608Metric, symbol #dzdb:g_res/R-15.4k-0603
- removed R26, R28: 4.99k, Resistor_SMD:R_0603_1608Metric, symbol #dzdb:g_res/R-4.99k-0603
- removed R29: 20k, Resistor_SMD:R_0603_1608Metric, symbol #dzdb:g_res/R-20k-0603
- removed R30: 100k, Resistor_SMD:R_0603_1608Metric, symbol #dzdb:g_res/R-100k-0603
- added C48, C49: 10uF, Capacitor_SMD:C_1210_3225Metric, symbol #dzdb:s_cap/C-MUR-GRM32EC72A106KE05
- added C50, C51, C52: 100nF, Capacitor_SMD:C_0603_1608Metric, symbol #dzdb:g_cap/C-100n-0603
- added C54: 47uF, Capacitor_SMD:C_0805_2012Metric, symbol #dzdb:s_cap/C-MUR-GRM21BR61A476ME15
- added IC3: TPS2121RUXT, dz_dio:TI_Switchover_TPS2121RUXT, symbol #dzdb:s_misc/TEXA-595-TPS2121RUXT
- added R14: 100k, Resistor_SMD:R_0603_1608Metric, symbol #dzdb:g_res/R-100k-0603
Connections:
- net CM4_OUT_3.3V: now also C49.1, C51.1, IC3.2 (IN2)
- net GND: now also C39.1, R27.1, C48.2, C49.2, C50.2, C51.2, C52.2, C54.2, IC3.12 (GND), IC3.3 (CP2), IC3.4 (OV2), IC3.5 (OV1), R14.2; no longer C39.2, R27.2
- net GPIO_VREF_3.3V: now also C52.1, C54.1, IC3.1 (OUT_1), IC3.8 (OUT_2), R14.1
- net STM_IN_3.3V: now also C48.1, C50.1, IC3.6 (PR1), IC3.7 (IN1)
- new net: C39.2, IC3.11 (SS)
- new net: IC3.10 (ILIM), R27.2
Other:
- note removed: "100nF CLOSE"
- note removed: "SAME AS IN 5V"
- note removed: "V-div (same ratio as 5V)"
- company: (none) -> Davide
- moved on the sheet: C39, R27

Commit message: Deploying to gh-pages from @ Nautilus-UUV/nautilus-mainboard-PCB@5b07cf6af03655ef9ddad269b1edd5eb03bfa75f 🚀
Other:
- title: (none) -> Nautilus_Mainboard
Changed lines of the file:
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@@
   (paper "A4")
   (title_block
+    (title "Nautilus_Mainboard")
     (date "2025-11-19")
     (rev "0")

Commit message: Deploying to gh-pages from @ Nautilus-UUV/nautilus-mainboard-PCB@62d9beca31554f779583bfc3c938b3f82a581309 🚀
Parts:
- added TP13: Test Point, TestPoint:TestPoint_Pad_D1.5mm, symbol #dzdb:g_mech/M-TEST-SMT_1.5mm_round
Connections:
- net GPIO_VREF_3.3V: now also TP13.1
Changed lines of the file:
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@@
+    )
+  )
+  (symbol (lib_id "#dzdb:g_mech/M-TEST-SMT_1.5mm_round") (at 172.72 77.47 0) (unit 1)
+    (exclude_from_sim no) (in_bom yes) (on_board yes) (dnp no)
+    (property "Reference" "TP13" (at 175.26 72.8979 0)
+      (effects (font (size 1.27 1.27)) (justify left))
+    )
+    (property "Value" "Test Point" (at 175.26 74.93 0)
+      (effects (font (size 1.27 1.27)) (justify left))
+    )
+    (property "Footprint" "TestPoint:TestPoint_Pad_D1.5mm" (at 177.8 77.47 0)
+      (effects (font (size 1.27 1.27)) (hide yes))
+    )
+    (property "Datasheet" "~" (at 177.8 77.47 0)
+      (effects (font (size 1.27 1.27)) (hide yes))
+    )
+    (property "Description" "SMT Test Point 1.5mm round" (at 172.72 77.47 0)
+      (effects (font (size 1.27 1.27)) (hide yes))
+    )
+    (property "IPN" "M-TEST-SMT_1.5mm_round" (at 172.72 77.47 0)
+      (effects (font (size 1.27 1.27)) (hide yes))
+    )
+    (property "Comments" "TestPoint 1.5mm" (at 172.72 77.47 0)
+      (effects (font (size 1.27 1.27)) (hide yes))
+    )
+    (pin "1")
+    (instances
+      (project "nautilus_mainboard"
+        (path "/ce1819b2-f280-40ed-834f-6fe4d12f809d/c1998c4d-3f9a-4761-b447-a813532738a0/b9b676f4-45ad-4d4b-96a9-894c1f9d02cb"
+          (reference "TP13") (unit 1)
+        )
+      )
     )
   )
