File: Browse/3.3V_Logic.kicad_sch (KiCad schematic)
At the start: 13 parts, among them IC5 TPS2121RUXT

Commit message: Deploying to gh-pages from @ Nautilus-UUV/nautilus-mainboard-PCB@4372544f9d98c8c318df3aa79b1ddc615587ee00 🚀
Parts:
- renumbered C28 to C21, C29 to C22, C30 to C23, C31 to C24, C32 to C25, C33 to C26, C34 to C27, IC5 to IC3, R21 to R14, R22 to R16, R23 to R17, R24 to R18, R25 to R19

Commit message: Deploying to gh-pages from @ Nautilus-UUV/nautilus-mainboard-PCB@f87e8fd5b4d00ad24387b205f01c25b4db3035ed 🚀
Connections:
- net STM_IN_3.3V renamed +3.3V
Changed lines of the file:
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@@
     (stroke (width 0) (type default))
   )
-  (text "100nF CLOSE" (exclude_from_sim no) (at 122.936 97.536 0)
+  (text "100nF CLOSE" (exclude_from_sim no) (at 116.332 98.044 0)
     (effects (font (size 1.27 1.27)))
   )
@@
   (hierarchical_label "Battery_Out_3.3V" (shape output) (at 95.25 85.09 180)
     (effects (font (size 1.27 1.27)) (justify right))
-  )
-  (hierarchical_label "STM_IN_3.3V" (shape output) (at 172.72 85.09 0)
-    (effects (font (size 1.27 1.27)) (justify left))
   )
   (hierarchical_label "STM_Plug_3.3V" (shape output) (at 95.25 100.33 180)
@@
   (symbol (lib_id "#dzdb:s_cap/C-MUR-GRM32EC72A106KE05") (at 110.49 104.14 0) (unit 1)
     (exclude_from_sim no) (in_bom yes) (on_board yes) (dnp no)
-    (property "Reference" "C22" (at 108.966 101.854 0)
-      (effects (font (size 1.27 1.27)) (justify left))
-    )
-    (property "Value" "10uF" (at 108.458 106.426 0)
+    (property "Reference" "C22" (at 106.172 101.854 0)
+      (effects (font (size 1.27 1.27)) (justify left))
+    )
+    (property "Value" "10uF" (at 105.41 106.426 0)
       (effects (font (size 1.27 1.27)) (justify left))
     )
@@
   (symbol (lib_id "#dzdb:g_cap/C-100n-0603") (at 119.38 104.14 0) (unit 1)
     (exclude_from_sim no) (in_bom yes) (on_board yes) (dnp no)
-    (property "Reference" "C24" (at 117.348 102.108 0)
-      (effects (font (size 1.27 1.27)) (justify left))
-    )
-    (property "Value" "100nF" (at 116.332 106.172 0)
+    (property "Reference" "C24" (at 115.062 101.854 0)
+      (effects (font (size 1.27 1.27)) (justify left))
+    )
+    (property "Value" "100nF" (at 113.284 106.426 0)
       (effects (font (size 1.27 1.27)) (justify left))
     )
@@
   (symbol (lib_id "#dzdb:g_cap/C-330n-0603") (at 157.48 106.68 90) (unit 1)
     (exclude_from_sim no) (in_bom yes) (on_board yes) (dnp no)
-    (property "Reference" "C25" (at 157.48 105.41 90)
+    (property "Reference" "C25" (at 160.782 105.41 90)
       (effects (font (size 1.27 1.27)))
     )
-    (property "Value" "330nF" (at 157.734 107.95 90)
+    (property "Value" "330nF" (at 161.798 108.204 90)
       (effects (font (size 1.27 1.27)))
     )
@@
     )
   )
+  (symbol (lib_id "power:+3.3V") (at 172.72 85.09 0) (unit 1)
+    (exclude_from_sim no) (in_bom yes) (on_board yes) (dnp no) (fields_autoplaced)
+    (property "Reference" "#PWR033" (at 172.72 88.9 0)
+      (effects (font (size 1.27 1.27)) (hide yes))
+    )
+    (property "Value" "+3.3V" (at 172.72 80.01 0)
+      (effects (font (size 1.27 1.27)))
+    )
+    (property "Footprint" "" (at 172.72 85.09 0)
+      (effects (font (size 1.27 1.27)) (hide yes))
+    )
+    (property "Datasheet" "" (at 172.72 85.09 0)
+      (effects (font (size 1.27 1.27)) (hide yes))
+    )
+    (property "Description" "Power symbol creates a global label with name \"+3.3V\"" (at 172.72 85.09 0)
+      (effects (font (size 1.27 1.27)) (hide yes))
+    )
+    (pin "1")
+    (instances
+      (project ""
+        (path "/ce1819b2-f280-40ed-834f-6fe4d12f809d/c1998c4d-3f9a-4761-b447-a813532738a0/b867d855-894b-4aa9-b170-e48a88a70717"
+          (reference "#PWR033") (unit 1)
+        )
+      )
+    )
+  )
   (symbol (lib_id "#dzdb:g_res/R-15.4k-0603") (at 123.19 81.28 0) (unit 1)
     (exclude_from_sim no) (in_bom yes) (on_board yes) (dnp no)
@@
   (symbol (lib_id "#dzdb:s_cap/C-MUR-GRM32EC72A106KE05") (at 110.49 88.9 0) (unit 1)
     (exclude_from_sim no) (in_bom yes) (on_board yes) (dnp no)
-    (property "Reference" "C21" (at 108.966 86.614 0)
-      (effects (font (size 1.27 1.27)) (justify left))
-    )
-    (property "Value" "10uF" (at 108.458 91.186 0)
+    (property "Reference" "C21" (at 105.918 86.614 0)
+      (effects (font (size 1.27 1.27)) (justify left))
+    )
+    (property "Value" "10uF" (at 105.41 91.186 0)
       (effects (font (size 1.27 1.27)) (justify left))
     )
@@
   (symbol (lib_id "#dzdb:g_cap/C-100n-0603") (at 119.38 88.9 0) (unit 1)
     (exclude_from_sim no) (in_bom yes) (on_board yes) (dnp no)
-    (property "Reference" "C23" (at 117.602 87.122 0)
-      (effects (font (size 1.27 1.27)) (justify left))
-    )
-    (property "Value" "100nF" (at 116.078 90.932 0)
-      (effects (font (size 1.27 1.27)) (justify left))
-    )
+    (property "Reference" "C23" (at 114.554 87.122 0)
+      (effects (font (size 1.27 1.27)) (justify left))
+    )
+    (property "Value" "100nF" (at 113.03 90.932 0)
+      (effects (font (size 1.27 1.27)) (justify left))
+    )

Commit message: Deploying to gh-pages from @ Nautilus-UUV/nautilus-mainboard-PCB@a81f7ffbfc5f9b51f47d7f388c30fcea2673b9ea 🚀
Connections:
- net +3.3V renamed STM_In_3.3V
Changed lines of the file:
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@@
     (effects (font (size 1.27 1.27)) (justify right))
+  )
+  (hierarchical_label "STM_In_3.3V" (shape output) (at 172.72 85.09 0)
+    (effects (font (size 1.27 1.27)) (justify left))
   )
   (hierarchical_label "STM_Plug_3.3V" (shape output) (at 95.25 100.33 180)
@@
         )
       )
-    )
-  )
-  (symbol (lib_id "power:+3.3V") (at 172.72 85.09 0) (unit 1)
-    (exclude_from_sim no) (in_bom yes) (on_board yes) (dnp no) (fields_autoplaced)
-    (property "Reference" "#PWR033" (at 172.72 88.9 0)
-      (effects (font (size 1.27 1.27)) (hide yes))
-    )
-    (property "Value" "+3.3V" (at 172.72 80.01 0)
-      (effects (font (size 1.27 1.27)))
-    )
-    (property "Footprint" "" (at 172.72 85.09 0)
-      (effects (font (size 1.27 1.27)) (hide yes))
-    )
-    (property "Datasheet" "" (at 172.72 85.09 0)
-      (effects (font (size 1.27 1.27)) (hide yes))
-    )
-    (property "Description" "Power symbol creates a global label with name \"+3.3V\"" (at 172.72 85.09 0)
-      (effects (font (size 1.27 1.27)) (hide yes))
-    )
-    (pin "1")
-    (instances
-      (project ""
-        (path "/ce1819b2-f280-40ed-834f-6fe4d12f809d/c1998c4d-3f9a-4761-b447-a813532738a0/b867d855-894b-4aa9-b170-e48a88a70717"
-          (reference "#PWR033") (unit 1)
-        )
-      )

Commit message: Deploying to gh-pages from @ Nautilus-UUV/nautilus-mainboard-PCB@2d3890115fd9d3c0bb909c9898aa64801bed9e67 🚀
Parts:
- removed IC3: TPS2121RUXT, dz_dio:TI_Switchover_TPS2121RUXT, symbol #dzdb:s_misc/TEXA-595-TPS2121RUXT
- removed R14: 15.4k, Resistor_SMD:R_0603_1608Metric, symbol #dzdb:g_res/R-15.4k-0603
- removed R16, R18: 4.99k, Resistor_SMD:R_0603_1608Metric, symbol #dzdb:g_res/R-4.99k-0603
- removed R19: 20k, Resistor_SMD:R_0603_1608Metric, symbol #dzdb:g_res/R-20k-0603
- added IC6: TPS2121RUXT, dz_dio:TI_Switchover_TPS2121RUXT, symbol #dzdb:s_misc/TEXA-595-TPS2121RUXT
Connections:
- net Battery_Out_3.3V: now also IC6.6 (PR1), IC6.7 (IN1)
- net GND: now also C25.1, IC6.12 (GND), IC6.3 (CP2), IC6.4 (OV2), IC6.5 (OV1); no longer C25.2
- net STM_In_3.3V: now also IC6.1 (OUT_1), IC6.8 (OUT_2)
- net STM_Plug_3.3V: now also IC6.2 (IN2)
- net at R17.1: now also IC6.10 (ILIM)
- new net: C25.2, IC6.11 (SS)
Other:
- note removed: "100nF CLOSE"
- note removed: "SAME AS IN 5V"
- note removed: "V-div (same ratio as 5V)"
- company: (none) -> Davide
- moved on the sheet: C21, C22, C23, C24, C25, C26, C27, R17

Commit message: Deploying to gh-pages from @ Nautilus-UUV/nautilus-mainboard-PCB@5b07cf6af03655ef9ddad269b1edd5eb03bfa75f 🚀
Other:
- title: (none) -> Nautilus_Mainboard
Changed lines of the file:
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@@
   (paper "A4")
   (title_block
+    (title "Nautilus_Mainboard")
     (date "2025-11-19")
     (rev "0")

Commit message: Deploying to gh-pages from @ Nautilus-UUV/nautilus-mainboard-PCB@5f5fdd9436d408a604bb268d740c0ac7ce1f5af5 🚀
Parts:
- removed IC6: TPS2121RUXT, dz_dio:TI_Switchover_TPS2121RUXT, symbol #dzdb:s_misc/TEXA-595-TPS2121RUXT
- added IC3: TPS2121RUXT, dz_dio:TI_Switchover_TPS2121RUXT, symbol #dzdb:s_misc/TEXA-595-TPS2121RUXT
- added R14: 15.4k, Resistor_SMD:R_0603_1608Metric, symbol #dzdb:g_res/R-15.4k-0603
- added R16, R18: 4.99k, Resistor_SMD:R_0603_1608Metric, symbol #dzdb:g_res/R-4.99k-0603
- added R19: 20k, Resistor_SMD:R_0603_1608Metric, symbol #dzdb:g_res/R-20k-0603
Connections:
- net Battery_Out_3.3V: now also IC3.7 (IN1), R14.2
- net GND: now also C25.2, IC3.12 (GND), IC3.4 (OV2), IC3.5 (OV1), R16.1, R18.1; no longer C25.1
- net STM_Plug_3.3V: now also IC3.2 (IN2), R19.2
- net at R17.1: now also IC3.10 (ILIM)
- net STM_In_3.3V renamed STM_IN_3.3V
- net STM_IN_3.3V: now also IC3.1 (OUT_1), IC3.8 (OUT_2)
- new net: C25.1, IC3.11 (SS)
- new net: IC3.3 (CP2), R18.2, R19.1
- new net: IC3.6 (PR1), R14.1, R16.2
Other:
- note added: "100nF CLOSE"
- note added: "SAME AS IN 5V"
- note added: "V-div (same ratio as 5V)"
- company: Davide -> (none)
- title: Nautilus_Mainboard -> (none)
- moved on the sheet: C21, C22, C23, C24, C25, C26, C27, R17
