File: Browse/3.3V_Logic.kicad_sch (KiCad schematic)
At the start: 13 parts, among them IC3 TPS2121RUXT

Commit message: Deploying to gh-pages from @ Nautilus-UUV/nautilus-mainboard-PCB@f1dd6ce1e57c066b805694b10777c719502cca87 🚀
Parts:
- removed IC3: TPS2121RUXT, dz_dio:TI_Switchover_TPS2121RUXT, symbol #dzdb:s_misc/TEXA-595-TPS2121RUXT
- removed R14: 15.4k, Resistor_SMD:R_0603_1608Metric, symbol #dzdb:g_res/R-15.4k-0603
- removed R16, R18: 4.99k, Resistor_SMD:R_0603_1608Metric, symbol #dzdb:g_res/R-4.99k-0603
- removed R19: 20k, Resistor_SMD:R_0603_1608Metric, symbol #dzdb:g_res/R-20k-0603
- added IC6: TPS2121RUXT, dz_dio:TI_Switchover_TPS2121RUXT, symbol #dzdb:s_misc/TEXA-595-TPS2121RUXT
Connections:
- net Battery_Out_3.3V: now also IC6.6 (PR1), IC6.7 (IN1)
- net GND: now also C25.1, IC6.12 (GND), IC6.3 (CP2), IC6.4 (OV2), IC6.5 (OV1); no longer C25.2
- net STM_Plug_3.3V: now also IC6.2 (IN2)
- net at R17.1: now also IC6.10 (ILIM)
- net STM_IN_3.3V renamed STM_In_3.3V
- net STM_In_3.3V: now also IC6.1 (OUT_1), IC6.8 (OUT_2)
- new net: C25.2, IC6.11 (SS)
Other:
- note removed: "100nF CLOSE"
- note removed: "SAME AS IN 5V"
- note removed: "V-div (same ratio as 5V)"
- company: (none) -> Davide
- title: (none) -> Nautilus_Mainboard
- moved on the sheet: C21, C22, C23, C24, C25, C26, C27, R17
