File: Browse/CM4_Module1A.kicad_sch (KiCad schematic)
At the start: 11 parts, among them Q2 50V

Commit message: Deploying to gh-pages from @ Nautilus-UUV/nautilus-mainboard-PCB@b62834b88bb3e2a9413bcb4ea8e223af403e20ba 🚀
Connections:
- net ET1 renamed TRD0.D-
- net ET2 renamed TRD0.D+
- net ET3 renamed TRD1.D-
- net ET4 renamed TRD1.D+
- net ET5 renamed TRD2.D-
- net ET6 renamed TRD2.D+
- net ET7 renamed TRD3.D-
- net ET8 renamed TRD3.D+

Commit message: Deploying to gh-pages from @ Nautilus-UUV/nautilus-mainboard-PCB@f87e8fd5b4d00ad24387b205f01c25b4db3035ed 🚀
Connections:
- net AIN0: no longer names the net of Module1.96 (AnalogIP0)
- net AIN1: no longer names the net of Module1.94 (AnalogIP1)
- no-connect marks 50 -> 52
Changed lines of the file:
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@@
   (no_connect (at 101.6 100.33))
   (no_connect (at 26.67 59.69))
+  (no_connect (at 40.64 143.51))
   (no_connect (at 101.6 110.49))
   (no_connect (at 101.6 107.95))
+  (no_connect (at 40.64 140.97))
   (no_connect (at 40.64 148.59))
   (no_connect (at 26.67 90.17))
@@
     (stroke (width 0) (type default))
   )
-  (wire (pts (xy 26.67 140.97) (xy 40.64 140.97))
-    (stroke (width 0) (type default))
-  )
   (wire (pts (xy 101.6 87.63) (xy 152.4 87.63))
     (stroke (width 0) (type default))
@@
   )
   (wire (pts (xy 106.68 39.37) (xy 106.68 52.07))
-    (stroke (width 0) (type default))
-  )
-  (wire (pts (xy 26.67 143.51) (xy 40.64 143.51))
     (stroke (width 0) (type default))
   )
@@
     (effects (font (size 1.27 1.27)) (justify left bottom))
   )
-  (label "AIN0" (at 26.67 143.51 0)
-    (effects (font (size 1.27 1.27)) (justify left bottom))
-  )
   (label "TRD2.D+" (at 185.42 45.72 0)
     (effects (font (size 1.27 1.27)) (justify left bottom))
@@
     (effects (font (size 1.27 1.27)) (justify right bottom))
   )
-  (label "AIN1" (at 26.67 140.97 0)
-    (effects (font (size 1.27 1.27)) (justify left bottom))
-  )
   (label "TRD3.D-" (at 185.42 48.26 0)

Commit message: Deploying to gh-pages from @ Nautilus-UUV/nautilus-mainboard-PCB@44ad8adb17f33e1aa4439bd10449a9ac7e221a1f 🚀
Connections:
- net CM4_IN_5V renamed +5V
Other:
- sheet CM4_Ethernet ports: added TRD0{D+ D-}, TRD1{D+ D-}, TRD2{D+ D-}, TRD3{D+ D-}; removed TRD0_N, TRD0_P, TRD1_N, TRD1_P, TRD2_N, TRD2_P, TRD3_N, TRD3_P

Commit message: Deploying to gh-pages from @ Nautilus-UUV/nautilus-mainboard-PCB@a81f7ffbfc5f9b51f47d7f388c30fcea2673b9ea 🚀
Connections:
- net CM4_OUT_3.3V renamed CM4_Out_3.3V
Other:
- sheet CM4_Ethernet ports: added LAN_IN_3.3V; removed none
- sheet CM4_LED1 ports: added Battery_Out_3.3V; removed none
- sheet CM4_LED2 ports: added Battery_Out_3.3V; removed none

Commit message: Deploying to gh-pages from @ Nautilus-UUV/nautilus-mainboard-PCB@2d3890115fd9d3c0bb909c9898aa64801bed9e67 🚀
Other:
- company: (none) -> Davide
Changed lines of the file:
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@@
 (kicad_sch (version 20250114) (generator "eeschema") (generator_version "9.0")
   (paper "A4")
+  (title_block
+    (date "2025-11-18")
+    (company "Davide")
+  )
   (junction (at 222.25 157.48) (diameter 0) (color 0 0 0 0)
   )

Commit message: Deploying to gh-pages from @ Nautilus-UUV/nautilus-mainboard-PCB@8b02e89ade7c168188296ba6f0516f3abec9166b 🚀
Changed lines of the file:
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@@
   (paper "A4")
   (title_block
-    (date "2025-11-18")
+    (date "2025-11-19")
+    (rev "0")
     (company "Davide")
   )
@@
       (effects (font (size 1.27 1.27)) (justify left top))
     )
-    (pin "PI_nLED_Activity" input (at 135.89 49.53 180)
-      (effects (font (size 1.27 1.27)) (justify left))
-    )
     (pin "Battery_Out_3.3V" input (at 135.89 46.99 180)
       (effects (font (size 1.27 1.27)) (justify left))
     )
+    (pin "PI_nLED_Activity" output (at 135.89 49.53 180)
+      (effects (font (size 1.27 1.27)) (justify left))
+    )

Commit message: Deploying to gh-pages from @ Nautilus-UUV/nautilus-mainboard-PCB@5b07cf6af03655ef9ddad269b1edd5eb03bfa75f 🚀
Other:
- title: (none) -> Nautilus_Mainboard
Changed lines of the file:
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@@
   (paper "A4")
   (title_block
+    (title "Nautilus_Mainboard")
     (date "2025-11-19")
     (rev "0")

Commit message: Deploying to gh-pages from @ Nautilus-UUV/nautilus-mainboard-PCB@5f5fdd9436d408a604bb268d740c0ac7ce1f5af5 🚀
Connections:
- net AIN1: now reaches Module1.94 (AnalogIP1)
- net AIN0: now reaches Module1.96 (AnalogIP0)
- net +5V renamed CM4_IN_5V
- net CM4_Out_3.3V renamed CM4_OUT_3.3V
- no-connect marks 52 -> 50
Other:
- sheet CM4_Ethernet ports: added TRD0_N, TRD0_P, TRD1_N, TRD1_P, TRD2_N, TRD2_P, TRD3_N, TRD3_P; removed LAN_IN_3.3V, TRD0{D+ D-}, TRD1{D+ D-}, TRD2{D+ D-}, TRD3{D+ D-}
- sheet CM4_LED1 ports: added none; removed Battery_Out_3.3V
- sheet CM4_LED2 ports: added none; removed Battery_Out_3.3V
- company: Davide -> (none)
- title: Nautilus_Mainboard -> (none)
