File: Browse/PinoutSTM.kicad_sch (KiCad schematic)
At the start: 23 parts, among them IC1 STM32H7B0RBT6, J1 FTSH-107-02-L-DV, J2 61300211121, J4 Header male 1x05, J5 1792876, Q1 50V, SW1 Button Switch SPST-No, Y1 CC4V-T1A-32.768kHz-6pF-20PPM-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

Commit message: Deploying to gh-pages from @ Nautilus-UUV/nautilus-mainboard-PCB@b7db83c6a38e7ed72f880de916f2e48939069e27 🚀
Changed lines of the file:
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@@
   (symbol (lib_id "#dzdb:g_res/R-0-0603") (at 60.96 20.32 180) (unit 1)
     (exclude_from_sim no) (in_bom yes) (on_board yes) (dnp no)
-    (property "Reference" "EXTERNALFAN5V1" (at 56.642 20.066 90)
+    (property "Reference" "EXTERNALFAN5V1" (at 49.53 13.208 0)
       (effects (font (size 1.27 1.27)))
     )
@@
   )
   (symbol (lib_id "#dzdb:g_cap/C-100n-0603") (at 186.69 163.83 0) (unit 1)
-    (exclude_from_sim no) (in_bom yes) (on_board yes) (dnp no) (fields_autoplaced)
-    (property "Reference" "C18" (at 190.5 162.5599 0)
-      (effects (font (size 1.27 1.27)) (justify left))
-    )
-    (property "Value" "100nF" (at 190.5 165.0999 0)
+    (exclude_from_sim no) (in_bom yes) (on_board yes) (dnp no)
+    (property "Reference" "C18" (at 189.992 162.052 0)
+      (effects (font (size 1.27 1.27)) (justify left))
+    )
+    (property "Value" "100nF" (at 189.738 164.846 0)
       (effects (font (size 1.27 1.27)) (justify left))
     )
@@
   (symbol (lib_id "#dzdb:s_cap/C-MUR-GRM32EC72A106KE05") (at 198.12 163.83 0) (unit 1)
     (exclude_from_sim no) (in_bom yes) (on_board yes) (dnp no)
-    (property "Reference" "C16" (at 196.596 161.544 0)
-      (effects (font (size 1.27 1.27)) (justify left))
-    )
-    (property "Value" "10uF" (at 196.088 166.116 0)
-      (effects (font (size 1.27 1.27)) (justify left))
-    )
+    (property "Reference" "C16" (at 201.168 162.814 0)
+      (effects (font (size 1.27 1.27)) (justify left))
+    )
+    (property "Value" "10uF" (at 200.66 164.846 0)
+      (effects (font (size 1.27 1.27)) (justify left))
+    )

Commit message: Deploying to gh-pages from @ Nautilus-UUV/nautilus-mainboard-PCB@44ad8adb17f33e1aa4439bd10449a9ac7e221a1f 🚀
Connections:
- net STM_IN_3.3V renamed +3.3V
Other:
- note added: "must be hirarchical lable RX,TX"
Changed lines of the file:
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@@
     (stroke (width 0) (type default))
   )
-  (wire (pts (xy 58.42 87.63) (xy 72.39 87.63))
+  (wire (pts (xy 59.69 87.63) (xy 72.39 87.63))
     (stroke (width 0) (type default))
   )
@@
     (effects (font (size 1.27 1.27)) (justify left))
   )
-  (text "logic handled in power section" (exclude_from_sim no) (at 213.36 68.58 0)
+  (text "must be hirarchical lable RX,TX" (exclude_from_sim no) (at 33.274 106.68 0)
+    (effects (font (size 1.27 1.27)))
+  )
+  (text "logic handled in power section" (exclude_from_sim no) (at 222.504 71.374 0)
     (effects (font (size 1.27 1.27)))
   )
@@
     (effects (font (size 1.27 1.27)) (justify right bottom))
   )
-  (label "nRST" (at 60.96 87.63 0)
+  (label "nRST" (at 59.69 87.63 0)
     (effects (font (size 1.27 1.27)) (justify left bottom))
   )
@@
     (effects (font (size 1.27 1.27)) (justify right bottom))
   )
-  (global_label "STM_IN_3.3V" (shape input) (at 203.2 72.39 0) (fields_autoplaced)
-    (effects (font (size 1.27 1.27)) (justify left))
-    (property "Intersheetrefs" "${INTERSHEET_REFS}" (at 217.7966 72.39 0)
-      (effects (font (size 1.27 1.27)) (justify left) (hide yes))
-    )
-  )
-  (global_label "STM_TX" (shape input) (at 59.69 105.41 180) (fields_autoplaced)
+  (global_label "STM_TX" (shape output) (at 59.69 105.41 180) (fields_autoplaced)
     (effects (font (size 1.27 1.27)) (justify right))
     (property "Intersheetrefs" "${INTERSHEET_REFS}" (at 49.9316 105.41 0)
@@
     (effects (font (size 1.27 1.27)) (justify right))
   )
-  (hierarchical_label "Pack1_SCL" (shape input) (at 87.63 48.26 90)
+  (hierarchical_label "Pack1_SCL" (shape bidirectional) (at 87.63 48.26 90)
     (effects (font (size 1.27 1.27)) (justify left))
   )
@@
     (effects (font (size 1.27 1.27)) (justify left))
   )
-  (hierarchical_label "Pack1_SDA" (shape input) (at 85.09 48.26 90)
+  (hierarchical_label "Pack1_SDA" (shape bidirectional) (at 85.09 48.26 90)
     (effects (font (size 1.27 1.27)) (justify left))
   )
@@
         )
       )
+    )
+  )
+  (symbol (lib_id "power:+3.3V") (at 203.2 72.39 0) (unit 1)
+    (exclude_from_sim no) (in_bom yes) (on_board yes) (dnp no)
+    (property "Reference" "#PWR045" (at 203.2 76.2 0)
+      (effects (font (size 1.27 1.27)) (hide yes))
+    )
+    (property "Value" "+3.3V" (at 203.2 67.564 0)
+      (effects (font (size 1.27 1.27)))
+    )
+    (property "Footprint" "" (at 203.2 72.39 0)
+      (effects (font (size 1.27 1.27)) (hide yes))
+    )
+    (property "Datasheet" "" (at 203.2 72.39 0)
+      (effects (font (size 1.27 1.27)) (hide yes))
+    )
+    (property "Description" "Power symbol creates a global label with name \"+3.3V\"" (at 203.2 72.39 0)
+      (effects (font (size 1.27 1.27)) (hide yes))
+    )
+    (pin "1")
+    (instances
+      (project ""
+        (path "/ce1819b2-f280-40ed-834f-6fe4d12f809d/46fb4fb5-44f2-465b-b1ff-e4e0fbef74ae/fadabe7f-e4de-4ec7-8fb6-d9f38e9db4fc"
+          (reference "#PWR045") (unit 1)
+        )
+      )

Commit message: Deploying to gh-pages from @ Nautilus-UUV/nautilus-mainboard-PCB@a81f7ffbfc5f9b51f47d7f388c30fcea2673b9ea 🚀
Connections:
- net Battery_Out_5V renamed +5V
Changed lines of the file:
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@@
   (junction (at 161.29 167.64) (diameter 0) (color 0 0 0 0)
   )
+  (junction (at 60.96 24.13) (diameter 0) (color 0 0 0 0)
+  )
   (junction (at 38.1 43.18) (diameter 0) (color 0 0 0 0)
   )
@@
     (stroke (width 0) (type default))
   )
-  (wire (pts (xy 251.46 16.51) (xy 251.46 20.32))
+  (wire (pts (xy 251.46 17.78) (xy 251.46 20.32))
     (stroke (width 0) (type default))
   )
@@
     (stroke (width 0) (type default))
   )
-  (wire (pts (xy 251.46 16.51) (xy 250.19 16.51))
+  (wire (pts (xy 251.46 17.78) (xy 250.19 17.78))
     (stroke (width 0) (type default))
   )
@@
     (stroke (width 0) (type default))
   )
+  (wire (pts (xy 55.88 31.75) (xy 60.96 31.75))
+    (stroke (width 0) (type default))
+  )
   (polyline (pts (xy 173.99 13.97) (xy 173.99 63.5))
     (stroke (width 0) (type default))
@@
     (stroke (width 0) (type default))
   )
+  (wire (pts (xy 60.96 31.75) (xy 60.96 24.13))
+    (stroke (width 0) (type default))
+  )
   (wire (pts (xy 134.62 167.64) (xy 135.89 167.64))
     (stroke (width 0) (type default))
@@
     )
   )
-  (global_label "STM_Plug_3.3V" (shape output) (at 250.19 16.51 180) (fields_autoplaced)
-    (effects (font (size 1.27 1.27)) (justify right))
-    (property "Intersheetrefs" "${INTERSHEET_REFS}" (at 233.2955 16.51 0)
-      (effects (font (size 1.27 1.27)) (justify right) (hide yes))
-    )
-  )
   (global_label "STM_RX" (shape input) (at 59.69 107.95 180) (fields_autoplaced)
     (effects (font (size 1.27 1.27)) (justify right))
@@
     )
   )
-  (global_label "Battery_Out_5V" (shape input) (at 60.96 24.13 270) (fields_autoplaced)
+  (hierarchical_label "STM_USART_RX" (shape input) (at 80.01 140.97 270)
     (effects (font (size 1.27 1.27)) (justify right))
-    (property "Intersheetrefs" "${INTERSHEET_REFS}" (at 60.96 41.2665 90)
-      (effects (font (size 1.27 1.27)) (justify right) (hide yes))
-    )
   )
-  (hierarchical_label "STM_USART_RX" (shape input) (at 80.01 140.97 270)
+  (hierarchical_label "STM_Plug_3.3V" (shape output) (at 250.19 17.78 180)
     (effects (font (size 1.27 1.27)) (justify right))
   )
@@
         )
       )
+    )
+  )
+  (symbol (lib_id "power:+5V") (at 55.88 31.75 0) (unit 1)
+    (exclude_from_sim no) (in_bom yes) (on_board yes) (dnp no) (fields_autoplaced)
+    (property "Reference" "#PWR047" (at 55.88 35.56 0)
+      (effects (font (size 1.27 1.27)) (hide yes))
+    )
+    (property "Value" "+5V" (at 55.88 26.67 0)
+      (effects (font (size 1.27 1.27)))
+    )
+    (property "Footprint" "" (at 55.88 31.75 0)
+      (effects (font (size 1.27 1.27)) (hide yes))
+    )
+    (property "Datasheet" "" (at 55.88 31.75 0)
+      (effects (font (size 1.27 1.27)) (hide yes))
+    )
+    (property "Description" "Power symbol creates a global label with name \"+5V\"" (at 55.88 31.75 0)
+      (effects (font (size 1.27 1.27)) (hide yes))
+    )
+    (pin "1")
+    (instances
+      (project ""
+        (path "/ce1819b2-f280-40ed-834f-6fe4d12f809d/46fb4fb5-44f2-465b-b1ff-e4e0fbef74ae/fadabe7f-e4de-4ec7-8fb6-d9f38e9db4fc"
+          (reference "#PWR047") (unit 1)
+        )
+      )

Commit message: Deploying to gh-pages from @ Nautilus-UUV/nautilus-mainboard-PCB@2d3890115fd9d3c0bb909c9898aa64801bed9e67 🚀
Connections:
- net Piezzo_Control: now reaches IC1.38 (PC7)
- no-connect marks 33 -> 32
Other:
- note added: "Chose a Pin here please."
- note added: "I chose 7 but please make sure its an actual pin evan. I just gambled."
- company: (none) -> Evan
Changed lines of the file:
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@@
 (kicad_sch (version 20250114) (generator "eeschema") (generator_version "9.0")
   (paper "A4")
+  (title_block
+    (date "2025-11-18")
+    (company "Evan")
+  )
   (junction (at 161.29 160.02) (diameter 0) (color 0 0 0 0)
   )
@@
   (no_connect (at 87.63 128.27))
   (no_connect (at 110.49 128.27))
-  (no_connect (at 125.73 97.79))
   (no_connect (at 125.73 100.33))
   (wire (pts (xy 34.29 86.36) (xy 31.75 86.36))
@@
     (stroke (width 0) (type default))
   )
+  (wire (pts (xy 125.73 97.79) (xy 149.86 97.79))
+    (stroke (width 0) (type default))
+  )
   (wire (pts (xy 241.3 38.1) (xy 241.3 40.64))
     (stroke (width 0) (type default))
@@
     (effects (font (size 1.27 1.27)))
   )
+  (text "Chose a Pin here please." (exclude_from_sim no) (at 150.114 100.33 0)
+    (effects (font (size 1.27 1.27)))
+  )
   (text "External interfaces\n\n" (exclude_from_sim no) (at 183.896 16.764 0)
     (effects (font (size 1.27 1.27)))
@@
     (effects (font (size 1.27 1.27)))
   )
+  (text "I chose 7 but please make sure its an actual pin evan. I just gambled." (exclude_from_sim no) (at 164.846 102.616 0)
+    (effects (font (size 1.27 1.27)))
+  )
   (label "UART4_TX" (at 60.96 105.41 0)
     (effects (font (size 1.27 1.27)) (justify left bottom))
@@
     (effects (font (size 1.27 1.27)) (justify right))
   )
+  (hierarchical_label "Piezzo_Control" (shape output) (at 149.86 97.79 0)
+    (effects (font (size 1.27 1.27)) (justify left))
+  )
   (hierarchical_label "STM_USART_TX" (shape output) (at 59.69 110.49 180)

Commit message: Deploying to gh-pages from @ Nautilus-UUV/nautilus-mainboard-PCB@8b02e89ade7c168188296ba6f0516f3abec9166b 🚀
Changed lines of the file:
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@@
   (paper "A4")
   (title_block
-    (date "2025-11-18")
+    (date "2025-11-19")
+    (rev "0")
     (company "Evan")
   )

Commit message: Deploying to gh-pages from @ Nautilus-UUV/nautilus-mainboard-PCB@5b07cf6af03655ef9ddad269b1edd5eb03bfa75f 🚀
Parts:
- added D2, D3, D4: 710-82402374, Package_TO_SOT_SMD:SOT-23-5, symbol #dzdb:s_dio/WURT-710-82402374
Connections:
- net +3.3V: now also D4.4 (K)
- net GND: now also D2.2 (A), D3.2 (A), D4.2 (A)
- net JTAG_ TDI: now also D3.4 (K)
- net JTAG_TCK/SWCLK: now also D4.1 (K)
- net JTAG_TDO/SWO: now also D3.5 (K)
- net JTAG_TMS/SWDIO: now also D4.3 (K)
- net STM_BOOT0: now also D2.1 (K)
- net STM_Plug_3.3V: now also D2.5 (K)
- net USART1_RX: now also D2.4 (K), D4.5 (K)
- net USART1_TX: now also D2.3 (K), D3.1 (K)
- net nRST: now also D3.3 (K)
- net STM_RX renamed STM.RX
- net STM_TX renamed STM.TX
Other:
- note added: "For review: if this pin is incorrect, Im sorry. I just guessed please let me know so that I can tell evan if it needs to be changed."
- note added: "This part should be changed... implement directly a fan not this 3 pin screw terminal that I randomly found @evan"
- title: (none) -> Nautilus_Mainboard
- moved on the sheet: EXTERNALFAN5V1, J1

Commit message: Deploying to gh-pages from @ Nautilus-UUV/nautilus-mainboard-PCB@2b5265db7706a31505c0a0411337a4a604b5fb21 🚀
Connections:
- net STM_Plug_3.3V: now also D2.4 (K); no longer D2.5 (K)
- net USART1_RX: now also D2.5 (K); no longer D2.4 (K)
Changed lines of the file:
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@@
   (junction (at 173.99 160.02) (diameter 0) (color 0 0 0 0)
   )
+  (junction (at 34.29 86.36) (diameter 0) (color 0 0 0 0)
+  )
+  (junction (at 186.69 160.02) (diameter 0) (color 0 0 0 0)
+  )
+  (junction (at 148.59 167.64) (diameter 0) (color 0 0 0 0)
+  )
+  (junction (at 241.3 27.94) (diameter 0) (color 0 0 0 0)
+  )
+  (junction (at 161.29 167.64) (diameter 0) (color 0 0 0 0)
+  )
+  (junction (at 38.1 43.18) (diameter 0) (color 0 0 0 0)
+  )
+  (junction (at 186.69 167.64) (diameter 0) (color 0 0 0 0)
+  )
+  (junction (at 165.1 41.91) (diameter 0) (color 0 0 0 0)
+  )
+  (junction (at 148.59 160.02) (diameter 0) (color 0 0 0 0)
+  )
   (junction (at 251.46 20.32) (diameter 0) (color 0 0 0 0)
-  )
-  (junction (at 34.29 86.36) (diameter 0) (color 0 0 0 0)
-  )
-  (junction (at 186.69 160.02) (diameter 0) (color 0 0 0 0)
-  )
-  (junction (at 148.59 167.64) (diameter 0) (color 0 0 0 0)
-  )
-  (junction (at 241.3 27.94) (diameter 0) (color 0 0 0 0)
-  )
-  (junction (at 161.29 167.64) (diameter 0) (color 0 0 0 0)
-  )
-  (junction (at 38.1 43.18) (diameter 0) (color 0 0 0 0)
-  )
-  (junction (at 186.69 167.64) (diameter 0) (color 0 0 0 0)
-  )
-  (junction (at 165.1 41.91) (diameter 0) (color 0 0 0 0)
-  )
-  (junction (at 148.59 160.02) (diameter 0) (color 0 0 0 0)
   )
   (junction (at 251.46 44.45) (diameter 0) (color 0 0 0 0)
@@
     (stroke (width 0) (type default))
   )
-  (wire (pts (xy 224.79 20.32) (xy 251.46 20.32))
-    (stroke (width 0) (type default))
-  )
   (wire (pts (xy 125.73 82.55) (xy 140.97 82.55))
     (stroke (width 0) (type default))
@@
     (stroke (width 0) (type default))
   )
+  (wire (pts (xy 251.46 20.32) (xy 240.03 20.32))
+    (stroke (width 0) (type default))
+  )
   (wire (pts (xy 189.23 39.37) (xy 208.28 39.37))
     (stroke (width 0) (type default))
@@
     (stroke (width 0) (type default))
   )
+  (wire (pts (xy 236.22 20.32) (xy 224.79 20.32))
+    (stroke (width 0) (type default))
+  )
   (wire (pts (xy 38.1 43.18) (xy 62.23 43.18))
     (stroke (width 0) (type default))
@@
     (stroke (width 0) (type default))
   )
+  (wire (pts (xy 236.22 22.86) (xy 236.22 20.32))
+    (stroke (width 0) (type default))
+  )
   (wire (pts (xy 53.34 80.01) (xy 72.39 80.01))
     (stroke (width 0) (type default))
@@
     (stroke (width 0) (type default))
   )
-  (wire (pts (xy 224.79 22.86) (xy 259.08 22.86))
-    (stroke (width 0) (type default))
-  )
   (wire (pts (xy 46.99 86.36) (xy 50.8 86.36))
     (stroke (width 0) (type default))
@@
     (stroke (width 0) (type default))
   )
+  (wire (pts (xy 240.03 21.59) (xy 228.6 21.59))
+    (stroke (width 0) (type default))
+  )
   (wire (pts (xy 38.1 36.83) (xy 38.1 43.18))
     (stroke (width 0) (type default))
@@
     (stroke (width 0) (type default))
   )
+  (wire (pts (xy 228.6 22.86) (xy 224.79 22.86))
+    (stroke (width 0) (type default))
+  )
   (wire (pts (xy 166.37 41.91) (xy 165.1 41.91))
     (stroke (width 0) (type default))
@@
     (stroke (width 0) (type default))
   )
+  (wire (pts (xy 240.03 20.32) (xy 240.03 21.59))
+    (stroke (width 0) (type default))
+  )
   (wire (pts (xy 52.07 24.13) (xy 52.07 22.86))
     (stroke (width 0) (type default))
@@
     (stroke (width 0) (type default))
   )
+  (wire (pts (xy 236.22 22.86) (xy 259.08 22.86))
+    (stroke (width 0) (type default))
+  )
+  (wire (pts (xy 228.6 21.59) (xy 228.6 22.86))
+    (stroke (width 0) (type default))
+  )

Commit message: Deploying to gh-pages from @ Nautilus-UUV/nautilus-mainboard-PCB@5f5fdd9436d408a604bb268d740c0ac7ce1f5af5 🚀
Parts:
- removed D2, D3, D4: 710-82402374, Package_TO_SOT_SMD:SOT-23-5, symbol #dzdb:s_dio/WURT-710-82402374
Connections:
- net +3.3V renamed STM_IN_3.3V
- net +5V renamed Battery_Out_5V
- net Piezzo_Control: no longer names the net of IC1.38 (PC7)
- net STM.RX renamed STM_RX
- net STM.TX renamed STM_TX
- no-connect marks 32 -> 33
Other:
- note removed: "Chose a Pin here please."
- note removed: "For review: if this pin is incorrect, Im sorry. I just guessed please let me know so that I can tell evan if it needs to be changed."
- note removed: "I chose 7 but please make sure its an actual pin evan. I just gambled."
- note removed: "This part should be changed... implement directly a fan not this 3 pin screw terminal that I randomly found @evan"
- note removed: "must be hirarchical lable RX,TX"
- company: Evan -> (none)
- title: Nautilus_Mainboard -> (none)
- moved on the sheet: EXTERNALFAN5V1, J1
