File: Browse/CM4_LED1.kicad_sch (KiCad schematic)
At the start: 3 parts, among them U3 Buffers & Line Driver

Commit message: Deploying to gh-pages from @ Nautilus-UUV/nautilus-mainboard-PCB@2d3890115fd9d3c0bb909c9898aa64801bed9e67 🚀
Other:
- company: (none) -> Davide
Changed lines of the file:
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@@
 (kicad_sch (version 20250114) (generator "eeschema") (generator_version "9.0")
   (paper "A4")
+  (title_block
+    (date "2025-11-18")
+    (company "Davide")
+  )
   (junction (at 105.41 53.34) (diameter 0) (color 0 0 0 0)
   )

Commit message: Deploying to gh-pages from @ Nautilus-UUV/nautilus-mainboard-PCB@8b02e89ade7c168188296ba6f0516f3abec9166b 🚀
Parts:
- removed D1: APHHS1005LSECK/J3-PF, LED_SMD:LED_0402_1005Metric, symbol #dzdb:s_dio/D-KIN-APHHS1005LSECK/J3-PF
- added LED8: 710-150060YS83000, dz_dio:Wuerth_LED_150060RS83000, symbol #dzdb:s_dio/D-WURT-710-150060YS83000
Connections:
- net Battery_Out_3.3V: now also LED8.2 (A)
- net at R5.2: now also LED8.1 (K)
Changed lines of the file:
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@@
   (paper "A4")
   (title_block
-    (date "2025-11-18")
+    (date "2025-11-19")
+    (rev "0")
     (company "Davide")
   )
@@
     (stroke (width 0) (type default))
   )
+  (wire (pts (xy 165.1 74.93) (xy 170.18 74.93))
+    (stroke (width 0) (type default))
+  )
+  (wire (pts (xy 105.41 53.34) (xy 170.18 53.34))
+    (stroke (width 0) (type default))
+  )
   (wire (pts (xy 137.16 74.93) (xy 157.48 74.93))
-    (stroke (width 0) (type default))
-  )
-  (wire (pts (xy 165.1 74.93) (xy 170.18 74.93))
-    (stroke (width 0) (type default))
-  )
-  (wire (pts (xy 105.41 53.34) (xy 170.18 53.34))
     (stroke (width 0) (type default))
   )
@@
     (effects (font (size 1.27 1.27)) (justify right))
   )
-  (symbol (lib_id "#dzdb:s_dio/D-KIN-APHHS1005LSECK/J3-PF") (at 161.29 74.93 0) (mirror x) (unit 1)
-    (exclude_from_sim no) (in_bom yes) (on_board yes) (dnp no)
-    (property "Reference" "D1" (at 159.7025 81.28 0)
-      (effects (font (size 1.27 1.27)))
-    )
-    (property "Value" "APHHS1005LSECK/J3-PF" (at 159.7025 78.74 0)
-      (effects (font (size 1.27 1.27)))
-    )
-    (property "Footprint" "LED_SMD:LED_0402_1005Metric" (at 161.29 74.93 0)
-      (effects (font (size 1.27 1.27)) (hide yes))
-    )
-    (property "Datasheet" "https://www.kingbrightusa.com/images/catalog/spec/APHHS1005LSECK-J3-PF.pdf" (at 161.29 74.93 0)
-      (effects (font (size 1.27 1.27)) (hide yes))
-    )
-    (property "Description" "LED RED 625nm 80mcd@2mA 40mcd@1mA 1.8V" (at 161.29 74.93 0)
-      (effects (font (size 1.27 1.27)) (hide yes))
-    )
-    (property "Sim.Pins" "1=K 2=A" (at 161.29 74.93 0)
-      (effects (font (size 1.27 1.27)) (hide yes))
-    )
-    (property "IPN" "D-KIN-APHHS1005LSECK/J3-PF" (at 161.29 74.93 0)
-      (effects (font (size 1.27 1.27)) (hide yes))
-    )
-    (property "MPN" "APHHS1005LSECK/J3-PF" (at 161.29 74.93 0)
-      (effects (font (size 1.27 1.27)) (hide yes))
-    )
-    (property "Manufacturer" "Kingbright" (at 161.29 74.93 0)
-      (effects (font (size 1.27 1.27)) (hide yes))
-    )
-    (property "Type" "LED RED" (at 161.29 74.93 0)
-      (effects (font (size 1.27 1.27)) (hide yes))
-    )
-    (property "Vf" "1.8V" (at 161.29 74.93 0)
-      (effects (font (size 1.27 1.27)) (hide yes))
-    )
-    (property "If" "2mA" (at 161.29 74.93 0)
-      (effects (font (size 1.27 1.27)) (hide yes))
-    )
-    (property "Supplier" "Mouser" (at 161.29 74.93 0)
-      (effects (font (size 1.27 1.27)) (hide yes))
-    )
-    (property "SPN" "604-APHHS1005LSECKJ3" (at 161.29 74.93 0)
-      (effects (font (size 1.27 1.27)) (hide yes))
-    )
-    (property "LCSC" "" (at 161.29 74.93 0)
-      (effects (font (size 1.27 1.27)) (hide yes))
-    )
-    (property "Comment" "lifecycle=Active" (at 161.29 74.93 0)
-      (effects (font (size 1.27 1.27)) (hide yes))
-    )
-    (pin "1")
-    (pin "2")
-    (instances
-      (project "nautilus_mainboard"
-        (path "/ce1819b2-f280-40ed-834f-6fe4d12f809d/c2b6dac3-d6fd-4d5d-bd17-0cff91db88eb/0837dad1-ec16-488a-a684-981e55247089/e0935ee6-fc77-4de6-a0ac-caf50bea3bcd"
-          (reference "D1") (unit 1)
-        )
-      )
-    )
-  )
   (symbol (lib_id "power:GND") (at 105.41 91.44 0) (unit 1)
     (exclude_from_sim no) (in_bom yes) (on_board yes) (dnp no) (fields_autoplaced)
@@
         )
       )
+    )
+  )
+  (symbol (lib_id "#dzdb:s_dio/D-WURT-710-150060YS83000") (at 161.29 74.93 0) (mirror y) (unit 1)
+    (exclude_from_sim no) (in_bom yes) (on_board yes) (dnp no)
+    (property "Reference" "LED8" (at 154.94 71.12 0)
+      (effects (font (size 1.27 1.27)))
+    )
+    (property "Value" "710-150060YS83000" (at 158.75 67.818 0)
+      (effects (font (size 1.27 1.27)))
+    )
+    (property "Footprint" "dz_dio:Wuerth_LED_150060RS83000" (at 148.59 168.58 0)
+      (effects (font (size 1.27 1.27)) (justify left bottom) (hide yes))
+    )
+    (property "Datasheet" "https://www.we-online.com/catalog/datasheet/150060SY83000.pdf" (at 148.59 268.58 0)
+      (effects (font (size 1.27 1.27)) (justify left bottom) (hide yes))
+    )
+    (property "Description" "Einfarbige LEDs leds WL-SMCW SMT 0603 Dome Yellow Typ 650mcd 2V" (at 161.29 74.93 0)
+      (effects (font (size 1.27 1.27)) (hide yes))
+    )
+    (property "Height" "0.95" (at 148.59 468.58 0)
+      (effects (font (size 1.27 1.27)) (justify left bottom) (hide yes))
+    )
+    (property "Mouser Part Number" "" (at 148.59 568.58 0)
+      (effects (font (size 1.27 1.27)) (justify left bottom) (hide yes))
+    )
+    (property "Mouser Price/Stock" "" (at 148.59 668.58 0)
+      (effects (font (size 1.27 1.27)) (justify left bottom) (hide yes))
+    )
+    (property "Manufacturer_Name" "Wurth Elektronik" (at 148.59 768.58 0)
+      (effects (font (size 1.27 1.27)) (justify left bottom) (hide yes))
+    )
+    (property "Manufacturer_Part_Number" "150060RS83000" (at 148.59 868.58 0)
+      (effects (font (size 1.27 1.27)) (justify left bottom) (hide yes))
+    )
+    (property "IPN" "D-WURT-710-150060YS83000" (at 161.29 74.93 0)
+      (effects (font (size 1.27 1.27)) (hide yes))
+    )
+    (property "MPN" "710-150060YS83000" (at 161.29 74.93 0)
+      (effects (font (size 1.27 1.27)) (hide yes))
+    )
+    (property "Manufacturer" "Wurth Elektronik" (at 161.29 74.93 0)
+      (effects (font (size 1.27 1.27)) (hide yes))
+    )
+    (property "Type" "Einfarbige LEDs leds" (at 161.29 74.93 0)
+      (effects (font (size 1.27 1.27)) (hide yes))
+    )
+    (property "Vf" "2V" (at 161.29 74.93 0)
+      (effects (font (size 1.27 1.27)) (hide yes))
+    )
+    (property "If" "20 mA" (at 161.29 74.93 0)
+      (effects (font (size 1.27 1.27)) (hide yes))
+    )
+    (property "Supplier" "Mouser" (at 161.29 74.93 0)
+      (effects (font (size 1.27 1.27)) (hide yes))
+    )
+    (property "SPN" "710-150060YS83000" (at 161.29 74.93 0)
+      (effects (font (size 1.27 1.27)) (hide yes))
+    )
+    (property "LCSC" "" (at 161.29 74.93 0)
+      (effects (font (size 1.27 1.27)) (hide yes))
+    )
+    (property "Comment" "lifecycle=New Product" (at 161.29 74.93 0)
+      (effects (font (size 1.27 1.27)) (hide yes))
+    )
+    (pin "2")
+    (pin "1")
+    (instances
+      (project ""
+        (path "/ce1819b2-f280-40ed-834f-6fe4d12f809d/c2b6dac3-d6fd-4d5d-bd17-0cff91db88eb/0837dad1-ec16-488a-a684-981e55247089/e0935ee6-fc77-4de6-a0ac-caf50bea3bcd"
+          (reference "LED8") (unit 1)
+        )
+      )

Commit message: Deploying to gh-pages from @ Nautilus-UUV/nautilus-mainboard-PCB@5b07cf6af03655ef9ddad269b1edd5eb03bfa75f 🚀
Other:
- note added: "From the CM4 io board"
- title: (none) -> Nautilus_Mainboard

Commit message: Deploying to gh-pages from @ Nautilus-UUV/nautilus-mainboard-PCB@5f5fdd9436d408a604bb268d740c0ac7ce1f5af5 🚀
Parts:
- removed LED8: 710-150060YS83000, dz_dio:Wuerth_LED_150060RS83000, symbol #dzdb:s_dio/D-WURT-710-150060YS83000
- added D1: APHHS1005LSECK/J3-PF, LED_SMD:LED_0402_1005Metric, symbol #dzdb:s_dio/D-KIN-APHHS1005LSECK/J3-PF
- added TP1: Test Point, TestPoint:TestPoint_Pad_D1.5mm, symbol #dzdb:g_mech/M-TEST-SMT_1.5mm_round
Connections:
- net at R5.2: now also D1.1 (K), TP1.1
- new net CM4_LED_IN_3.3V: D1.2 (A)
Other:
- note added: "<---"
- note added: "issue: will that logic work if I use USB vin only?"
- note added: "only use when connected completely? not over usb???"
- note added: "then I would in theory compare internal voltage with internal voltage... so probably not..."
- note removed: "From the CM4 io board"
- company: Davide -> (none)
- title: Nautilus_Mainboard -> (none)

Commit message: Deploying to gh-pages from @ Nautilus-UUV/nautilus-mainboard-PCB@f1dd6ce1e57c066b805694b10777c719502cca87 🚀
Parts:
- removed D1: APHHS1005LSECK/J3-PF, LED_SMD:LED_0402_1005Metric, symbol #dzdb:s_dio/D-KIN-APHHS1005LSECK/J3-PF
- removed TP1: Test Point, TestPoint:TestPoint_Pad_D1.5mm, symbol #dzdb:g_mech/M-TEST-SMT_1.5mm_round
- added LED8: 710-150060YS83000, dz_dio:Wuerth_LED_150060RS83000, symbol #dzdb:s_dio/D-WURT-710-150060YS83000
Connections:
- net Battery_Out_3.3V: now also LED8.2 (A)
- net at R5.2: now also LED8.1 (K)
Other:
- note added: "From the CM4 io board"
- note removed: "<---"
- note removed: "issue: will that logic work if I use USB vin only?"
- note removed: "only use when connected completely? not over usb???"
- note removed: "then I would in theory compare internal voltage with internal voltage... so probably not..."
- company: (none) -> Davide
- title: (none) -> Nautilus_Mainboard
