File: Browse/Piezzo.kicad_sch (KiCad schematic)
At the start: 5 parts, among them Q3 50V

Commit message: Deploying to gh-pages from @ Nautilus-UUV/nautilus-mainboard-PCB@b7db83c6a38e7ed72f880de916f2e48939069e27 🚀
Parts:
- removed LS1: ~, dz_mech:PT-1140PEQ, symbol #dzdb:s_misc/MALL-539-PT-1140PEQ
- added LS1: Piezo Buzzers & Audio Indicators 12mmx9mm deep Ma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, dz_mech:CMT1209590T, symbol #dzdb:s_mech/M-SAMESKY-CMT-1209-590T
- added R33: 10k, Resistor_SMD:R_0603_1608Metric, symbol #dzdb:g_res/R-10k-0603
Connections:
- net GND: now also R33.2
- net at R38.1, R39.2: now also LS1.1 (+)
- net at Q3.3, R38.2: now also LS1.2 (-)
- net at Q3.1, R40.2: now also R33.1
- net 10V renamed +5V
Other:
- moved on the sheet: R40

Commit message: Deploying to gh-pages from @ Nautilus-UUV/nautilus-mainboard-PCB@7631dd883fe8dd0df8a9e059de031ff5e1d7424d 🚀
Parts:
- removed R38: 1k, Resistor_SMD:R_0603_1608Metric, symbol #dzdb:g_res/R-1k-0603
- added D9: DDZ5V1B-7, dz_dio:SOD3716X145N, symbol #dzdb:s_dio/D-DIO-DDZ5V1B-7
Connections:
- net at LS1.1 (+), R39.2: now also D9.1
- net at LS1.2 (-), Q3.3: now also D9.2
Other:
- moved on the sheet: R39

Commit message: Deploying to gh-pages from @ Nautilus-UUV/nautilus-mainboard-PCB@2d3890115fd9d3c0bb909c9898aa64801bed9e67 🚀
Other:
- company: (none) -> Evan
Changed lines of the file:
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@@
 (kicad_sch (version 20250114) (generator "eeschema") (generator_version "9.0")
   (paper "A4")
+  (title_block
+    (date "2025-11-18")
+    (company "Evan")
+  )
   (junction (at 172.72 92.71) (diameter 0) (color 0 0 0 0)
   )

Commit message: Deploying to gh-pages from @ Nautilus-UUV/nautilus-mainboard-PCB@5b07cf6af03655ef9ddad269b1edd5eb03bfa75f 🚀
Other:
- title: (none) -> Nautilus_Mainboard
Changed lines of the file:
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@@
   (paper "A4")
   (title_block
+    (title "Nautilus_Mainboard")
     (date "2025-11-19")
     (rev "0")

Commit message: Deploying to gh-pages from @ Nautilus-UUV/nautilus-mainboard-PCB@5f5fdd9436d408a604bb268d740c0ac7ce1f5af5 🚀
Other:
- note removed: "Optimally replace the 1k with a fast switching diode."
- company: Evan -> (none)
- title: Nautilus_Mainboard -> (none)
Changed lines of the file:
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@@
 (kicad_sch (version 20250114) (generator "eeschema") (generator_version "9.0")
   (paper "A4")
-  (title_block
-    (title "Nautilus_Mainboard")
-    (date "2025-11-19")
-    (rev "0")
-    (company "Evan")
-  )
   (junction (at 172.72 92.71) (diameter 0) (color 0 0 0 0)
   )
@@
     (stroke (width 0) (type default))
   )
-  (text "Optimally replace the 1k with a\nfast switching diode. \n" (exclude_from_sim no) (at 146.05 84.328 0)
-    (effects (font (size 1.27 1.27)))
-  )
   (text "This 0R is a placeholder. \nApply different resistors to get different volumes\n" (exclude_from_sim no) (at 204.47 73.66 0)

Commit message: Deploying to gh-pages from @ Nautilus-UUV/nautilus-mainboard-PCB@f1dd6ce1e57c066b805694b10777c719502cca87 🚀
Other:
- note added: "Optimally replace the 1k with a fast switching diode."
- company: (none) -> Evan
- title: (none) -> Nautilus_Mainboard
Changed lines of the file:
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@@
 (kicad_sch (version 20250114) (generator "eeschema") (generator_version "9.0")
   (paper "A4")
+  (title_block
+    (title "Nautilus_Mainboard")
+    (date "2025-11-19")
+    (rev "0")
+    (company "Evan")
+  )
   (junction (at 172.72 92.71) (diameter 0) (color 0 0 0 0)
   )
@@
     (stroke (width 0) (type default))
   )
+  (text "Optimally replace the 1k with a\nfast switching diode. \n" (exclude_from_sim no) (at 146.05 84.328 0)
+    (effects (font (size 1.27 1.27)))
+  )
   (text "This 0R is a placeholder. \nApply different resistors to get different volumes\n" (exclude_from_sim no) (at 204.47 73.66 0)

Commit message: Deploying to gh-pages from @ Nautilus-UUV/nautilus-mainboard-PCB@7cbe43864a66a110f5cd8f57d0dac694c5d0b0c8 🚀
Parts:
- removed R39: 0, Resistor_SMD:R_0603_1608Metric, symbol #dzdb:g_res/R-0-0603
- added JP18: -, Jumper:SolderJumper-2_P1.3mm_Open_RoundedPad1.0x1.5mm, symbol #dzdb:g_mech/Jumper-2P1.3mm_Rounded
Connections:
- net +5V: now also JP18.2 (B)
- net at D9.1, LS1.1 (+): now also JP18.1 (A)
Changed lines of the file:
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@@
+    )
+  )
+  (symbol (lib_id "#dzdb:g_mech/Jumper-2P1.3mm_Rounded") (at 172.72 72.39 90) (unit 1)
+    (exclude_from_sim no) (in_bom no) (on_board yes) (dnp no)
+    (property "Reference" "JP18" (at 169.164 72.39 90)
+      (effects (font (size 1.27 1.27)))
+    )
+    (property "Value" "-" (at 170.688 73.406 90)
+      (effects (font (size 1.27 1.27)))
+    )
+    (property "Footprint" "Jumper:SolderJumper-2_P1.3mm_Open_RoundedPad1.0x1.5mm" (at 172.72 72.39 0)
+      (effects (font (size 1.27 1.27)) (hide yes))
+    )
+    (property "Datasheet" "~" (at 172.72 72.39 0)
+      (effects (font (size 1.27 1.27)) (hide yes))
+    )
+    (property "Description" "Solder Jumper" (at 172.72 72.39 0)
+      (effects (font (size 1.27 1.27)) (hide yes))
+    )
+    (property "IPN" "Jumper-2P1.3mm_Rounded" (at 172.72 72.39 0)
+      (effects (font (size 1.27 1.27)) (hide yes))
+    )
+    (property "Comments" "Rounded Jumper Pads 1.0x1.5mm" (at 172.72 72.39 0)
+      (effects (font (size 1.27 1.27)) (hide yes))
+    )
+    (pin "2")
+    (pin "1")
+    (instances
+      (project "nautilus_mainboard"
+        (path "/ce1819b2-f280-40ed-834f-6fe4d12f809d/7439593a-de4f-4d56-b463-481360a4f617"
+          (reference "JP18") (unit 1)
+        )
+      )
     )
   )
@@
         )
       )
-    )
-  )
-  (symbol (lib_id "#dzdb:g_res/R-0-0603") (at 172.72 72.39 0) (unit 1)
-    (exclude_from_sim no) (in_bom yes) (on_board yes) (dnp no) (fields_autoplaced)
-    (property "Reference" "R39" (at 175.26 71.1199 0)
-      (effects (font (size 1.27 1.27)) (justify left))
-    )
-    (property "Value" "0" (at 175.26 73.6599 0)
-      (effects (font (size 1.27 1.27)) (justify left))
-    )
-    (property "Footprint" "Resistor_SMD:R_0603_1608Metric" (at 170.942 72.39 90)
-      (effects (font (size 1.27 1.27)) (hide yes))
-    )
-    (property "Datasheet" "https://www.we-online.com/components/products/datasheet/560112116001.pdf" (at 172.72 72.39 0)
-      (effects (font (size 1.27 1.27)) (hide yes))
-    )
-    (property "Description" "Thick Film Resistors - SMD WRIS-RSKS <0.05 Ohms  0.1 W Jumper 0603" (at 172.72 72.39 0)
-      (effects (font (size 1.27 1.27)) (hide yes))
-    )
-    (property "IPN" "R-0-0603" (at 172.72 72.39 0)
-      (effects (font (size 1.27 1.27)) (hide yes))
-    )
-    (property "MPN" "560112116001" (at 172.72 72.39 0)
-      (effects (font (size 1.27 1.27)) (hide yes))
-    )
-    (property "Manufacturer" "Wurth Elektronik" (at 172.72 72.39 0)
-      (effects (font (size 1.27 1.27)) (hide yes))
-    )
-    (property "Resistance" "0" (at 172.72 72.39 0)
-      (effects (font (size 1.27 1.27)) (hide yes))
-    )
-    (property "Power" "0.1W" (at 172.72 72.39 0)
-      (effects (font (size 1.27 1.27)) (hide yes))
-    )
-    (property "Material" "Thick film" (at 172.72 72.39 0)
-      (effects (font (size 1.27 1.27)) (hide yes))
-    )
-    (property "Tolerance" "5%" (at 172.72 72.39 0)
-      (effects (font (size 1.27 1.27)) (hide yes))
-    )
-    (property "Supplier" "Mouser" (at 172.72 72.39 0)
-      (effects (font (size 1.27 1.27)) (hide yes))
-    )
-    (property "SPN" "710-560112116001" (at 172.72 72.39 0)
-      (effects (font (size 1.27 1.27)) (hide yes))
-    )
-    (property "LCSC" "CXXXXX" (at 172.72 72.39 0)
-      (effects (font (size 1.27 1.27)) (hide yes))
-    )
-    (property "Comment" "lifecycle=Active; note=Auto-generated" (at 172.72 72.39 0)
-      (effects (font (size 1.27 1.27)) (hide yes))
-    )
-    (pin "2")
-    (pin "1")
-    (instances
-      (project "nautilus_mainboard"
-        (path "/ce1819b2-f280-40ed-834f-6fe4d12f809d/7439593a-de4f-4d56-b463-481360a4f617"
-          (reference "R39") (unit 1)
-        )
-      )
