File: Browse/IMU1.kicad_sch (KiCad schematic)
At the start: 6 parts, among them U1 262-BMI088

Commit message: Deploying to gh-pages from @ Nautilus-UUV/nautilus-mainboard-PCB@5b07cf6af03655ef9ddad269b1edd5eb03bfa75f 🚀
Other:
- title: (none) -> Nautilus_Mainboard
Changed lines of the file:
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@@
   (paper "A4")
   (title_block
+    (title "Nautilus_Mainboard")
     (date "2025-11-19")
     (rev "0")

Commit message: Deploying to gh-pages from @ Nautilus-UUV/nautilus-mainboard-PCB@b731ca7531dd1e48b6b7a45790de08634e79c176 🚀
Parts:
- removed R50, R51, R53: 0, Resistor_SMD:R_0603_1608Metric, symbol #dzdb:g_res/R-0-0603
- added JP19, JP20, JP21: -, Jumper:SolderJumper-2_P1.3mm_Open_RoundedPad1.0x1.5mm, symbol #dzdb:g_mech/Jumper-2P1.3mm_Rounded
Connections:
- net BMI_In_3.3V: now also JP21.1 (A)
- net IMU_SCL: now also JP19.1 (A)
- net IMU_SDA: now also JP20.1 (A)
- net at U1.9 (SDA/SDI): now also JP20.2 (B)
- net at U1.8 (SCL/SCK): now also JP19.2 (B)
- net at U1.14 (CSB1), U1.7 (PS): now also JP21.2 (B)
