File: Browse/PCIE_Interface.kicad_sch (KiCad schematic)
At the start: 7 parts, among them J6 MDT275M02001

Commit message: Deploying to gh-pages from @ Nautilus-UUV/nautilus-mainboard-PCB@a81f7ffbfc5f9b51f47d7f388c30fcea2673b9ea 🚀
Connections:
- net PCIE_CLK_N renamed PCIE_CLK._N
- net PCIE_CLK_P renamed PCIE_CLK._P
- net PCIE_RX_N renamed PCIE_RX._N
- net PCIE_RX_P renamed PCIE_RX._P
- net PCIE_TX_N renamed PCIE_TX._N
- net PCIE_TX_P renamed PCIE_TX._P
Changed lines of the file:
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@@
   (no_connect (at 143.51 101.6))
   (no_connect (at 99.06 114.3))
+  (bus_entry (at 69.85 134.62) (size 2.54 2.54)
+    (stroke (width 0) (type default))
+  )
+  (bus_entry (at 74.93 144.78) (size 2.54 2.54)
+    (stroke (width 0) (type default))
+  )
+  (bus_entry (at 74.93 129.54) (size 2.54 2.54)
+    (stroke (width 0) (type default))
+  )
+  (bus_entry (at 69.85 137.16) (size 2.54 2.54)
+    (stroke (width 0) (type default))
+  )
+  (bus_entry (at 74.93 142.24) (size 2.54 2.54)
+    (stroke (width 0) (type default))
+  )
+  (bus_entry (at 74.93 127) (size 2.54 2.54)
+    (stroke (width 0) (type default))
+  )
   (wire (pts (xy 96.52 67.31) (xy 96.52 81.28))
     (stroke (width 0) (type default))
@@
     (stroke (width 0) (type default))
   )
-  (wire (pts (xy 80.01 144.78) (xy 118.11 144.78))
+  (bus (pts (xy 74.93 127) (xy 74.93 129.54))
     (stroke (width 0) (type default))
   )
@@
     (stroke (width 0) (type default))
   )
+  (bus (pts (xy 69.85 133.35) (xy 69.85 134.62))
+    (stroke (width 0) (type default))
+  )
   (wire (pts (xy 38.1 125.73) (xy 40.64 125.73))
     (stroke (width 0) (type default))
@@
     (stroke (width 0) (type default))
   )
+  (wire (pts (xy 72.39 139.7) (xy 118.11 139.7))
+    (stroke (width 0) (type default))
+  )
   (wire (pts (xy 99.06 99.06) (xy 118.11 99.06))
     (stroke (width 0) (type default))
   )
+  (wire (pts (xy 77.47 129.54) (xy 118.11 129.54))
+    (stroke (width 0) (type default))
+  )
   (wire (pts (xy 143.51 139.7) (xy 167.64 139.7))
     (stroke (width 0) (type default))
@@
     (stroke (width 0) (type default))
   )
+  (wire (pts (xy 77.47 147.32) (xy 118.11 147.32))
+    (stroke (width 0) (type default))
+  )
   (wire (pts (xy 96.52 170.18) (xy 130.81 170.18))
     (stroke (width 0) (type default))
@@
     (stroke (width 0) (type default))
   )
+  (wire (pts (xy 77.47 132.08) (xy 118.11 132.08))
+    (stroke (width 0) (type default))
+  )
   (wire (pts (xy 96.52 149.86) (xy 96.52 157.48))
     (stroke (width 0) (type default))
@@
     (stroke (width 0) (type default))
   )
-  (wire (pts (xy 74.93 139.7) (xy 118.11 139.7))
-    (stroke (width 0) (type default))
-  )
   (wire (pts (xy 143.51 160.02) (xy 158.75 160.02))
     (stroke (width 0) (type default))
@@
     (stroke (width 0) (type default))
   )
-  (wire (pts (xy 80.01 147.32) (xy 118.11 147.32))
-    (stroke (width 0) (type default))
-  )
   (wire (pts (xy 158.75 173.99) (xy 158.75 160.02))
     (stroke (width 0) (type default))
@@
     (stroke (width 0) (type default))
   )
-  (wire (pts (xy 74.93 137.16) (xy 118.11 137.16))
-    (stroke (width 0) (type default))
-  )
   (wire (pts (xy 96.52 142.24) (xy 118.11 142.24))
     (stroke (width 0) (type default))
@@
     (stroke (width 0) (type default))
   )
-  (wire (pts (xy 80.01 129.54) (xy 118.11 129.54))
-    (stroke (width 0) (type default))
-  )
   (wire (pts (xy 96.52 119.38) (xy 118.11 119.38))
     (stroke (width 0) (type default))
@@
     (stroke (width 0) (type default))
   )
+  (wire (pts (xy 77.47 144.78) (xy 118.11 144.78))
+    (stroke (width 0) (type default))
+  )
   (wire (pts (xy 96.52 111.76) (xy 96.52 96.52))
     (stroke (width 0) (type default))
   )
+  (bus (pts (xy 74.93 142.24) (xy 74.93 144.78))
+    (stroke (width 0) (type default))
+  )
   (wire (pts (xy 113.03 152.4) (xy 118.11 152.4))
     (stroke (width 0) (type default))
@@
     (stroke (width 0) (type default))
   )
-  (wire (pts (xy 80.01 132.08) (xy 118.11 132.08))
-    (stroke (width 0) (type default))
-  )
   (wire (pts (xy 96.52 96.52) (xy 96.52 88.9))
     (stroke (width 0) (type default))
@@
     (stroke (width 0) (type default))
   )
+  (wire (pts (xy 72.39 137.16) (xy 118.11 137.16))
+    (stroke (width 0) (type default))
+  )
   (wire (pts (xy 143.51 93.98) (xy 158.75 93.98))
     (stroke (width 0) (type default))
   )
+  (bus (pts (xy 69.85 134.62) (xy 69.85 137.16))
+    (stroke (width 0) (type default))
+  )
   (wire (pts (xy 96.52 96.52) (xy 118.11 96.52))
     (stroke (width 0) (type default))
@@
     (stroke (width 0) (type default))
   )
+  (bus (pts (xy 74.93 124.46) (xy 74.93 127))
+    (stroke (width 0) (type default))
+  )
   (wire (pts (xy 99.06 109.22) (xy 118.11 109.22))
+    (stroke (width 0) (type default))
+  )
+  (bus (pts (xy 74.93 140.97) (xy 74.93 142.24))
     (stroke (width 0) (type default))
   )
@@
     (effects (font (size 1.27 1.27)) (justify left bottom))
   )
+  (label "PCIE_TX._P" (at 74.93 139.7 0)
+    (effects (font (size 1.27 1.27)) (justify left bottom))
+  )
   (label "PETp2" (at 99.06 109.22 0)
     (effects (font (size 1.27 1.27)) (justify left bottom))
@@
     (effects (font (size 1.27 1.27)) (justify left bottom))
   )
+  (label "PCIE_CLK._N" (at 80.01 144.78 0)
+    (effects (font (size 1.27 1.27)) (justify left bottom))
+  )
+  (label "PCIE_RX._P" (at 80.01 132.08 0)
+    (effects (font (size 1.27 1.27)) (justify left bottom))
+  )
   (label "PETp1" (at 99.06 124.46 0)
     (effects (font (size 1.27 1.27)) (justify left bottom))
@@
     (effects (font (size 1.27 1.27)) (justify left bottom))
   )
+  (label "PCIE_RX._N" (at 80.01 129.54 0)
+    (effects (font (size 1.27 1.27)) (justify left bottom))
+  )
   (label "PERST#" (at 148.59 139.7 0)
     (effects (font (size 1.27 1.27)) (justify left bottom))
@@
     (effects (font (size 1.27 1.27)) (justify left bottom))
   )
+  (label "PCIE_CLK._P" (at 80.01 147.32 0)
+    (effects (font (size 1.27 1.27)) (justify left bottom))
+  )
   (label "PERn2" (at 99.06 99.06 0)
     (effects (font (size 1.27 1.27)) (justify left bottom))
@@
     (effects (font (size 1.27 1.27)) (justify left bottom))
   )
+  (label "PCIE_TX._N" (at 74.93 137.16 0)
+    (effects (font (size 1.27 1.27)) (justify left bottom))
+  )
   (label "PEWAKE#" (at 148.59 144.78 0)
     (effects (font (size 1.27 1.27)) (justify left bottom))
@@
     (effects (font (size 1.27 1.27)) (justify left bottom))
   )
-  (global_label "Battery_Out_3.3V" (shape input) (at 158.75 173.99 180) (fields_autoplaced)
-    (effects (font (size 1.27 1.27)) (justify right))
-    (property "Intersheetrefs" "${INTERSHEET_REFS}" (at 139.7992 173.99 0)
-      (effects (font (size 1.27 1.27)) (justify right) (hide yes))
-    )
-  )
-  (hierarchical_label "PCIE_RX_N" (shape bidirectional) (at 80.01 129.54 180)
-    (effects (font (size 1.27 1.27)) (justify right))
+  (hierarchical_label "PCIE_CLK{_N,_P}" (shape bidirectional) (at 74.93 140.97 0)
+    (effects (font (size 1.27 1.27)) (justify left))
+  )
+  (hierarchical_label "PCIE_TX{_N,_P}" (shape bidirectional) (at 69.85 133.35 0)
+    (effects (font (size 1.27 1.27)) (justify left))
   )
   (hierarchical_label "PCIE_nRST" (shape input) (at 167.64 139.7 0)
     (effects (font (size 1.27 1.27)) (justify left))
   )
-  (hierarchical_label "PCIE_TX_P" (shape bidirectional) (at 74.93 139.7 180)
+  (hierarchical_label "Battery_Out_3.3V" (shape input) (at 158.75 173.99 180)
     (effects (font (size 1.27 1.27)) (justify right))
   )
-  (hierarchical_label "PCIE_TX_N" (shape bidirectional) (at 74.93 137.16 180)
-    (effects (font (size 1.27 1.27)) (justify right))
-  )
-  (hierarchical_label "PCIE_CLK_P" (shape bidirectional) (at 80.01 147.32 180)
-    (effects (font (size 1.27 1.27)) (justify right))
-  )
-  (hierarchical_label "PCIE_RX_P" (shape bidirectional) (at 80.01 132.08 180)
-    (effects (font (size 1.27 1.27)) (justify right))
-  )
-  (hierarchical_label "PCIE_CLK_N" (shape bidirectional) (at 80.01 144.78 180)
-    (effects (font (size 1.27 1.27)) (justify right))
+  (hierarchical_label "PCIE_RX{_N,_P}" (shape bidirectional) (at 74.93 124.46 0)
+    (effects (font (size 1.27 1.27)) (justify left))
   )
   (symbol (lib_id "#dzdb:g_res/R-0-0603") (at 34.29 120.65 90) (unit 1)

Commit message: Deploying to gh-pages from @ Nautilus-UUV/nautilus-mainboard-PCB@2d3890115fd9d3c0bb909c9898aa64801bed9e67 🚀
Other:
- company: (none) -> Davide
Changed lines of the file:
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@@
 (kicad_sch (version 20250114) (generator "eeschema") (generator_version "9.0")
   (paper "A4")
+  (title_block
+    (date "2025-11-18")
+    (company "Davide")
+  )
   (junction (at 96.52 157.48) (diameter 0) (color 0 0 0 0)
   )

Commit message: Deploying to gh-pages from @ Nautilus-UUV/nautilus-mainboard-PCB@8b02e89ade7c168188296ba6f0516f3abec9166b 🚀
Parts:
- removed CONFIG_1, CONFIG_2, CONFIG_3, CONFIG_4: 0, Resistor_SMD:R_0603_1608Metric, symbol #dzdb:g_res/R-0-0603
- removed D8: APHHS1005LCGCK, LED_SMD:LED_0402_1005Metric, symbol #dzdb:s_dio/D-KIN-APHHS1005LCGCK
- added LED4: 710-150060VS83000, dz_dio:Wuerth_LED_150060RS83000, symbol #dzdb:s_dio/D-WURT-710-150060VS83000
- added R19, R20, R21, R23: 0, Resistor_SMD:R_0603_1608Metric, symbol #dzdb:g_res/R-0-0603
Connections:
- net CONFIG_0: now also R19.2
- net CONFIG_1: now also R20.2
- net CONFIG_2: now also R21.2
- net CONFIG_3: now also R23.2
- net GND: now also LED4.1 (K), R19.1, R20.1, R21.1, R23.1
- net LED1_M2: now also LED4.2 (A)

Commit message: Deploying to gh-pages from @ Nautilus-UUV/nautilus-mainboard-PCB@5b07cf6af03655ef9ddad269b1edd5eb03bfa75f 🚀
Other:
- title: (none) -> Nautilus_Mainboard
Changed lines of the file:
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@@
   (paper "A4")
   (title_block
+    (title "Nautilus_Mainboard")
     (date "2025-11-19")
     (rev "0")

Commit message: Deploying to gh-pages from @ Nautilus-UUV/nautilus-mainboard-PCB@7cbe43864a66a110f5cd8f57d0dac694c5d0b0c8 🚀
Parts:
- removed R19, R20, R21, R23: 0, Resistor_SMD:R_0603_1608Metric, symbol #dzdb:g_res/R-0-0603
- added JP14, JP15, JP16, JP17: -, Jumper:SolderJumper-2_P1.3mm_Open_RoundedPad1.0x1.5mm, symbol #dzdb:g_mech/Jumper-2P1.3mm_Rounded
Connections:
- net CONFIG_0: now also JP14.2 (B)
- net CONFIG_1: now also JP15.2 (B)
- net CONFIG_2: now also JP16.2 (B)
- net CONFIG_3: now also JP17.2 (B)
- net GND: now also JP14.1 (A), JP15.1 (A), JP16.1 (A), JP17.1 (A)

Commit message: Deploying to gh-pages from @ Nautilus-UUV/nautilus-mainboard-PCB@b731ca7531dd1e48b6b7a45790de08634e79c176 🚀
Changed lines of the file:
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@@
     (pin "57")
     (pin "56")
+    (pin "59")
     (instances
       (project "nautilus_mainboard"
